File: Projects/StationModules/Module_1/Module_1.kicad_pcb (KiCad board)
At the start: 2 copper layers, 156 x 101.5 mm, 139 parts, among them J2 +310, J3 -310, J4 PowerTrans1, J5 PowerTrans2, M1 BluePillStm32, Q1 STD20NF06T4, Q2 STD20NF06T4, Q3 STD20NF06T4, Q4 STD20NF06T4, Q5 IRGB10B60KD, Q6 IRGB10B60KD, Q7 IRGB10B60KD, Q8 IRGB10B60KD, T1 Transformer_SP_2S, T2 Transformer_SP_2S, U1 PC817, U2 L7805, U3 TC1047AxNB, U5 LM311, U6 6N137

Commit message: add bom and pos
Changed lines of the file:
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@@
       (plot_on_all_layers_selection 0x0000000_00000000)
       (disableapertmacros false)
-      (usegerberextensions false)
-      (usegerberattributes true)
-      (usegerberadvancedattributes true)
-      (creategerberjobfile true)
+      (usegerberextensions true)
+      (usegerberattributes false)
+      (usegerberadvancedattributes false)
+      (creategerberjobfile false)
       (dashed_line_dash_ratio 12.000000)
       (dashed_line_gap_ratio 3.000000)
@@
       (psa4output false)
       (plotreference true)
-      (plotvalue true)
+      (plotvalue false)
       (plotinvisibletext false)
       (sketchpadsonfab false)
-      (subtractmaskfromsilk false)
+      (subtractmaskfromsilk true)
       (outputformat 1)
       (mirror false)
       (drillshape 0)
       (scaleselection 1)
-      (outputdirectory "Prod/")
+      (outputdirectory "Module_1_gerbers/")
     )
   )
@@
     (fp_line (start 3.55 2.1) (end 3.55 -2.1)
       (stroke (width 0.1) (type solid)) (layer "B.Fab"))
-    (pad "1" smd roundrect (at -2.5125 0 180) (size 3.025 4.45) (layers "B.Cu" "B.Paste" "B.Mask") (roundrect_rratio 0.082645)
+    (pad "1" smd roundrect (at -2.5125 0 180) (size 3.025 4.45) (layers "B.Cu" "B.Paste" "B.Mask") (roundrect_rratio 0.08264495868)
       (net 50 "/Shunt+") (pintype "passive"))
-    (pad "2" smd roundrect (at 2.5125 0 180) (size 3.025 4.45) (layers "B.Cu" "B.Paste" "B.Mask") (roundrect_rratio 0.082645)
+    (pad "2" smd roundrect (at 2.5125 0 180) (size 3.025 4.45) (layers "B.Cu" "B.Paste" "B.Mask") (roundrect_rratio 0.08264495868)
       (net 12 "/Shunt-") (pintype "passive"))
     (model "${KICAD6_3DMODEL_DIR}/Resistor_SMD.3dshapes/R_2816_7142Metric.wrl"
@@
     (fp_line (start 3.55 2.1) (end 3.55 -2.1)
       (stroke (width 0.1) (type solid)) (layer "B.Fab"))
-    (pad "1" smd roundrect (at -2.5125 0 180) (size 3.025 4.45) (layers "B.Cu" "B.Paste" "B.Mask") (roundrect_rratio 0.082645)
+    (pad "1" smd roundrect (at -2.5125 0 180) (size 3.025 4.45) (layers "B.Cu" "B.Paste" "B.Mask") (roundrect_rratio 0.08264495868)
       (net 50 "/Shunt+") (pintype "passive"))
-    (pad "2" smd roundrect (at 2.5125 0 180) (size 3.025 4.45) (layers "B.Cu" "B.Paste" "B.Mask") (roundrect_rratio 0.082645)
+    (pad "2" smd roundrect (at 2.5125 0 180) (size 3.025 4.45) (layers "B.Cu" "B.Paste" "B.Mask") (roundrect_rratio 0.08264495868)
       (net 12 "/Shunt-") (pintype "passive"))
     (model "${KICAD6_3DMODEL_DIR}/Resistor_SMD.3dshapes/R_2816_7142Metric.wrl"
@@
     (fp_line (start 3.65 2.15) (end -2.65 2.15)
       (stroke (width 0.1) (type solid)) (layer "B.Fab"))
-    (pad "1" smd roundrect (at -3.1125 0) (size 2.075 2.55) (layers "B.Cu" "B.Paste" "B.Mask") (roundrect_rratio 0.120482)
+    (pad "1" smd roundrect (at -3.1125 0) (size 2.075 2.55) (layers "B.Cu" "B.Paste" "B.Mask") (roundrect_rratio 0.1204819277)
       (net 3 "+12V") (pintype "passive"))
-    (pad "2" smd roundrect (at 3.1125 0) (size 2.075 2.55) (layers "B.Cu" "B.Paste" "B.Mask") (roundrect_rratio 0.120482)
+    (pad "2" smd roundrect (at 3.1125 0) (size 2.075 2.55) (layers "B.Cu" "B.Paste" "B.Mask") (roundrect_rratio 0.1204819277)
       (net 1 "GND") (pintype "passive"))
     (model "${KICAD6_3DMODEL_DIR}/Capacitor_Tantalum_SMD.3dshapes/CP_EIA-7343-15_Kemet-W.wrl"
@@
     (fp_line (start 1.6 0.8) (end 1.6 -0.8)
       (stroke (width 0.1) (type solid)) (layer "B.Fab"))
-    (pad "1" smd roundrect (at -1.475 0 180) (size 1.15 1.8) (layers "B.Cu" "B.Paste" "B.Mask") (roundrect_rratio 0.217391)
+    (pad "1" smd roundrect (at -1.475 0 180) (size 1.15 1.8) (layers "B.Cu" "B.Paste" "B.Mask") (roundrect_rratio 0.2173913043)
       (net 52 "/OS") (pintype "passive"))
-    (pad "2" smd roundrect (at 1.475 0 180) (size 1.15 1.8) (layers "B.Cu" "B.Paste" "B.Mask") (roundrect_rratio 0.217391)
+    (pad "2" smd roundrect (at 1.475 0 180) (size 1.15 1.8) (layers "B.Cu" "B.Paste" "B.Mask") (roundrect_rratio 0.2173913043)
       (net 1 "GND") (pintype "passive"))
     (model "${KICAD6_3DMODEL_DIR}/Capacitor_SMD.3dshapes/C_1206_3216Metric.wrl"
@@
     (fp_line (start 3.55 2.1) (end 3.55 -2.1)
       (stroke (width 0.1) (type solid)) (layer "B.Fab"))
-    (pad "1" smd roundrect (at -2.5125 0 180) (size 3.025 4.45) (layers "B.Cu" "B.Paste" "B.Mask") (roundrect_rratio 0.082645)
+    (pad "1" smd roundrect (at -2.5125 0 180) (size 3.025 4.45) (layers "B.Cu" "B.Paste" "B.Mask") (roundrect_rratio 0.08264495868)
       (net 50 "/Shunt+") (pintype "passive"))
-    (pad "2" smd roundrect (at 2.5125 0 180) (size 3.025 4.45) (layers "B.Cu" "B.Paste" "B.Mask") (roundrect_rratio 0.082645)
+    (pad "2" smd roundrect (at 2.5125 0 180) (size 3.025 4.45) (layers "B.Cu" "B.Paste" "B.Mask") (roundrect_rratio 0.08264495868)
       (net 12 "/Shunt-") (pintype "passive"))
     (model "${KICAD6_3DMODEL_DIR}/Resistor_SMD.3dshapes/R_2816_7142Metric.wrl"
