File: Projects/StationModules/Module_1/Module_1.kicad_pcb (KiCad board)
At the start: 2 copper layers, 156 x 101.5 mm, 139 parts, among them J2 +310, J3 -310, J4 PowerTrans1, J5 PowerTrans2, M1 BluePillStm32, Q1 STD20NF06T4, Q2 STD20NF06T4, Q3 STD20NF06T4, Q4 STD20NF06T4, Q5 IRGB10B60KD, Q6 IRGB10B60KD, Q7 IRGB10B60KD, Q8 IRGB10B60KD, T1 Transformer_SP_2S, T2 Transformer_SP_2S, U1 PC817, U2 L7805, U3 TC1047AxNB, U5 LM311, U6 6N137

Commit message: change module1,2
Parts:
- C10, C9: value 10pF -> 10nF
- C23, C24, C25, C26: value 2n2 600v -> 1n 630v
- C28: value 0,1u 600V -> 0,47u 600V
- J4, J5: footprint Z_pin:PinD4mm -> Z_pin:PinD3mm
- Q5, Q6, Q7, Q8: value IRGB10B60KD -> STW20NM60
- R16: value 360 -> 150
- R19, R20, R21, R22: value 3,6k -> 3,3k
- R23, R24, R25, R26: value 360 -> 75
- R27, R28: value 300 -> 330
- R29, R30, R31, R32: value 20 -> 75
- R3, R4: value 4k7 -> 4,7k
- R40, R41, R42, R43: value 18 2W -> 18
- RV1, RV2: value 4k7 3296W -> 5k
- U4: value ~ -> 78L05S

Commit message: Corection all modules
Parts:
- added J6: -310V, TestPoint:TestPoint_THTPad_2.5x2.5mm_Drill1.2mm, F.Cu at (130.7, 133.2)
- added J7: -12V, TestPoint:TestPoint_THTPad_2.5x2.5mm_Drill1.2mm, F.Cu at (112.8, 40.4)
- added TP1: TestPoint, TestPoint:TestPoint_Pad_2.0x2.0mm, F.Cu at (158.2, 36.6)
- added TP2: TestPoint, TestPoint:TestPoint_Pad_2.0x2.0mm, F.Cu at (101.3, 134.9)
- added TP3: TestPoint, TestPoint:TestPoint_Pad_2.0x2.0mm, F.Cu at (97.8, 120.4)
- C17: value 1n -> 2,2n
Routing:
- net /Shunt-: track 114.5 -> 122.8 mm
- net Net-(U5-+): track 20.0 -> 27.1 mm, vias 0 -> 1
- net Net-(U6-C): track 11.3 -> 16.7 mm
- net /TMP: track 138.9 -> 142.2 mm, vias 0 -> 1

Commit message: change for final 20.03.2024
Parts:
- J4, J5: footprint Z_pin:PinD3mm -> Z_pin:PinD2mm
- renumbered TP2 to P, TP1 to T
Changed lines of the file:
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@@
     (property "ki_keywords" "test point tp")
     (attr exclude_from_pos_files)
-    (fp_text reference "TP1" (at -2.921 -0.635) (layer "F.SilkS")
+    (fp_text reference "T" (at -2.921 -0.635) (layer "F.SilkS")
         (effects (font (size 1 1) (thickness 0.15)))
     )
@@
     )
   )
-  (footprint "Z_pin:PinD3mm" (layer "F.Cu")
+  (footprint "Z_pin:PinD2mm" (layer "F.Cu")
     (at 206 122)
     (property "Description" "")
@@
     (property "ki_keywords" "screw terminal")
     (attr through_hole)
-    (fp_text reference "J5" (at 5.582 -0.334 unlocked) (layer "F.SilkS")
+    (fp_text reference "J5" (at 5.328 -2.112 unlocked) (layer "F.SilkS")
         (effects (font (size 1 1) (thickness 0.1)))
     )
@@
         (effects (font (size 1 1) (thickness 0.15)))
     )
-    (fp_rect (start -3.556 -3.429) (end 3.556 3.429)
+    (fp_rect (start -2.54 -2.54) (end 2.54 2.54)
       (stroke (width 0.1) (type default)) (fill none) (layer "F.SilkS"))
-    (pad "1" thru_hole circle (at 0 0) (size 6 6) (drill 3) (layers "*.Cu" "*.Mask")
+    (pad "1" thru_hole circle (at 0 0) (size 4 4) (drill 2) (layers "*.Cu" "*.Mask")
       (net 26 "Net-(D18-A2)") (pinfunction "Pin_1") (pintype "passive"))
   )
-  (footprint "Z_pin:PinD3mm" (layer "F.Cu")
+  (footprint "Z_pin:PinD2mm" (layer "F.Cu")
     (at 206 86)
     (property "Description" "")
@@
     (property "ki_keywords" "screw terminal")
     (attr through_hole)
-    (fp_text reference "J4" (at 5.328 -0.402 unlocked) (layer "F.SilkS")
+    (fp_text reference "J4" (at 5.074 -1.926 unlocked) (layer "F.SilkS")
         (effects (font (size 1 1) (thickness 0.1)))
     )
@@
         (effects (font (size 1 1) (thickness 0.15)))
     )
-    (fp_rect (start -3.556 -3.429) (end 3.556 3.429)
+    (fp_rect (start -2.54 -2.54) (end 2.54 2.54)
       (stroke (width 0.1) (type default)) (fill none) (layer "F.SilkS"))
-    (pad "1" thru_hole circle (at 0 0) (size 6 6) (drill 3) (layers "*.Cu" "*.Mask")
+    (pad "1" thru_hole circle (at 0 0) (size 4 4) (drill 2) (layers "*.Cu" "*.Mask")
       (net 28 "Net-(J4-Pin_1)") (pinfunction "Pin_1") (pintype "passive"))
   )
@@
     (property "ki_keywords" "test point tp")
     (attr exclude_from_pos_files)
-    (fp_text reference "TP2" (at 0 -1.998) (layer "F.SilkS")
-        (effects (font (size 1 1) (thickness 0.15)))
-    )
+    (fp_text reference "P" (at 2.286 0.508) (layer "F.SilkS")
+        (effects (font (size 1 1) (thickness 0.15)))
+    )
