File: Projects/StationModules/Module_1/DriverFet.kicad_sch (KiCad schematic)
At the start: 22 parts, among them Q1 STD20NF06T4, Q2 STD20NF06T4

Commit message: add bom module 1
Parts:
- C15: LCSC (none) -> C277483; MFR.Part (none) -> CC1206KKX7R9BB474
- C17: LCSC (none) -> C527247; MFR.Part (none) -> CC1206GRNPO9BN102
- D5, D6: LCSC (none) -> C2891733; MFR.Part (none) -> LL4148
- Q1, Q2: LCSC (none) -> C668203; MFR.Part (none) -> STD20NF06L
- R13, R14: value 3,6k -> 3,3k; LCSC (none) -> C125845; MFR.Part (none) -> RC1206JR-073K3L
- R18, R19: LCSC (none) -> C246069; MFR.Part (none) -> RC1206JR-07360RL
- R22: value 300 -> 330; LCSC (none) -> C137152; MFR.Part (none) -> RC1206JR-07330RL

Commit message: finaly on summer
Parts:
- R13, R14: LCSC C125845 -> C26041; MFR.Part RC1206JR-073K3L -> 1206W4J0332T5E
Changed lines of the file:
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@@
       (effects (font (size 1.27 1.27)) hide)
     )
-    (property "MFR.Part" "RC1206JR-073K3L" (at 62.23 123.19 0)
+    (property "MFR.Part" "1206W4J0332T5E" (at 62.23 123.19 0)
       (effects (font (size 1.27 1.27)) hide)
     )
@@
       (effects (font (size 1.27 1.27)) hide)
     )
-    (property "LCSC" "C125845" (at 62.23 123.19 0)
+    (property "LCSC" "C26041" (at 62.23 123.19 0)
       (effects (font (size 1.27 1.27)) hide)
     )
@@
       (effects (font (size 1.27 1.27)) hide)
     )
-    (property "MFR.Part" "RC1206JR-073K3L" (at 62.23 62.23 0)
+    (property "MFR.Part" "1206W4J0332T5E" (at 62.23 62.23 0)
       (effects (font (size 1.27 1.27)) hide)
     )
@@
       (effects (font (size 1.27 1.27)) hide)
     )
-    (property "LCSC" "C125845" (at 62.23 62.23 0)
+    (property "LCSC" "C26041" (at 62.23 62.23 0)
       (effects (font (size 1.27 1.27)) hide)
     )
@@
       (effects (font (size 1.27 1.27)) hide)
     )
-    (property "MFR.Part" "RC1206JR-073K3L" (at 62.23 113.03 0)
+    (property "MFR.Part" "1206W4J0332T5E" (at 62.23 113.03 0)
       (effects (font (size 1.27 1.27)) hide)
     )
@@
       (effects (font (size 1.27 1.27)) hide)
     )
-    (property "LCSC" "C125845" (at 62.23 113.03 0)
+    (property "LCSC" "C26041" (at 62.23 113.03 0)
       (effects (font (size 1.27 1.27)) hide)
     )
@@
       (effects (font (size 1.27 1.27)) hide)
     )
-    (property "MFR.Part" "RC1206JR-073K3L" (at 62.23 52.07 0)
+    (property "MFR.Part" "1206W4J0332T5E" (at 62.23 52.07 0)
       (effects (font (size 1.27 1.27)) hide)
     )
@@
       (effects (font (size 1.27 1.27)) hide)
     )
-    (property "LCSC" "C125845" (at 62.23 52.07 0)
-      (effects (font (size 1.27 1.27)) hide)
-    )
+    (property "LCSC" "C26041" (at 62.23 52.07 0)
+      (effects (font (size 1.27 1.27)) hide)
+    )

Commit message: change module1,2
Parts:
- R18, R19: value 360 -> 75; LCSC C246069 -> C17987; MFR.Part RC1206JR-07360RL -> 1206W4F750JT5E
Changed lines of the file:
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@@
       (effects (font (size 1.27 1.27)))
     )
-    (property "Value" "360" (at 80.01 43.18 90)
+    (property "Value" "75" (at 80.01 43.18 90)
       (effects (font (size 1.27 1.27)))
     )
@@
       (effects (font (size 1.27 1.27)) hide)
     )
-    (property "MFR.Part" "RC1206JR-07360RL" (at 80.01 45.72 0)
-      (effects (font (size 1.27 1.27)) hide)
-    )
-    (property "Description" "250mW Thick Film Resistors ±100ppm/℃ ±5% 360Ω 1206 Chip Resistor - Surface Mount ROHS" (at 80.01 45.72 0)
-      (effects (font (size 1.27 1.27)) hide)
-    )
-    (property "LCSC" "C246069" (at 80.01 45.72 0)
+    (property "MFR.Part" "1206W4F750JT5E" (at 80.01 45.72 0)
+      (effects (font (size 1.27 1.27)) hide)
+    )
+    (property "Description" "250mW Thick Film Resistors ±100ppm/℃ ±1% 75Ω 1206 Chip Resistor - Surface Mount ROHS" (at 80.01 45.72 0)
+      (effects (font (size 1.27 1.27)) hide)
+    )
+    (property "LCSC" "C17987" (at 80.01 45.72 0)
       (effects (font (size 1.27 1.27)) hide)
     )
@@
       (effects (font (size 1.27 1.27)))
     )
-    (property "Value" "360" (at 80.01 104.14 90)
+    (property "Value" "75" (at 80.01 104.14 90)
       (effects (font (size 1.27 1.27)))
     )
@@
       (effects (font (size 1.27 1.27)) hide)
     )
-    (property "MFR.Part" "RC1206JR-07360RL" (at 80.01 106.68 0)
-      (effects (font (size 1.27 1.27)) hide)
-    )
-    (property "Description" "250mW Thick Film Resistors ±100ppm/℃ ±5% 360Ω 1206 Chip Resistor - Surface Mount ROHS" (at 80.01 106.68 0)
-      (effects (font (size 1.27 1.27)) hide)
-    )
-    (property "LCSC" "C246069" (at 80.01 106.68 0)
+    (property "MFR.Part" "1206W4F750JT5E" (at 80.01 106.68 0)
+      (effects (font (size 1.27 1.27)) hide)
+    )
+    (property "Description" "250mW Thick Film Resistors ±100ppm/℃ ±1% 75Ω 1206 Chip Resistor - Surface Mount ROHS" (at 80.01 106.68 0)
+      (effects (font (size 1.27 1.27)) hide)
+    )
+    (property "LCSC" "C17987" (at 80.01 106.68 0)
       (effects (font (size 1.27 1.27)) hide)
     )
@@
       (effects (font (size 1.27 1.27)))
     )
-    (property "Value" "360" (at 80.01 66.04 90)
+    (property "Value" "75" (at 80.01 66.04 90)
       (effects (font (size 1.27 1.27)))
     )
@@
       (effects (font (size 1.27 1.27)) hide)
     )
-    (property "MFR.Part" "RC1206JR-07360RL" (at 80.01 68.58 0)
-      (effects (font (size 1.27 1.27)) hide)
-    )
-    (property "Description" "250mW Thick Film Resistors ±100ppm/℃ ±5% 360Ω 1206 Chip Resistor - Surface Mount ROHS" (at 80.01 68.58 0)
-      (effects (font (size 1.27 1.27)) hide)
-    )
-    (property "LCSC" "C246069" (at 80.01 68.58 0)
+    (property "MFR.Part" "1206W4F750JT5E" (at 80.01 68.58 0)
+      (effects (font (size 1.27 1.27)) hide)
+    )
+    (property "Description" "250mW Thick Film Resistors ±100ppm/℃ ±1% 75Ω 1206 Chip Resistor - Surface Mount ROHS" (at 80.01 68.58 0)
+      (effects (font (size 1.27 1.27)) hide)
+    )
+    (property "LCSC" "C17987" (at 80.01 68.58 0)
       (effects (font (size 1.27 1.27)) hide)
     )
@@
       (effects (font (size 1.27 1.27)))
     )
-    (property "Value" "360" (at 80.01 127 90)
+    (property "Value" "75" (at 80.01 127 90)
       (effects (font (size 1.27 1.27)))
     )
@@
       (effects (font (size 1.27 1.27)) hide)
     )
-    (property "MFR.Part" "RC1206JR-07360RL" (at 80.01 129.54 0)
-      (effects (font (size 1.27 1.27)) hide)
-    )
-    (property "Description" "250mW Thick Film Resistors ±100ppm/℃ ±5% 360Ω 1206 Chip Resistor - Surface Mount ROHS" (at 80.01 129.54 0)
-      (effects (font (size 1.27 1.27)) hide)
-    )
-    (property "LCSC" "C246069" (at 80.01 129.54 0)
-      (effects (font (size 1.27 1.27)) hide)
-    )
+    (property "MFR.Part" "1206W4F750JT5E" (at 80.01 129.54 0)
+      (effects (font (size 1.27 1.27)) hide)
+    )
+    (property "Description" "250mW Thick Film Resistors ±100ppm/℃ ±1% 75Ω 1206 Chip Resistor - Surface Mount ROHS" (at 80.01 129.54 0)
+      (effects (font (size 1.27 1.27)) hide)
+    )
+    (property "LCSC" "C17987" (at 80.01 129.54 0)
+      (effects (font (size 1.27 1.27)) hide)
+    )

Commit message: change on 25_02_24
Parts:
- C15, C17, D5, D6, Q1, Q2, R13, R14, R18, R19, R22: Mounting (none) -> Yes
Changed lines of the file:
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@@
+      (effects (font (size 1.27 1.27)) hide)
+    )
+    (property "Mounting" "Yes" (at 62.23 123.19 0)
       (effects (font (size 1.27 1.27)) hide)
     )
@@
       (effects (font (size 1.27 1.27)) hide)
     )
+    (property "Mounting" "Yes" (at 80.01 45.72 0)
+      (effects (font (size 1.27 1.27)) hide)
+    )
     (pin "1")
     (pin "2")
@@
       (effects (font (size 1.27 1.27)) hide)
     )
+    (property "Mounting" "Yes" (at 121.92 129.54 0)
+      (effects (font (size 1.27 1.27)) hide)
+    )
     (pin "1")
     (pin "2")
@@
       (effects (font (size 1.27 1.27)) hide)
     )
+    (property "Mounting" "Yes" (at 80.01 76.2 0)
+      (effects (font (size 1.27 1.27)) hide)
+    )
     (pin "1")
     (pin "2")
@@
       (effects (font (size 1.27 1.27)) hide)
     )
+    (property "Mounting" "Yes" (at 121.92 106.68 0)
+      (effects (font (size 1.27 1.27)) hide)
+    )
     (pin "1")
     (pin "2")
@@
       (effects (font (size 1.27 1.27)) hide)
     )
+    (property "Mounting" "Yes" (at 80.01 38.1 0)
+      (effects (font (size 1.27 1.27)) hide)
+    )
     (pin "1")
     (pin "2")
@@
       (effects (font (size 1.27 1.27)) hide)
     )
+    (property "Mounting" "Yes" (at 80.01 106.68 0)
+      (effects (font (size 1.27 1.27)) hide)
+    )
     (pin "1")
     (pin "2")
@@
       (effects (font (size 1.27 1.27)) hide)
     )
+    (property "Mounting" "Yes" (at 80.01 137.16 0)
+      (effects (font (size 1.27 1.27)) hide)
+    )
     (pin "1")
     (pin "2")
@@
       (effects (font (size 1.27 1.27)) hide)
     )
+    (property "Mounting" "Yes" (at 110.49 118.11 0)
+      (effects (font (size 1.27 1.27)) hide)
+    )
     (pin "1")
     (pin "2")
@@
     )
     (property "LCSC" "C17987" (at 80.01 68.58 0)
+      (effects (font (size 1.27 1.27)) hide)
+    )
+    (property "Mounting" "Yes" (at 80.01 68.58 0)
       (effects (font (size 1.27 1.27)) hide)
     )
@@
       (effects (font (size 1.27 1.27)) hide)
     )
+    (property "Mounting" "Yes" (at 100.33 68.58 0)
+      (effects (font (size 1.27 1.27)) hide)
+    )
     (pin "1")
     (pin "2")
@@
       (effects (font (size 1.27 1.27)) hide)
     )
+    (property "Mounting" "Yes" (at 121.92 68.58 0)
+      (effects (font (size 1.27 1.27)) hide)
+    )
     (pin "1")
     (pin "2")
@@
     )
     (property "LCSC" "C137152" (at 121.92 45.72 0)
+      (effects (font (size 1.27 1.27)) hide)
+    )
+    (property "Mounting" "Yes" (at 121.92 45.72 0)
       (effects (font (size 1.27 1.27)) hide)
     )
@@
       (effects (font (size 1.27 1.27)) hide)
     )
+    (property "Mounting" "Yes" (at 80.01 99.06 0)
+      (effects (font (size 1.27 1.27)) hide)
+    )
     (pin "1")
     (pin "2")
@@
     )
     (property "LCSC" "C277483" (at 110.49 57.15 0)
+      (effects (font (size 1.27 1.27)) hide)
+    )
+    (property "Mounting" "Yes" (at 110.49 57.15 0)
       (effects (font (size 1.27 1.27)) hide)
     )
@@
       (effects (font (size 1.27 1.27)) hide)
     )
+    (property "Mounting" "Yes" (at 100.33 129.54 0)
+      (effects (font (size 1.27 1.27)) hide)
+    )
     (pin "1")
     (pin "2")
@@
       (effects (font (size 1.27 1.27)) hide)
     )
+    (property "Mounting" "Yes" (at 100.33 106.68 0)
+      (effects (font (size 1.27 1.27)) hide)
+    )
     (pin "1")
     (pin "2")
@@
     )
     (property "LCSC" "C26041" (at 62.23 62.23 0)
+      (effects (font (size 1.27 1.27)) hide)
+    )
+    (property "Mounting" "Yes" (at 62.23 62.23 0)
       (effects (font (size 1.27 1.27)) hide)
     )
@@
       (effects (font (size 1.27 1.27)) hide)
     )
+    (property "Mounting" "Yes" (at 100.33 45.72 0)
+      (effects (font (size 1.27 1.27)) hide)
+    )
     (pin "1")
     (pin "2")
@@
       (effects (font (size 1.27 1.27)) hide)
     )
+    (property "Mounting" "Yes" (at 62.23 113.03 0)
+      (effects (font (size 1.27 1.27)) hide)
+    )
     (pin "1")
     (pin "2")
@@
       (effects (font (size 1.27 1.27)) hide)
     )
+    (property "Mounting" "Yes" (at 80.01 129.54 0)
+      (effects (font (size 1.27 1.27)) hide)
+    )
     (pin "1")
     (pin "2")
@@
       (effects (font (size 1.27 1.27)) hide)
     )
+    (property "Mounting" "Yes" (at 62.23 52.07 0)
+      (effects (font (size 1.27 1.27)) hide)
+    )
