File: Projects/StationModules/Module_1/Module_1.kicad_sch (KiCad schematic)
At the start: 60 parts, among them M1 BluePillStm32, U1 PC817, U2 L7805, U3 TC1047AxNB, U4 78L05S, U5 LM311, U6 6N137

Commit message: Corection all modules
Parts:
- added J7: -12V, TestPoint:TestPoint_THTPad_2.5x2.5mm_Drill1.2mm, symbol Connector:Conn_01x01_Pin
- added TP1, TP2, TP3: TestPoint, TestPoint:TestPoint_Pad_2.0x2.0mm, symbol Connector:TestPoint
- C17: value 1n -> 2,2n; LCSC C527247 -> C107194; MFR.Part CC1206GRNPO9BN102 -> CC1206KKX7RCBB222
Connections:
- net GND: now also J7.1 (Pin_1)
- net TMP: now also TP1.1
- net at U5.7, U6.3 (C): now also TP3.1
- net at R16.2, RV2.3, U5.2 (+): now also TP2.1
Changed lines of the file:
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@@
   (junction (at 101.6 120.65) (diameter 0) (color 0 0 0 0)
   )
+  (junction (at 210.82 50.8) (diameter 0) (color 0 0 0 0)
+  )
   (junction (at 170.18 62.23) (diameter 0) (color 0 0 0 0)
   )
@@
   (junction (at 106.68 181.61) (diameter 0) (color 0 0 0 0)
   )
+  (junction (at 247.65 53.34) (diameter 0) (color 0 0 0 0)
+  )
   (junction (at 31.75 158.75) (diameter 0) (color 0 0 0 0)
   )
@@
     (stroke (width 0) (type default))
   )
+  (wire (pts (xy 247.65 50.8) (xy 247.65 53.34))
+    (stroke (width 0) (type default))
+  )
   (wire (pts (xy 87.63 170.18) (xy 87.63 172.72))
     (stroke (width 0) (type default))
@@
     (stroke (width 0) (type default))
   )
+  (wire (pts (xy 20.32 168.91) (xy 31.75 168.91))
+    (stroke (width 0) (type default))
+  )
   (wire (pts (xy 120.65 143.51) (xy 120.65 147.32))
     (stroke (width 0) (type default))
@@
     (stroke (width 0) (type default))
   )
+  (wire (pts (xy 208.28 50.8) (xy 210.82 50.8))
+    (stroke (width 0) (type default))
+  )
   (wire (pts (xy 113.03 71.12) (xy 114.3 71.12))
     (stroke (width 0) (type default))
@@
     (stroke (width 0) (type default))
   )
+  (wire (pts (xy 123.19 102.87) (xy 123.19 111.76))
+    (stroke (width 0) (type default))
+  )
   (wire (pts (xy 123.19 113.03) (xy 123.19 111.76))
     (stroke (width 0) (type default))
@@
     (stroke (width 0) (type default))
   )
+  (wire (pts (xy 208.28 25.4) (xy 208.28 50.8))
+    (stroke (width 0) (type default))
+  )
   (wire (pts (xy 120.65 138.43) (xy 120.65 137.16))
     (stroke (width 0) (type default))
@@
     (stroke (width 0) (type default))
   )
+  (wire (pts (xy 246.38 50.8) (xy 247.65 50.8))
+    (stroke (width 0) (type default))
+  )
   (wire (pts (xy 34.29 90.17) (xy 40.64 90.17))
     (stroke (width 0) (type default))
@@
     (stroke (width 0) (type default))
   )
+  (wire (pts (xy 20.32 165.1) (xy 20.32 168.91))
+    (stroke (width 0) (type default))
+  )
   (wire (pts (xy 27.94 36.83) (xy 44.45 36.83))
     (stroke (width 0) (type default))
@@
     (stroke (width 0) (type default))
   )
+  (wire (pts (xy 246.38 25.4) (xy 246.38 50.8))
+    (stroke (width 0) (type default))
+  )
   (wire (pts (xy 52.07 137.16) (xy 59.69 137.16))
     (stroke (width 0) (type default))
@@
     )
   )
+  (symbol (lib_id "Connector:Conn_01x01_Pin") (at 20.32 160.02 270) (unit 1)
+    (in_bom yes) (on_board yes) (dnp no) (fields_autoplaced)
+    (property "Reference" "J7" (at 21.59 160.02 90)
+      (effects (font (size 1.27 1.27)) (justify left))
+    )
+    (property "Value" "-12V" (at 21.59 162.56 90)
+      (effects (font (size 1.27 1.27)) (justify left))
+    )
+    (property "Footprint" "TestPoint:TestPoint_THTPad_2.5x2.5mm_Drill1.2mm" (at 20.32 160.02 0)
+      (effects (font (size 1.27 1.27)) hide)
+    )
+    (property "Datasheet" "~" (at 20.32 160.02 0)
+      (effects (font (size 1.27 1.27)) hide)
+    )
+    (property "Description" "Plugin,P=2.54mm Pin Headers ROHS" (at 20.32 160.02 0)
+      (effects (font (size 1.27 1.27)) hide)
+    )
+    (property "LCSC" "C5156075" (at 20.32 160.02 0)
+      (effects (font (size 1.27 1.27)) hide)
+    )
+    (property "MFR.Part" "54101-T30-00LF" (at 20.32 160.02 0)
+      (effects (font (size 1.27 1.27)) hide)
+    )
+    (pin "1")
+    (instances
+      (project "Module_1"
+        (path "/52aeb9ce-9f3b-4d8f-8c36-7e23df4a5f32"
+          (reference "J7") (unit 1)
+        )
+      )
+    )
+  )
   (symbol (lib_id "power:GND") (at 87.63 156.21 0) (unit 1)
     (in_bom yes) (on_board yes) (dnp no) (fields_autoplaced)
@@
     )
   )
+  (symbol (lib_id "Connector:TestPoint") (at 123.19 102.87 0) (unit 1)
+    (in_bom yes) (on_board yes) (dnp no) (fields_autoplaced)
+    (property "Reference" "TP1" (at 125.73 98.933 0)
+      (effects (font (size 1.27 1.27)) (justify left))
+    )
+    (property "Value" "TestPoint" (at 125.73 101.473 0)
+      (effects (font (size 1.27 1.27)) (justify left))
+    )
+    (property "Footprint" "TestPoint:TestPoint_Pad_2.0x2.0mm" (at 128.27 102.87 0)
+      (effects (font (size 1.27 1.27)) hide)
+    )
+    (property "Datasheet" "~" (at 128.27 102.87 0)
+      (effects (font (size 1.27 1.27)) hide)
+    )
+    (pin "1")
+    (instances
+      (project "Module_1"
+        (path "/52aeb9ce-9f3b-4d8f-8c36-7e23df4a5f32"
+          (reference "TP1") (unit 1)
+        )
+      )
+    )
+  )
   (symbol (lib_id "Z_led:Led") (at 118.11 71.12 0) (unit 1)
     (in_bom yes) (on_board yes) (dnp no)
@@
   (symbol (lib_id "Device:R_Potentiometer") (at 210.82 45.72 0) (unit 1)
     (in_bom yes) (on_board yes) (dnp no)
-    (property "Reference" "RV2" (at 209.55 38.1 0)
+    (property "Reference" "RV2" (at 214.63 40.64 0)
       (effects (font (size 1.27 1.27)) (justify right))
     )
@@
     )
   )
+  (symbol (lib_id "Connector:TestPoint") (at 208.28 25.4 0) (unit 1)
+    (in_bom yes) (on_board yes) (dnp no) (fields_autoplaced)
+    (property "Reference" "TP2" (at 210.82 21.463 0)
+      (effects (font (size 1.27 1.27)) (justify left))
+    )
+    (property "Value" "TestPoint" (at 210.82 24.003 0)
+      (effects (font (size 1.27 1.27)) (justify left))
+    )
+    (property "Footprint" "TestPoint:TestPoint_Pad_2.0x2.0mm" (at 213.36 25.4 0)
+      (effects (font (size 1.27 1.27)) hide)
+    )
+    (property "Datasheet" "~" (at 213.36 25.4 0)
+      (effects (font (size 1.27 1.27)) hide)
+    )
+    (pin "1")
+    (instances
+      (project "Module_1"
+        (path "/52aeb9ce-9f3b-4d8f-8c36-7e23df4a5f32"
+          (reference "TP2") (unit 1)
+        )
+      )
+    )
+  )
+  (symbol (lib_id "Connector:TestPoint") (at 246.38 25.4 0) (unit 1)
+    (in_bom yes) (on_board yes) (dnp no) (fields_autoplaced)
+    (property "Reference" "TP3" (at 248.92 21.463 0)
+      (effects (font (size 1.27 1.27)) (justify left))
+    )
+    (property "Value" "TestPoint" (at 248.92 24.003 0)
+      (effects (font (size 1.27 1.27)) (justify left))
+    )
+    (property "Footprint" "TestPoint:TestPoint_Pad_2.0x2.0mm" (at 251.46 25.4 0)
+      (effects (font (size 1.27 1.27)) hide)
+    )
+    (property "Datasheet" "~" (at 251.46 25.4 0)
+      (effects (font (size 1.27 1.27)) hide)
+    )
+    (pin "1")
+    (instances
+      (project "Module_1"
+        (path "/52aeb9ce-9f3b-4d8f-8c36-7e23df4a5f32"
+          (reference "TP3") (unit 1)
+        )
+      )
+    )
+  )
   (symbol (lib_id "Diode:LL4148") (at 158.75 48.26 180) (unit 1)
     (in_bom yes) (on_board yes) (dnp no) (fields_autoplaced)
@@
   )
   (symbol (lib_id "Device:C_Small") (at 227.33 59.69 0) (unit 1)
-    (in_bom yes) (on_board yes) (dnp no) (fields_autoplaced)
-    (property "Reference" "C17" (at 229.87 59.0613 0)
+    (in_bom yes) (on_board yes) (dnp no)
+    (property "Reference" "C17" (at 229.87 60.96 0)
       (effects (font (size 1.27 1.27)) (justify left))
     )
-    (property "Value" "1n" (at 229.87 61.6013 0)
+    (property "Value" "2,2n" (at 229.87 63.5 0)
       (effects (font (size 1.27 1.27)) (justify left))
     )
@@
       (effects (font (size 1.27 1.27)) hide)
     )
-    (property "MFR.Part" "CC1206GRNPO9BN102" (at 227.33 59.69 0)
+    (property "MFR.Part" "CC1206KKX7RCBB222" (at 227.33 59.69 0)
       (effects (font (size 1.27 1.27)) hide)
     )
-    (property "Description" "50V 1nF NP0 ±2% 1206 Multilayer Ceramic Capacitors MLCC - SMD/SMT ROHS" (at 227.33 59.69 0)
+    (property "Description" "1kV 2.2nF X7R ±10% 1206 Multilayer Ceramic Capacitors MLCC - SMD/SMT ROHS" (at 227.33 59.69 0)
       (effects (font (size 1.27 1.27)) hide)
     )
-    (property "LCSC" "C527247" (at 227.33 59.69 0)
+    (property "LCSC" "C107194" (at 227.33 59.69 0)
       (effects (font (size 1.27 1.27)) hide)
     )
