File: Projects/StationModules/Module_1/PowerFet.kicad_sch (KiCad schematic)
At the start: 43 parts, among them J2 +310, J3 -310, J4 PowerTrans1, J5 PowerTrans2, Q5 IRGB10B60KD, Q6 IRGB10B60KD, Q7 IRGB10B60KD, Q8 IRGB10B60KD, T1 Transformer_SP_2S, T2 Transformer_SP_2S

Commit message: Place elements 1
Parts:
- C27: footprint Capacitor_THT:C_Rect_L41.5mm_W20.0mm_P37.50mm_MKS4 -> Capacitor_THT:C_Rect_L31.5mm_W15.0mm_P27.50mm_MKS4
- C28: footprint Capacitor_THT:C_Rect_L24.0mm_W10.1mm_P22.50mm_MKT -> Capacitor_THT:C_Rect_L26.5mm_W10.5mm_P22.50mm_MKS4
- Q5, Q6, Q7, Q8: footprint Package_TO_SOT_THT:TO-247-3_Vertical -> Z_Package_TO:TO-247-3_Horizontal_TabUp
- R37, R38, R39: footprint Resistor_THT:R_Axial_DIN0516_L15.5mm_D5.0mm_P20.32mm_Horizontal -> Resistor_THT:R_Axial_DIN0411_L9.9mm_D3.6mm_P15.24mm_Horizontal
Connections:
- net Shunt+: now also D17.2 (A2), D19.2 (A2); no longer D17.1 (A1), D19.1 (A1)
- net at C26.1, D22.1 (A1), J5.1 (Pin_1)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: now also D18.2 (A2); no longer D18.1 (A1)
- net at D1.2 (A), Q8.1 (G), R12.1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: now also D19.1 (A1); no longer D19.2 (A2)
- net at D1.2 (A), Q5.1 (G), R12.1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: now also D16.1 (A1); no longer D16.2 (A2)
- net at D1.2 (A), Q7.1 (G), R12.1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: now also D18.1 (A1); no longer D18.2 (A2)
- net at C24.1, C27.1, D20.1 (A1)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: now also D16.2 (A2); no longer D16.1 (A1)
- net at D1.2 (A), Q6.1 (G), R12.1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: now also D17.1 (A1); no longer D17.2 (A2)
Other:
- moved on the sheet: D16, D17, D18, D19
Changed lines of the file:
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@@
       (effects (font (size 1.27 1.27)) (justify left))
     )
-    (property "Footprint" "Package_TO_SOT_THT:TO-247-3_Vertical" (at 128.27 90.17 0)
+    (property "Footprint" "Z_Package_TO:TO-247-3_Horizontal_TabUp" (at 128.27 90.17 0)
       (effects (font (size 1.27 1.27) italic) hide)
     )
@@
       (effects (font (size 1.27 1.27)) (justify left))
     )
-    (property "Footprint" "Capacitor_THT:C_Rect_L24.0mm_W10.1mm_P22.50mm_MKT" (at 207.01 57.15 0)
+    (property "Footprint" "Capacitor_THT:C_Rect_L26.5mm_W10.5mm_P22.50mm_MKS4" (at 207.01 57.15 0)
       (effects (font (size 1.27 1.27)) hide)
     )
@@
       (effects (font (size 1.27 1.27)) (justify left))
     )
-    (property "Footprint" "Resistor_THT:R_Axial_DIN0516_L15.5mm_D5.0mm_P20.32mm_Horizontal" (at 122.682 111.76 90)
+    (property "Footprint" "Resistor_THT:R_Axial_DIN0411_L9.9mm_D3.6mm_P15.24mm_Horizontal" (at 122.682 111.76 90)
       (effects (font (size 1.27 1.27)) hide)
     )
@@
     )
   )
-  (symbol (lib_id "Diode:1.5KExxCA") (at 96.52 95.25 90) (unit 1)
+  (symbol (lib_id "Diode:1.5KExxCA") (at 96.52 95.25 270) (unit 1)
     (in_bom yes) (on_board yes) (dnp no) (fields_autoplaced)
     (property "Reference" "D19" (at 99.06 94.615 90)
-      (effects (font (size 1.27 1.27)) (justify right))
+      (effects (font (size 1.27 1.27)) (justify left))
     )
     (property "Value" "P6KE18CA" (at 99.06 97.155 90)
-      (effects (font (size 1.27 1.27)) (justify right))
-    )
-    (property "Footprint" "Diode_THT:D_DO-201AE_P15.24mm_Horizontal" (at 101.6 95.25 0)
+      (effects (font (size 1.27 1.27)) (justify left))
+    )
+    (property "Footprint" "Diode_THT:D_DO-201AE_P15.24mm_Horizontal" (at 91.44 95.25 0)
       (effects (font (size 1.27 1.27)) hide)
     )
@@
     )
   )
-  (symbol (lib_id "Diode:1.5KExxCA") (at 96.52 80.01 90) (unit 1)
+  (symbol (lib_id "Diode:1.5KExxCA") (at 96.52 80.01 270) (unit 1)
     (in_bom yes) (on_board yes) (dnp no) (fields_autoplaced)
     (property "Reference" "D18" (at 99.06 79.375 90)
-      (effects (font (size 1.27 1.27)) (justify right))
+      (effects (font (size 1.27 1.27)) (justify left))
     )
     (property "Value" "P6KE18CA" (at 99.06 81.915 90)
-      (effects (font (size 1.27 1.27)) (justify right))
-    )
-    (property "Footprint" "Diode_THT:D_DO-201AE_P15.24mm_Horizontal" (at 101.6 80.01 0)
+      (effects (font (size 1.27 1.27)) (justify left))
+    )
+    (property "Footprint" "Diode_THT:D_DO-201AE_P15.24mm_Horizontal" (at 91.44 80.01 0)
       (effects (font (size 1.27 1.27)) hide)
     )
@@
       (effects (font (size 1.27 1.27)) (justify left))
     )
-    (property "Footprint" "Resistor_THT:R_Axial_DIN0516_L15.5mm_D5.0mm_P20.32mm_Horizontal" (at 129.032 111.76 90)
+    (property "Footprint" "Resistor_THT:R_Axial_DIN0411_L9.9mm_D3.6mm_P15.24mm_Horizontal" (at 129.032 111.76 90)
       (effects (font (size 1.27 1.27)) hide)
     )
@@
     )
   )
-  (symbol (lib_id "Diode:1.5KExxCA") (at 96.52 41.91 90) (unit 1)
+  (symbol (lib_id "Diode:1.5KExxCA") (at 96.52 41.91 270) (unit 1)
     (in_bom yes) (on_board yes) (dnp no) (fields_autoplaced)
     (property "Reference" "D16" (at 99.06 41.275 90)
-      (effects (font (size 1.27 1.27)) (justify right))
+      (effects (font (size 1.27 1.27)) (justify left))
     )
     (property "Value" "P6KE18CA" (at 99.06 43.815 90)
-      (effects (font (size 1.27 1.27)) (justify right))
-    )
-    (property "Footprint" "Diode_THT:D_DO-201AE_P15.24mm_Horizontal" (at 101.6 41.91 0)
+      (effects (font (size 1.27 1.27)) (justify left))
+    )
+    (property "Footprint" "Diode_THT:D_DO-201AE_P15.24mm_Horizontal" (at 91.44 41.91 0)
       (effects (font (size 1.27 1.27)) hide)
     )
@@
       (effects (font (size 1.27 1.27)) (justify left))
     )
-    (property "Footprint" "Package_TO_SOT_THT:TO-247-3_Vertical" (at 128.27 54.61 0)
+    (property "Footprint" "Z_Package_TO:TO-247-3_Horizontal_TabUp" (at 128.27 54.61 0)
       (effects (font (size 1.27 1.27) italic) hide)
     )
@@
       (effects (font (size 1.27 1.27)) (justify left))
     )
-    (property "Footprint" "Resistor_THT:R_Axial_DIN0516_L15.5mm_D5.0mm_P20.32mm_Horizontal" (at 135.382 111.76 90)
+    (property "Footprint" "Resistor_THT:R_Axial_DIN0411_L9.9mm_D3.6mm_P15.24mm_Horizontal" (at 135.382 111.76 90)
       (effects (font (size 1.27 1.27)) hide)
     )
@@
       (effects (font (size 1.27 1.27)) (justify left))
     )
-    (property "Footprint" "Package_TO_SOT_THT:TO-247-3_Vertical" (at 128.27 36.83 0)
+    (property "Footprint" "Z_Package_TO:TO-247-3_Horizontal_TabUp" (at 128.27 36.83 0)
       (effects (font (size 1.27 1.27) italic) hide)
     )
@@
       (effects (font (size 1.27 1.27)))
     )
-    (property "Footprint" "Capacitor_THT:C_Rect_L41.5mm_W20.0mm_P37.50mm_MKS4" (at 163.83 49.53 0)
+    (property "Footprint" "Capacitor_THT:C_Rect_L31.5mm_W15.0mm_P27.50mm_MKS4" (at 163.83 49.53 0)
       (effects (font (size 1.27 1.27)) hide)
     )
@@
       (effects (font (size 1.27 1.27)) (justify left))
     )
-    (property "Footprint" "Package_TO_SOT_THT:TO-247-3_Vertical" (at 128.27 76.2 0)
+    (property "Footprint" "Z_Package_TO:TO-247-3_Horizontal_TabUp" (at 128.27 76.2 0)
       (effects (font (size 1.27 1.27) italic) hide)
     )
@@
     )
   )
-  (symbol (lib_id "Diode:1.5KExxCA") (at 96.52 59.69 90) (unit 1)
+  (symbol (lib_id "Diode:1.5KExxCA") (at 96.52 59.69 270) (unit 1)
     (in_bom yes) (on_board yes) (dnp no) (fields_autoplaced)
     (property "Reference" "D17" (at 99.06 59.055 90)
-      (effects (font (size 1.27 1.27)) (justify right))
+      (effects (font (size 1.27 1.27)) (justify left))
     )
     (property "Value" "P6KE18CA" (at 99.06 61.595 90)
-      (effects (font (size 1.27 1.27)) (justify right))
-    )
-    (property "Footprint" "Diode_THT:D_DO-201AE_P15.24mm_Horizontal" (at 101.6 59.69 0)
-      (effects (font (size 1.27 1.27)) hide)
-    )
+      (effects (font (size 1.27 1.27)) (justify left))
+    )
+    (property "Footprint" "Diode_THT:D_DO-201AE_P15.24mm_Horizontal" (at 91.44 59.69 0)
+      (effects (font (size 1.27 1.27)) hide)
+    )

Commit message: add bom module 1
Parts:
- added D24, D25, D26, D27: SMBJ18CA, Diode_SMD:D_SMB, symbol Device:D_TVS
- added D28, D29, D30, D31: ES3JC, Diode_SMD:D_SMC, symbol Device:D
- added R44, R45, R46: 0,01, Resistor_SMD:R_2816_7142Metric, symbol Device:R
- C23, C24, C25, C26: LCSC (none) -> C424416; MFR.Part (none) -> CL112J222J0501
- C27: LCSC (none) -> C330414; MFR.Part (none) -> C3D1U205KB00C00
- C28: value 0,1u 600V -> 0,47u 600V; LCSC (none) -> C2928856; MFR.Part (none) -> MPB474J2V2701
- D1: LCSC (none) -> C2891733; MFR.Part (none) -> LL4148
- D16, D17, D18, D19: LCSC (none) -> C600792; MFR.Part (none) -> P6KE18CA
- D20, D21, D22, D23: LCSC (none) -> C424502; MFR.Part (none) -> UF5408
- Q5, Q6, Q7, Q8: value IRGB10B60KD -> STW20NM60; LCSC (none) -> C262986; MFR.Part (none) -> STW20NM60
- R12: LCSC (none) -> C137178; MFR.Part (none) -> RC1206JR-0720RL
- R12: LCSC (none) -> C137167; MFR.Part (none) -> RC1206JR-072K2L
- R37, R38, R39: value 0,1 -> 0,01
- R40, R41, R42, R43: LCSC (none) -> C2903435; MFR.Part (none) -> CR2W-18Ω±5%-9T73
Connections:
- net Shunt+: now also D24.2 (A2), D26.2 (A2), D29.1 (K), D31.1 (K), R44.1, R45.1, R46.1
- net Shunt-: now also R44.2, R45.2, R46.2
- net at C26.1, D18.2 (A2), D22.1 (A1)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: now also D25.2 (A2), D30.1 (K)
- net at D1.2 (A), D19.1 (A1), Q8.1 (G)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: now also D24.1 (A1)
- net at C24.2, D21.2 (A2), R41.1: now also D29.2 (A)
- net at C25.2, D22.2 (A2), R42.1: now also D30.2 (A)
- net at D1.2 (A), D16.1 (A1), Q5.1 (G)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: now also D27.1 (A1)
- net at D1.2 (A), D18.1 (A1), Q7.1 (G)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: now also D25.1 (A1)
- net at C23.2, D20.2 (A2), R40.1: now also D28.2 (A)
- net at C26.2, D23.2 (A2), R43.1: now also D31.2 (A)
- net at C24.1, C27.1, D16.2 (A2)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: now also D27.2 (A2), D28.1 (K)
- net at D1.2 (A), D17.1 (A1), Q6.1 (G)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: now also D26.1 (A1)
Other:
- note added: "SMD"

Commit message: add bom and pos
Parts:
- R40, R41, R42, R43: value 18 2W -> 18
Changed lines of the file:
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@@
       (effects (font (size 1.27 1.27)) (justify left))
     )
-    (property "Value" "18 2W" (at 130.81 82.55 0)
+    (property "Value" "18" (at 130.81 82.55 0)
       (effects (font (size 1.27 1.27)) (justify left))
     )
@@
       (effects (font (size 1.27 1.27)) (justify left))
     )
-    (property "Value" "18 2W" (at 130.81 97.79 0)
+    (property "Value" "18" (at 130.81 97.79 0)
       (effects (font (size 1.27 1.27)) (justify left))
     )
@@
       (effects (font (size 1.27 1.27)) (justify left))
     )
-    (property "Value" "18 2W" (at 130.81 45.72 0)
+    (property "Value" "18" (at 130.81 45.72 0)
       (effects (font (size 1.27 1.27)) (justify left))
     )
@@
       (effects (font (size 1.27 1.27)) (justify left))
     )
-    (property "Value" "18 2W" (at 130.81 62.23 0)
-      (effects (font (size 1.27 1.27)) (justify left))
-    )
+    (property "Value" "18" (at 130.81 62.23 0)
+      (effects (font (size 1.27 1.27)) (justify left))
+    )

Commit message: finaly on summer
Parts:
- C23, C24, C25, C26: LCSC C424416 -> C2991065
- R12: value 20 -> 100; LCSC C137178 -> C113307; MFR.Part RC1206JR-0720RL -> RC1206JR-07100RL
- R40, R41, R42, R43: LCSC C2903435 -> C119690
Changed lines of the file:
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@@
       (effects (font (size 1.27 1.27)) hide)
     )
-    (property "LCSC" "C2903435" (at 138.43 81.28 0)
+    (property "LCSC" "C119690" (at 138.43 81.28 0)
       (effects (font (size 1.27 1.27)) hide)
     )
@@
       (effects (font (size 1.27 1.27)))
     )
-    (property "Value" "20" (at 73.66 86.36 90)
+    (property "Value" "100" (at 73.66 86.36 90)
       (effects (font (size 1.27 1.27)))
     )
@@
       (effects (font (size 1.27 1.27)) hide)
     )
-    (property "MFR.Part" "RC1206JR-0720RL" (at 73.66 88.9 0)
-      (effects (font (size 1.27 1.27)) hide)
-    )
-    (property "Description" "250mW Thick Film Resistors ±100ppm/℃ ±5% 20Ω 1206 Chip Resistor - Surface Mount ROHS" (at 73.66 88.9 0)
-      (effects (font (size 1.27 1.27)) hide)
-    )
-    (property "LCSC" "C137178" (at 73.66 88.9 0)
+    (property "MFR.Part" "RC1206JR-07100RL" (at 73.66 88.9 0)
+      (effects (font (size 1.27 1.27)) hide)
+    )
+    (property "Description" "250mW Thick Film Resistors ±100ppm/℃ ±5% 100Ω 1206 Chip Resistor - Surface Mount ROHS" (at 73.66 88.9 0)
+      (effects (font (size 1.27 1.27)) hide)
+    )
+    (property "LCSC" "C113307" (at 73.66 88.9 0)
       (effects (font (size 1.27 1.27)) hide)
     )
@@
       (effects (font (size 1.27 1.27)) hide)
     )
-    (property "LCSC" "C424416" (at 138.43 34.29 0)
+    (property "LCSC" "C2991065" (at 138.43 34.29 0)
       (effects (font (size 1.27 1.27)) hide)
     )
@@
       (effects (font (size 1.27 1.27)) hide)
     )
-    (property "LCSC" "C424416" (at 138.43 87.63 0)
+    (property "LCSC" "C2991065" (at 138.43 87.63 0)
       (effects (font (size 1.27 1.27)) hide)
     )
@@
       (effects (font (size 1.27 1.27)) hide)
     )
-    (property "LCSC" "C424416" (at 138.43 73.66 0)
+    (property "LCSC" "C2991065" (at 138.43 73.66 0)
       (effects (font (size 1.27 1.27)) hide)
     )
@@
       (effects (font (size 1.27 1.27)) hide)
     )
-    (property "LCSC" "C2903435" (at 138.43 96.52 0)
+    (property "LCSC" "C119690" (at 138.43 96.52 0)
       (effects (font (size 1.27 1.27)) hide)
     )
@@
       (effects (font (size 1.27 1.27)) hide)
     )
-    (property "LCSC" "C2903435" (at 138.43 45.72 0)
+    (property "LCSC" "C119690" (at 138.43 45.72 0)
       (effects (font (size 1.27 1.27)) hide)
     )
@@
       (effects (font (size 1.27 1.27)))
     )
-    (property "Value" "20" (at 76.2 59.69 90)
+    (property "Value" "100" (at 76.2 59.69 90)
       (effects (font (size 1.27 1.27)))
     )
@@
       (effects (font (size 1.27 1.27)) hide)
     )
-    (property "MFR.Part" "RC1206JR-0720RL" (at 74.93 57.15 0)
-      (effects (font (size 1.27 1.27)) hide)
-    )
-    (property "Description" "250mW Thick Film Resistors ±100ppm/℃ ±5% 20Ω 1206 Chip Resistor - Surface Mount ROHS" (at 74.93 57.15 0)
-      (effects (font (size 1.27 1.27)) hide)
-    )
-    (property "LCSC" "C137178" (at 74.93 57.15 0)
+    (property "MFR.Part" "RC1206JR-07100RL" (at 74.93 57.15 0)
+      (effects (font (size 1.27 1.27)) hide)
+    )
+    (property "Description" "250mW Thick Film Resistors ±100ppm/℃ ±5% 100Ω 1206 Chip Resistor - Surface Mount ROHS" (at 74.93 57.15 0)
+      (effects (font (size 1.27 1.27)) hide)
+    )
+    (property "LCSC" "C113307" (at 74.93 57.15 0)
       (effects (font (size 1.27 1.27)) hide)
     )
@@
       (effects (font (size 1.27 1.27)))
     )
-    (property "Value" "20" (at 76.2 41.91 90)
+    (property "Value" "100" (at 76.2 41.91 90)
       (effects (font (size 1.27 1.27)))
     )
@@
       (effects (font (size 1.27 1.27)) hide)
     )
-    (property "MFR.Part" "RC1206JR-0720RL" (at 74.93 39.37 0)
-      (effects (font (size 1.27 1.27)) hide)
-    )
-    (property "Description" "250mW Thick Film Resistors ±100ppm/℃ ±5% 20Ω 1206 Chip Resistor - Surface Mount ROHS" (at 74.93 39.37 0)
-      (effects (font (size 1.27 1.27)) hide)
-    )
-    (property "LCSC" "C137178" (at 74.93 39.37 0)
+    (property "MFR.Part" "RC1206JR-07100RL" (at 74.93 39.37 0)
+      (effects (font (size 1.27 1.27)) hide)
+    )
+    (property "Description" "250mW Thick Film Resistors ±100ppm/℃ ±5% 100Ω 1206 Chip Resistor - Surface Mount ROHS" (at 74.93 39.37 0)
+      (effects (font (size 1.27 1.27)) hide)
+    )
+    (property "LCSC" "C113307" (at 74.93 39.37 0)
       (effects (font (size 1.27 1.27)) hide)
     )
@@
       (effects (font (size 1.27 1.27)) hide)
     )
-    (property "LCSC" "C424416" (at 138.43 52.07 0)
+    (property "LCSC" "C2991065" (at 138.43 52.07 0)
       (effects (font (size 1.27 1.27)) hide)
     )
@@
       (effects (font (size 1.27 1.27)) hide)
     )
-    (property "LCSC" "C2903435" (at 138.43 60.96 0)
+    (property "LCSC" "C119690" (at 138.43 60.96 0)
       (effects (font (size 1.27 1.27)) hide)
     )
@@
       (effects (font (size 1.27 1.27)))
     )
-    (property "Value" "20" (at 73.66 72.39 90)
+    (property "Value" "100" (at 73.66 72.39 90)
       (effects (font (size 1.27 1.27)))
     )
@@
       (effects (font (size 1.27 1.27)) hide)
     )
-    (property "MFR.Part" "RC1206JR-0720RL" (at 73.66 74.93 0)
-      (effects (font (size 1.27 1.27)) hide)
-    )
-    (property "Description" "250mW Thick Film Resistors ±100ppm/℃ ±5% 20Ω 1206 Chip Resistor - Surface Mount ROHS" (at 73.66 74.93 0)
-      (effects (font (size 1.27 1.27)) hide)
-    )
-    (property "LCSC" "C137178" (at 73.66 74.93 0)
-      (effects (font (size 1.27 1.27)) hide)
-    )
+    (property "MFR.Part" "RC1206JR-07100RL" (at 73.66 74.93 0)
+      (effects (font (size 1.27 1.27)) hide)
+    )
+    (property "Description" "250mW Thick Film Resistors ±100ppm/℃ ±5% 100Ω 1206 Chip Resistor - Surface Mount ROHS" (at 73.66 74.93 0)
+      (effects (font (size 1.27 1.27)) hide)
+    )
+    (property "LCSC" "C113307" (at 73.66 74.93 0)
+      (effects (font (size 1.27 1.27)) hide)
+    )
