File: Projects/StationModules/Module_1/PowerFet.kicad_sch (KiCad schematic)
At the start: 54 parts, among them J2 +310, J3 -310, J4 PowerTrans1, J5 PowerTrans2, Q5 STW20NM60, Q6 STW20NM60, Q7 STW20NM60, Q8 STW20NM60, T1 Transformer_SP_2S, T2 Transformer_SP_2S

Commit message: change module1,2
Parts:
- C23, C24, C25, C26: value 2n2 600v -> 1n 630v; LCSC C2991065 -> C2764154; MFR.Part CL112J222J0501 -> 2J102J114CL010
- J4, J5: footprint Z_pin:PinD4mm -> Z_pin:PinD3mm
- R12: value 100 -> 75; LCSC C113307 -> C17987; MFR.Part RC1206JR-07100RL -> 1206W4F750JT5E
Changed lines of the file:
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@@
       (effects (font (size 1.27 1.27)))
     )
-    (property "Value" "100" (at 73.66 86.36 90)
+    (property "Value" "75" (at 73.66 86.36 90)
       (effects (font (size 1.27 1.27)))
     )
@@
       (effects (font (size 1.27 1.27)) hide)
     )
-    (property "MFR.Part" "RC1206JR-07100RL" (at 73.66 88.9 0)
-      (effects (font (size 1.27 1.27)) hide)
-    )
-    (property "Description" "250mW Thick Film Resistors ±100ppm/℃ ±5% 100Ω 1206 Chip Resistor - Surface Mount ROHS" (at 73.66 88.9 0)
-      (effects (font (size 1.27 1.27)) hide)
-    )
-    (property "LCSC" "C113307" (at 73.66 88.9 0)
+    (property "MFR.Part" "1206W4F750JT5E" (at 73.66 88.9 0)
+      (effects (font (size 1.27 1.27)) hide)
+    )
+    (property "Description" "250mW Thick Film Resistors ±100ppm/℃ ±1% 75Ω 1206 Chip Resistor - Surface Mount ROHS" (at 73.66 88.9 0)
+      (effects (font (size 1.27 1.27)) hide)
+    )
+    (property "LCSC" "C17987" (at 73.66 88.9 0)
       (effects (font (size 1.27 1.27)) hide)
     )
@@
       (effects (font (size 1.27 1.27)))
     )
-    (property "Footprint" "Z_pin:PinD4mm" (at 182.88 58.42 0)
+    (property "Footprint" "Z_pin:PinD3mm" (at 182.88 58.42 0)
       (effects (font (size 1.27 1.27)) hide)
     )
@@
       (effects (font (size 1.27 1.27)) (justify left))
     )
-    (property "Value" "2n2 600v" (at 140.97 36.2013 0)
+    (property "Value" "1n 630v" (at 140.97 36.2013 0)
       (effects (font (size 1.27 1.27)) (justify left))
     )
@@
       (effects (font (size 1.27 1.27)) hide)
     )
-    (property "MFR.Part" "CL112J222J0501" (at 138.43 34.29 0)
-      (effects (font (size 1.27 1.27)) hide)
-    )
-    (property "Description" "±5% 630V 2.2nF PET Plugin,P=5mm Film Capacitors ROHS" (at 138.43 34.29 0)
-      (effects (font (size 1.27 1.27)) hide)
-    )
-    (property "LCSC" "C2991065" (at 138.43 34.29 0)
+    (property "MFR.Part" "2J102J114CL010" (at 138.43 34.29 0)
+      (effects (font (size 1.27 1.27)) hide)
+    )
+    (property "Description" "±5% 630V 1nF PET Plugin,P=5mm Film Capacitors ROHS" (at 138.43 34.29 0)
+      (effects (font (size 1.27 1.27)) hide)
+    )
+    (property "LCSC" "C2764154" (at 138.43 34.29 0)
       (effects (font (size 1.27 1.27)) hide)
     )
@@
       (effects (font (size 1.27 1.27)) (justify left))
     )
-    (property "Value" "2n2 600v" (at 140.97 89.5413 0)
+    (property "Value" "1n 630v" (at 140.97 89.5413 0)
       (effects (font (size 1.27 1.27)) (justify left))
     )
@@
       (effects (font (size 1.27 1.27)) hide)
     )
-    (property "MFR.Part" "CL112J222J0501" (at 138.43 87.63 0)
-      (effects (font (size 1.27 1.27)) hide)
-    )
-    (property "Description" "±5% 630V 2.2nF PET Plugin,P=5mm Film Capacitors ROHS" (at 138.43 87.63 0)
-      (effects (font (size 1.27 1.27)) hide)
-    )
-    (property "LCSC" "C2991065" (at 138.43 87.63 0)
+    (property "MFR.Part" "2J102J114CL010" (at 138.43 87.63 0)
+      (effects (font (size 1.27 1.27)) hide)
+    )
+    (property "Description" "±5% 630V 1nF PET Plugin,P=5mm Film Capacitors ROHS" (at 138.43 87.63 0)
+      (effects (font (size 1.27 1.27)) hide)
+    )
+    (property "LCSC" "C2764154" (at 138.43 87.63 0)
       (effects (font (size 1.27 1.27)) hide)
     )
@@
       (effects (font (size 1.27 1.27)) (justify left))
     )
-    (property "Value" "2n2 600v" (at 140.97 75.5713 0)
+    (property "Value" "1n 630v" (at 140.97 75.5713 0)
       (effects (font (size 1.27 1.27)) (justify left))
     )
@@
       (effects (font (size 1.27 1.27)) hide)
     )
-    (property "MFR.Part" "CL112J222J0501" (at 138.43 73.66 0)
-      (effects (font (size 1.27 1.27)) hide)
-    )
-    (property "Description" "±5% 630V 2.2nF PET Plugin,P=5mm Film Capacitors ROHS" (at 138.43 73.66 0)
-      (effects (font (size 1.27 1.27)) hide)
-    )
-    (property "LCSC" "C2991065" (at 138.43 73.66 0)
+    (property "MFR.Part" "2J102J114CL010" (at 138.43 73.66 0)
+      (effects (font (size 1.27 1.27)) hide)
+    )
+    (property "Description" "±5% 630V 1nF PET Plugin,P=5mm Film Capacitors ROHS" (at 138.43 73.66 0)
+      (effects (font (size 1.27 1.27)) hide)
+    )
+    (property "LCSC" "C2764154" (at 138.43 73.66 0)
       (effects (font (size 1.27 1.27)) hide)
     )
@@
       (effects (font (size 1.27 1.27)))
     )
-    (property "Value" "100" (at 76.2 59.69 90)
+    (property "Value" "75" (at 76.2 59.69 90)
       (effects (font (size 1.27 1.27)))
     )
@@
       (effects (font (size 1.27 1.27)) hide)
     )
-    (property "MFR.Part" "RC1206JR-07100RL" (at 74.93 57.15 0)
-      (effects (font (size 1.27 1.27)) hide)
-    )
-    (property "Description" "250mW Thick Film Resistors ±100ppm/℃ ±5% 100Ω 1206 Chip Resistor - Surface Mount ROHS" (at 74.93 57.15 0)
-      (effects (font (size 1.27 1.27)) hide)
-    )
-    (property "LCSC" "C113307" (at 74.93 57.15 0)
+    (property "MFR.Part" "1206W4F750JT5E" (at 74.93 57.15 0)
+      (effects (font (size 1.27 1.27)) hide)
+    )
+    (property "Description" "250mW Thick Film Resistors ±100ppm/℃ ±1% 75Ω 1206 Chip Resistor - Surface Mount ROHS" (at 74.93 57.15 0)
+      (effects (font (size 1.27 1.27)) hide)
+    )
+    (property "LCSC" "C17987" (at 74.93 57.15 0)
       (effects (font (size 1.27 1.27)) hide)
     )
@@
       (effects (font (size 1.27 1.27)))
     )
-    (property "Value" "100" (at 76.2 41.91 90)
+    (property "Value" "75" (at 76.2 41.91 90)
       (effects (font (size 1.27 1.27)))
     )
@@
       (effects (font (size 1.27 1.27)) hide)
     )
-    (property "MFR.Part" "RC1206JR-07100RL" (at 74.93 39.37 0)
-      (effects (font (size 1.27 1.27)) hide)
-    )
-    (property "Description" "250mW Thick Film Resistors ±100ppm/℃ ±5% 100Ω 1206 Chip Resistor - Surface Mount ROHS" (at 74.93 39.37 0)
-      (effects (font (size 1.27 1.27)) hide)
-    )
-    (property "LCSC" "C113307" (at 74.93 39.37 0)
+    (property "MFR.Part" "1206W4F750JT5E" (at 74.93 39.37 0)
+      (effects (font (size 1.27 1.27)) hide)
+    )
+    (property "Description" "250mW Thick Film Resistors ±100ppm/℃ ±1% 75Ω 1206 Chip Resistor - Surface Mount ROHS" (at 74.93 39.37 0)
+      (effects (font (size 1.27 1.27)) hide)
+    )
+    (property "LCSC" "C17987" (at 74.93 39.37 0)
       (effects (font (size 1.27 1.27)) hide)
     )
@@
       (effects (font (size 1.27 1.27)) (justify left))
     )
-    (property "Value" "2n2 600v" (at 140.97 53.9813 0)
+    (property "Value" "1n 630v" (at 140.97 53.9813 0)
       (effects (font (size 1.27 1.27)) (justify left))
     )
@@
       (effects (font (size 1.27 1.27)) hide)
     )
-    (property "MFR.Part" "CL112J222J0501" (at 138.43 52.07 0)
-      (effects (font (size 1.27 1.27)) hide)
-    )
-    (property "Description" "±5% 630V 2.2nF PET Plugin,P=5mm Film Capacitors ROHS" (at 138.43 52.07 0)
-      (effects (font (size 1.27 1.27)) hide)
-    )
-    (property "LCSC" "C2991065" (at 138.43 52.07 0)
+    (property "MFR.Part" "2J102J114CL010" (at 138.43 52.07 0)
+      (effects (font (size 1.27 1.27)) hide)
+    )
+    (property "Description" "±5% 630V 1nF PET Plugin,P=5mm Film Capacitors ROHS" (at 138.43 52.07 0)
+      (effects (font (size 1.27 1.27)) hide)
+    )
+    (property "LCSC" "C2764154" (at 138.43 52.07 0)
       (effects (font (size 1.27 1.27)) hide)
     )
@@
       (effects (font (size 1.27 1.27)))
     )
-    (property "Footprint" "Z_pin:PinD4mm" (at 182.88 49.53 0)
+    (property "Footprint" "Z_pin:PinD3mm" (at 182.88 49.53 0)
       (effects (font (size 1.27 1.27)) hide)
     )
@@
       (effects (font (size 1.27 1.27)))
     )
-    (property "Value" "100" (at 73.66 72.39 90)
+    (property "Value" "75" (at 73.66 72.39 90)
       (effects (font (size 1.27 1.27)))
     )
@@
       (effects (font (size 1.27 1.27)) hide)
     )
-    (property "MFR.Part" "RC1206JR-07100RL" (at 73.66 74.93 0)
-      (effects (font (size 1.27 1.27)) hide)
-    )
-    (property "Description" "250mW Thick Film Resistors ±100ppm/℃ ±5% 100Ω 1206 Chip Resistor - Surface Mount ROHS" (at 73.66 74.93 0)
-      (effects (font (size 1.27 1.27)) hide)
-    )
-    (property "LCSC" "C113307" (at 73.66 74.93 0)
-      (effects (font (size 1.27 1.27)) hide)
-    )
+    (property "MFR.Part" "1206W4F750JT5E" (at 73.66 74.93 0)
+      (effects (font (size 1.27 1.27)) hide)
+    )
+    (property "Description" "250mW Thick Film Resistors ±100ppm/℃ ±1% 75Ω 1206 Chip Resistor - Surface Mount ROHS" (at 73.66 74.93 0)
+      (effects (font (size 1.27 1.27)) hide)
+    )
+    (property "LCSC" "C17987" (at 73.66 74.93 0)
+      (effects (font (size 1.27 1.27)) hide)
+    )

Commit message: change on 25_02_24
Parts:
- C23, C24, C25, C26: LCSC C2764154 -> C914547; MFR.Part 2J102J114CL010 -> CL11-2J102J-630V; Mounting (none) -> Yes
- C27, D1, D24, D25, D26, D27, D28, D29, D30, D31, R12, R40, R41, R42, R43, R44, R45, R46: Mounting (none) -> Yes
- C28: LCSC C2928856 -> C2803198; MFR.Part MPB474J2V2701 -> C2803198; Mounting (none) -> Yes
- D16, D17, D18, D19, D20, D21, D22, D23, J2, J3, J4, J5, Q5, Q6, Q7, Q8, R37, R38, R39, T1, T2: Mounting (none) -> No

Commit message: Corection all modules
Parts:
- added J6: -310V, TestPoint:TestPoint_THTPad_2.5x2.5mm_Drill1.2mm, symbol Connector:Conn_01x01_Pin
Connections:
- net Shunt-: now also J6.1 (Pin_1)
Changed lines of the file:
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@@
   (junction (at 138.43 77.47) (diameter 0) (color 0 0 0 0)
   )
+  (junction (at 185.42 118.11) (diameter 0) (color 0 0 0 0)
+  )
   (junction (at 138.43 64.77) (diameter 0) (color 0 0 0 0)
   )
@@
     (stroke (width 0) (type default))
   )
-  (wire (pts (xy 160.02 118.11) (xy 207.01 118.11))
+  (wire (pts (xy 160.02 118.11) (xy 185.42 118.11))
     (stroke (width 0) (type default))
   )
@@
     (stroke (width 0) (type default))
   )
+  (wire (pts (xy 185.42 115.57) (xy 185.42 118.11))
+    (stroke (width 0) (type default))
+  )
   (wire (pts (xy 144.78 105.41) (xy 152.4 105.41))
     (stroke (width 0) (type default))
@@
   )
   (wire (pts (xy 137.16 105.41) (xy 137.16 107.95))
+    (stroke (width 0) (type default))
+  )
+  (wire (pts (xy 185.42 118.11) (xy 207.01 118.11))
     (stroke (width 0) (type default))
   )
@@
         )
       )
+    )
+  )
+  (symbol (lib_id "Connector:Conn_01x01_Pin") (at 185.42 110.49 270) (unit 1)
+    (in_bom yes) (on_board yes) (dnp no) (fields_autoplaced)
+    (property "Reference" "J6" (at 186.69 110.49 90)
+      (effects (font (size 1.27 1.27)) (justify left))
+    )
+    (property "Value" "-310V" (at 186.69 113.03 90)
+      (effects (font (size 1.27 1.27)) (justify left))
+    )
+    (property "Footprint" "TestPoint:TestPoint_THTPad_2.5x2.5mm_Drill1.2mm" (at 185.42 110.49 0)
+      (effects (font (size 1.27 1.27)) hide)
+    )
+    (property "Datasheet" "~" (at 185.42 110.49 0)
+      (effects (font (size 1.27 1.27)) hide)
+    )
+    (property "Description" "Plugin,P=2.54mm Pin Headers ROHS" (at 185.42 110.49 0)
+      (effects (font (size 1.27 1.27)) hide)
+    )
+    (property "LCSC" "C5156075" (at 185.42 110.49 0)
+      (effects (font (size 1.27 1.27)) hide)
+    )
+    (property "MFR.Part" "54101-T30-00LF" (at 185.42 110.49 0)
+      (effects (font (size 1.27 1.27)) hide)
+    )
+    (pin "1")
+    (instances
+      (project "Module_1"
+        (path "/52aeb9ce-9f3b-4d8f-8c36-7e23df4a5f32/a62abef3-5f5d-4a40-b8c6-364ce9925bce"
+          (reference "J6") (unit 1)
+        )
+      )

Commit message: change for final 20.03.2024
Parts:
- J4, J5: footprint Z_pin:PinD3mm -> Z_pin:PinD2mm
Changed lines of the file:
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@@
       (effects (font (size 1.27 1.27)))
     )
-    (property "Footprint" "Z_pin:PinD3mm" (at 182.88 58.42 0)
+    (property "Footprint" "Z_pin:PinD2mm" (at 182.88 58.42 0)
       (effects (font (size 1.27 1.27)) hide)
     )
@@
       (effects (font (size 1.27 1.27)))
     )
-    (property "Footprint" "Z_pin:PinD3mm" (at 182.88 49.53 0)
-      (effects (font (size 1.27 1.27)) hide)
-    )
+    (property "Footprint" "Z_pin:PinD2mm" (at 182.88 49.53 0)
+      (effects (font (size 1.27 1.27)) hide)
+    )
