File: Projects/StationModules/Module_2/Module2_sheet2.kicad_sch (KiCad schematic)
At the start: 7 parts

Commit message: sheet 2 Module 2
Parts:
- added C14, C15: 47uF 16v, symbol Device:C_Polarized_Small
- added C16, C17: 4,7uF 16v, symbol Device:C_Polarized_Small
- added C18: 0,47uF, symbol Device:C_Small
- added C19: 0,15uF, symbol Device:C_Small
- added C20: 1,0uF, symbol Device:C_Small
- added C21: 0,1uF, symbol Device:C_Small
- added C22: C_Small, symbol Device:C_Small
- added D2, D3, D4, D5: D, symbol Device:D
- added J6: I, Connector_Pin:Pin_D1.0mm_L10.0mm, symbol Connector:Conn_01x01_Pin
- added J7: U, Connector_Pin:Pin_D1.0mm_L10.0mm, symbol Connector:Conn_01x01_Pin
- added J8: GND, Connector_Pin:Pin_D1.0mm_L10.0mm, symbol Connector:Conn_01x01_Pin
- added R15, R22, R23: 1k, symbol Device:R
- added R16, R20, R21, R25: 10k, symbol Device:R
- added R17: 100k, symbol Device:R
- added R18: 200k, symbol Device:R
- added R19: 10, symbol Device:R
- added R24: 1M, symbol Device:R
- added R26: R, symbol Device:R
- added RV1: 200k, symbol Device:R_Potentiometer
- added U4: LM2904, symbol Amplifier_Operational:LM2904
- added U5: LM358, symbol Amplifier_Operational:LM358
Connections:
- net +12V: now also C15.1, C21.1, D4.1 (K), R17.1, U4.8 (V+), U5.8 (V+)
- net +5V: now also D2.1 (K), D3.1 (K), D5.1 (K)
- net F_IN: now also R24.1, R25.1
- net GND: now also C14.2, C15.2, C16.2, C17.2, C19.2, C21.2, C22.2, J8.1 (Pin_1), R19.2, R24.2, U4.4 (V-), U5.4 (V-)
- new net: R18.2, RV1.1
- new net: C18.2, C19.1, R20.1, RV1.2, RV1.3, U4.1, U5.3 (+)
- new net: D4.2 (A), R25.2, U5.5 (+)
- new net: J7.1 (Pin_1), R15.1
- new net: R17.2, R19.1, U4.3 (+)
- new net: R22.1, U5.1, U5.2 (-)
- new net: C18.1, R16.2, R18.1, U4.2 (-)
- new net: C20.1, R20.2, U4.6 (-)
- new net: C17.1, R21.1, U4.5 (+)
- new net: C20.2, R23.1, U4.7
- new net: J6.1 (Pin_1), R16.1
- new net: R26.1, U5.6 (-), U5.7
- new net FI: C22.1, D5.2 (A), R26.2
- new net I_IN: C16.1, D2.2 (A), R22.2
- new net OS: D3.2 (A), R23.2
- new net PWM: R21.2
- new net U_IN: C14.1, R15.2
Other:
- moved on the sheet: C11, C13

Commit message: module 2 pcb ver1
Parts:
- C10: renamed from C14; footprint (none) -> Capacitor_THT:CP_Radial_D8.0mm_P5.00mm
- C13: renamed from C18; footprint (none) -> Capacitor_SMD:C_1206_3216Metric
- C15: footprint (none) -> Capacitor_THT:CP_Radial_D8.0mm_P5.00mm
- C17: renamed from C19; footprint (none) -> Capacitor_SMD:C_1206_3216Metric
- C18: renamed from C17; footprint (none) -> Capacitor_THT:CP_Radial_D8.0mm_P5.00mm
- C19: renamed from C21; footprint (none) -> Capacitor_SMD:C_1206_3216Metric
- C20: footprint (none) -> Capacitor_SMD:C_1206_3216Metric
- C21: renamed from C16; footprint (none) -> Capacitor_THT:CP_Radial_D8.0mm_P5.00mm
- C22: value C_Small -> 0,1uF; footprint (none) -> Capacitor_SMD:C_1206_3216Metric
- D2, D3, D4, D5: value D -> LL4148; footprint (none) -> Diode_SMD:D_MiniMELF
- J8: renamed from J5; footprint (none) -> Connector_IDC:IDC-Header_2x05_P2.54mm_Vertical
- R14: renamed from R15; footprint (none) -> Resistor_SMD:R_1206_3216Metric
- R16, R17, R20, R21, R22, R23, R24, R25: footprint (none) -> Resistor_SMD:R_1206_3216Metric
- R18: renamed from R19; footprint (none) -> Resistor_SMD:R_1206_3216Metric
- R19: renamed from R18; footprint (none) -> Resistor_SMD:R_1206_3216Metric
- R26: value R -> 1k; footprint (none) -> Resistor_SMD:R_1206_3216Metric
- RV1: footprint (none) -> Potentiometer_THT:Potentiometer_Bourns_3296W_Vertical
- U4, U5: footprint (none) -> Package_SO:SO-8_3.9x4.9mm_P1.27mm
- renumbered C10 to C11, C11 to C12, C13 to C14, C12 to C16, J6 to J5, J7 to J6, J8 to J7, R14 to R15
Connections:
- net U: now reaches J6.1 (Pin_1), R14.1
- net I: now reaches J5.1 (Pin_1), R16.1
Other:
- note added: "0...12v"
- moved on the sheet: C10, C11, C12, C13, C14, C15, C16, C17, C18, C19, C20, C21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

Commit message: module 2 board complit v1
Parts:
- added L2: 220uH THT, Inductor_THT:L_Axial_L7.0mm_D3.3mm_P10.16mm_Horizontal_Fastron_MICC, symbol Device:L
- L2: value 220uH -> 220uH SMD
Connections:
- net +12V: now also L2.2
- net +12VA: now reaches J8.1, J8.2, L2.1
- net +12VA: now also L2.1
Changed lines of the file:
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@@
   (junction (at 218.44 120.65) (diameter 0) (color 0 0 0 0)
   )
+  (junction (at 86.36 130.81) (diameter 0) (color 0 0 0 0)
+  )
   (junction (at 142.24 43.18) (diameter 0) (color 0 0 0 0)
   )
@@
   (junction (at 135.89 83.82) (diameter 0) (color 0 0 0 0)
   )
+  (junction (at 66.04 130.81) (diameter 0) (color 0 0 0 0)
+  )
   (junction (at 119.38 66.04) (diameter 0) (color 0 0 0 0)
   )
@@
   (junction (at 95.25 49.53) (diameter 0) (color 0 0 0 0)
   )
+  (junction (at 78.74 130.81) (diameter 0) (color 0 0 0 0)
+  )
   (junction (at 194.31 133.35) (diameter 0) (color 0 0 0 0)
   )
@@
     (stroke (width 0) (type default))
   )
+  (wire (pts (xy 66.04 130.81) (xy 74.93 130.81))
+    (stroke (width 0) (type default))
+  )
   (wire (pts (xy 144.78 54.61) (xy 162.56 54.61))
     (stroke (width 0) (type default))
@@
     (stroke (width 0) (type default))
   )
-  (wire (pts (xy 55.88 130.81) (xy 74.93 130.81))
+  (wire (pts (xy 55.88 130.81) (xy 66.04 130.81))
     (stroke (width 0) (type default))
   )
@@
     (stroke (width 0) (type default))
   )
+  (wire (pts (xy 78.74 123.19) (xy 78.74 130.81))
+    (stroke (width 0) (type default))
+  )
   (wire (pts (xy 74.93 135.89) (xy 73.66 135.89))
     (stroke (width 0) (type default))
@@
     (stroke (width 0) (type default))
   )
+  (wire (pts (xy 86.36 123.19) (xy 86.36 130.81))
+    (stroke (width 0) (type default))
+  )
   (wire (pts (xy 76.2 146.05) (xy 73.66 146.05))
     (stroke (width 0) (type default))
@@
   )
   (wire (pts (xy 171.45 118.11) (xy 175.26 118.11))
+    (stroke (width 0) (type default))
+  )
+  (wire (pts (xy 66.04 119.38) (xy 66.04 130.81))
     (stroke (width 0) (type default))
   )
@@
         (path "/d9631a92-6a8d-4456-a627-6fb12cee70ca/49eb342e-ce85-4fb3-a2fe-20bfac22dbdc"
           (reference "C15") (unit 1)
+        )
+      )
+    )
+  )
+  (symbol (lib_id "power:+12VA") (at 66.04 119.38 0) (unit 1)
+    (in_bom yes) (on_board yes) (dnp no) (fields_autoplaced)
+    (property "Reference" "#PWR042" (at 66.04 123.19 0)
+      (effects (font (size 1.27 1.27)) hide)
+    )
+    (property "Value" "+12VA" (at 66.04 115.57 0)
+      (effects (font (size 1.27 1.27)))
+    )
+    (property "Footprint" "" (at 66.04 119.38 0)
+      (effects (font (size 1.27 1.27)) hide)
+    )
+    (property "Datasheet" "" (at 66.04 119.38 0)
+      (effects (font (size 1.27 1.27)) hide)
+    )
+    (pin "1")
+    (instances
+      (project "Module_2"
+        (path "/d9631a92-6a8d-4456-a627-6fb12cee70ca/49eb342e-ce85-4fb3-a2fe-20bfac22dbdc"
+          (reference "#PWR042") (unit 1)
         )
       )
@@
     )
   )
+  (symbol (lib_id "Device:L") (at 82.55 123.19 90) (unit 1)
+    (in_bom yes) (on_board yes) (dnp no)
+    (property "Reference" "L2" (at 82.55 119.38 90)
+      (effects (font (size 1.27 1.27)))
+    )
+    (property "Value" "220uH THT" (at 83.262 121.3983 90)
+      (effects (font (size 1.27 1.27)))
+    )
+    (property "Footprint" "Inductor_THT:L_Axial_L7.0mm_D3.3mm_P10.16mm_Horizontal_Fastron_MICC" (at 82.55 123.19 0)
+      (effects (font (size 1.27 1.27)) hide)
+    )
+    (property "Datasheet" "~" (at 82.55 123.19 0)
+      (effects (font (size 1.27 1.27)) hide)
+    )
+    (property "Mfr. Part. No" "CY43-220UH" (at 82.55 123.19 0)
+      (effects (font (size 1.27 1.27)) hide)
+    )
+    (pin "1")
+    (pin "2")
+    (instances
+      (project "Module_2"
+        (path "/d9631a92-6a8d-4456-a627-6fb12cee70ca"
+          (reference "L2") (unit 1)
+        )
+        (path "/d9631a92-6a8d-4456-a627-6fb12cee70ca/49eb342e-ce85-4fb3-a2fe-20bfac22dbdc"
+          (reference "L3") (unit 1)
+        )
+      )
+    )
+  )
   (symbol (lib_id "power:GND") (at 99.06 154.94 0) (unit 1)
     (in_bom yes) (on_board yes) (dnp no)
@@
       (effects (font (size 1.27 1.27)))
     )
-    (property "Value" "220uH" (at 83.262 129.0183 90)
-      (effects (font (size 1.27 1.27)))
-    )
+    (property "Value" "220uH  SMD" (at 85.6139 128.8843 90)
+      (effects (font (size 1.27 1.27)))
+    )

Commit message: add bom module 1
Parts:
- L2: Mfr. Part. No CY43-220UH -> (none)

Commit message: add bom and pos
Parts:
- C10, C15: LCSC (none) -> C108854; MFR.Part (none) -> 16MS747MEFC5X7
- C11: LCSC (none) -> C108735; MFR.Part (none) -> 16YXJ100M5X11
- C12: LCSC (none) -> C694350; MFR.Part (none) -> 6.3YXJ1000M8X11.5
- C13: LCSC (none) -> C277483; MFR.Part (none) -> CC1206KKX7R9BB474
- C14, C19, C22: LCSC (none) -> C82601; MFR.Part (none) -> CC1206KRX7R9BB104
- C16: value 0,1uf -> 0,1uF; LCSC (none) -> C82601; MFR.Part (none) -> CC1206KRX7R9BB104
- C17: LCSC (none) -> C2171172; MFR.Part (none) -> CC1206JKX7R9BB154
- C18, C21: LCSC (none) -> C122950; MFR.Part (none) -> 50PX4R7MEFC5X11
- C20: LCSC (none) -> C107185; MFR.Part (none) -> CC1206KKX7R9BB105
- D2, D3, D4, D5: LCSC (none) -> C2891733; MFR.Part (none) -> LL4148
- J8: LCSC (none) -> C6332196; MFR.Part (none) -> HB-PH3-25413PB2GOP
- L2: LCSC (none) -> C492283; MFR.Part (none) -> CD43YP0403-221M
- R14, R22, R23, R26: LCSC (none) -> C112223; MFR.Part (none) -> RC1206JR-071KL
- R15: LCSC (none) -> C137179; MFR.Part (none) -> RC1206JR-0720KL
- R16, R20, R21, R25: LCSC (none) -> C136460; MFR.Part (none) -> RC1206JR-0710KL
- R17: LCSC (none) -> C136470; MFR.Part (none) -> RC1206JR-07100KL
- R18: LCSC (none) -> C137208; MFR.Part (none) -> RC1206JR-0710RL
- R19: LCSC (none) -> C137180; MFR.Part (none) -> RC1206JR-07200KL
- R24: LCSC (none) -> C148194; MFR.Part (none) -> RC1206JR-071ML
- RV1: LCSC (none) -> C58354; MFR.Part (none) -> 3296W-1-204LF
- U4: LCSC (none) -> C2941725; MFR.Part (none) -> LM2904
- U5: LCSC (none) -> C2683482; MFR.Part (none) -> LM358D

Commit message: change module1,2
Parts:
- R18: value 10 -> 0; LCSC C137208 -> C17888; MFR.Part RC1206JR-0710RL -> 1206W4F0000T5E
- R19: value 200k -> 330k; LCSC C137180 -> C17929; MFR.Part RC1206JR-07200KL -> 1206W4F3303T5E
- R20: value 10k -> 39k; LCSC C136460 -> C2907491; MFR.Part RC1206JR-0710KL -> FRC1206J393 TS
Changed lines of the file:
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@@
       (effects (font (size 1.27 1.27)))
     )
-    (property "Value" "10" (at 90.17 74.93 90)
+    (property "Value" "0" (at 90.17 74.93 90)
       (effects (font (size 1.27 1.27)))
     )
@@
       (effects (font (size 1.27 1.27)) hide)
     )
-    (property "MFR.Part" "RC1206JR-0710RL" (at 90.17 74.93 0)
-      (effects (font (size 1.27 1.27)) hide)
-    )
-    (property "Description" "250mW Thick Film Resistors ±5% ±200ppm/℃ 10Ω 1206 Chip Resistor - Surface Mount ROHS" (at 90.17 74.93 0)
-      (effects (font (size 1.27 1.27)) hide)
-    )
-    (property "LCSC" "C137208" (at 90.17 74.93 0)
+    (property "MFR.Part" "1206W4F0000T5E" (at 90.17 74.93 0)
+      (effects (font (size 1.27 1.27)) hide)
+    )
+    (property "Description" "250mW Thick Film Resistors ±800ppm/℃ ±1% 0Ω 1206 Chip Resistor - Surface Mount ROHS" (at 90.17 74.93 0)
+      (effects (font (size 1.27 1.27)) hide)
+    )
+    (property "LCSC" "C17888" (at 90.17 74.93 0)
       (effects (font (size 1.27 1.27)) hide)
     )
@@
       (effects (font (size 1.27 1.27)))
     )
-    (property "Value" "200k" (at 100.33 49.53 90)
+    (property "Value" "330k" (at 100.33 49.53 90)
       (effects (font (size 1.27 1.27)))
     )
@@
       (effects (font (size 1.27 1.27)) hide)
     )
-    (property "MFR.Part" "RC1206JR-07200KL" (at 100.33 49.53 0)
-      (effects (font (size 1.27 1.27)) hide)
-    )
-    (property "Description" "250mW Thick Film Resistors ±100ppm/℃ ±5% 200kΩ 1206 Chip Resistor - Surface Mount ROHS" (at 100.33 49.53 0)
-      (effects (font (size 1.27 1.27)) hide)
-    )
-    (property "LCSC" "C137180" (at 100.33 49.53 0)
+    (property "MFR.Part" "1206W4F3303T5E" (at 100.33 49.53 0)
+      (effects (font (size 1.27 1.27)) hide)
+    )
+    (property "Description" "250mW Thick Film Resistors ±100ppm/℃ ±1% 330kΩ 1206 Chip Resistor - Surface Mount ROHS" (at 100.33 49.53 0)
+      (effects (font (size 1.27 1.27)) hide)
+    )
+    (property "LCSC" "C17929" (at 100.33 49.53 0)
       (effects (font (size 1.27 1.27)) hide)
     )
@@
       (effects (font (size 1.27 1.27)))
     )
-    (property "Value" "10k" (at 125.73 66.04 90)
+    (property "Value" "39k" (at 125.73 66.04 90)
       (effects (font (size 1.27 1.27)))
     )
@@
       (effects (font (size 1.27 1.27)) hide)
     )
-    (property "MFR.Part" "RC1206JR-0710KL" (at 125.73 66.04 0)
-      (effects (font (size 1.27 1.27)) hide)
-    )
-    (property "Description" "250mW Thick Film Resistors ±100ppm/℃ ±5% 10kΩ 1206 Chip Resistor - Surface Mount ROHS" (at 125.73 66.04 0)
-      (effects (font (size 1.27 1.27)) hide)
-    )
-    (property "LCSC" "C136460" (at 125.73 66.04 0)
-      (effects (font (size 1.27 1.27)) hide)
-    )
+    (property "MFR.Part" "FRC1206J393 TS" (at 125.73 66.04 0)
+      (effects (font (size 1.27 1.27)) hide)
+    )
+    (property "Description" "250mW Thick Film Resistors ±100ppm/℃ ±5% 39kΩ 1206 Chip Resistor - Surface Mount ROHS" (at 125.73 66.04 0)
+      (effects (font (size 1.27 1.27)) hide)
+    )
+    (property "LCSC" "C2907491" (at 125.73 66.04 0)
+      (effects (font (size 1.27 1.27)) hide)
+    )

Commit message: change on 25_02_24
Parts:
- C10, C15: LCSC C108854 -> C59402; MFR.Part 16MS747MEFC5X7 -> KM470M016C110A; Mounting (none) -> Yes
- C11, C12, C13, C14, C16, C17, C18, C19, C20, C21, C22, D2, D3, D4, D5, L2, R15, R16, R18, R19, R20, R21, R24, R25, RV1, U4, U5: Mounting (none) -> Yes
- J5, J6, J7, L2, R17: Mounting (none) -> No
- J8: LCSC C6332196 -> C5665; MFR.Part HB-PH3-25413PB2GOP -> C5665; Mounting (none) -> Yes
- R14, R22, R23, R26: LCSC C112223 -> C4410; MFR.Part RC1206JR-071KL -> 1206W4F1001T5E; Mounting (none) -> Yes
