File: Projects/StationModules/Module_2/Module2_sheet3.kicad_sch (KiCad schematic)
At the start: 0 parts

Commit message: module 2 pcb ver1
Parts:
- added C23: C, Capacitor_THT:C_Rect_L7.0mm_W2.0mm_P5.00mm, symbol Device:C_Small
- added C24, C25: C, Capacitor_THT:C_Rect_L31.5mm_W15.0mm_P27.50mm_MKS4, symbol Device:C_Small
- added D6: 20B100, Package_TO_SOT_THT:TO-247-3_Horizontal_TabUp, symbol Device:D_Dual_CommonCathode_AKA_Parallel
- added J12, J13, J14, J15: Screw_Terminal_01x01, Z_pin:PinD3mm, symbol Connector:Screw_Terminal_01x01
- added J18: Screw_Terminal_01x03, Z_connectors:Klema3, symbol Connector:Screw_Terminal_01x03
- added J9: Screw_Terminal_01x02, Z_connectors:Klema2, symbol Connector:Screw_Terminal_01x02
- added R27, R28: R 2W, Resistor_THT:R_Axial_DIN0516_L15.5mm_D5.0mm_P20.32mm_Horizontal, symbol Device:R
- added R29, R30: R, Resistor_SMD:R_1206_3216Metric, symbol Device:R
- added R31, R32, R33, R34, R35: 0,01, Resistor_SMD:R_2816_7142Metric, symbol Device:R
- added RV2: 4k7 3296W, Potentiometer_THT:Potentiometer_Bourns_3296W_Vertical, symbol Device:R_Potentiometer
Connections:
- new net: D6.1 (K), J18.1 (Pin_1), R27.1, R28.1
- new net: C23.1, R27.2, R28.2
- new net: C24.1, C25.1, J13.1 (Pin_1), J9.2 (Pin_2), R29.1
- new net: R30.2, RV2.1
- new net: R29.2, R30.1
- new net: D6.2 (A), J12.1 (Pin_1)
- new net: C23.2, D6.3 (K), J18.2 (Pin_2)
- new net GND: J15.1 (Pin_1), J9.1 (Pin_1), R31.2, R32.2, R33.2, R34.2, R35.2, RV2.3
- new net I: C24.2, C25.2, J14.1 (Pin_1), J18.3 (Pin_3), R31.1, R32.1, R33.1, R34.1, R35.1
- new net U: RV2.2

Commit message: add bom and pos
Parts:
- D6: LCSC (none) -> C916352; MFR.Part (none) -> MBRF20100CT
- R29, R30: value R -> 22k; LCSC (none) -> C229910; MFR.Part (none) -> AC1206JR-0722KL
- R31, R32, R33, R34, R35: LCSC (none) -> C843884; MFR.Part (none) -> WSL2816R0100FEH
- RV2: value 4k7 3296W -> 5k; LCSC (none) -> C118907; MFR.Part (none) -> 3296W-1-502

Commit message: finaly on summer
Parts:
- C23: value C -> 4n7; footprint Capacitor_THT:C_Rect_L7.0mm_W2.0mm_P5.00mm -> Capacitor_THT:C_Rect_L11.5mm_W5.2mm_P10.00mm_MKT; LCSC (none) -> C506828; MFR.Part (none) -> MPP472J2J10AJ22610
- C24, C25: value C -> 10uF; LCSC (none) -> C5116053; MFR.Part (none) -> KP106J2E2701
- R27, R28: value R 2W -> 20; LCSC (none) -> C119690; MFR.Part (none) -> MF3WS-20Ω±1% T
Changed lines of the file:
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@@
       (effects (font (size 1.27 1.27)) (justify left))
     )
-    (property "Value" "R 2W" (at 63.5 59.69 0)
+    (property "Value" "20" (at 63.5 59.69 0)
       (effects (font (size 1.27 1.27)) (justify left))
     )
@@
       (effects (font (size 1.27 1.27)) hide)
     )
-    (property "MFR.Part" "" (at 69.85 60.96 0)
-      (effects (font (size 1.27 1.27)) hide)
-    )
-    (property "Description" "" (at 69.85 60.96 0)
-      (effects (font (size 1.27 1.27)) hide)
-    )
-    (property "LCSC" "" (at 69.85 60.96 0)
+    (property "MFR.Part" "MF3WS-20Ω±1% T" (at 69.85 60.96 0)
+      (effects (font (size 1.27 1.27)) hide)
+    )
+    (property "Description" "Metal Film Resistors 20Ω 3W ±100ppm/℃ ±1% Plugin,5x15.5mm Through Hole Resistors ROHS" (at 69.85 60.96 0)
+      (effects (font (size 1.27 1.27)) hide)
+    )
+    (property "LCSC" "C119690" (at 69.85 60.96 0)
       (effects (font (size 1.27 1.27)) hide)
     )
@@
       (effects (font (size 1.27 1.27)))
     )
-    (property "Value" "R 2W" (at 83.82 59.69 0)
+    (property "Value" "20" (at 83.82 59.69 0)
       (effects (font (size 1.27 1.27)))
     )
@@
       (effects (font (size 1.27 1.27)) hide)
     )
-    (property "MFR.Part" "" (at 80.01 60.96 0)
-      (effects (font (size 1.27 1.27)) hide)
-    )
-    (property "Description" "" (at 80.01 60.96 0)
-      (effects (font (size 1.27 1.27)) hide)
-    )
-    (property "LCSC" "" (at 80.01 60.96 0)
+    (property "MFR.Part" "MF3WS-20Ω±1% T" (at 80.01 60.96 0)
+      (effects (font (size 1.27 1.27)) hide)
+    )
+    (property "Description" "Metal Film Resistors 20Ω 3W ±100ppm/℃ ±1% Plugin,5x15.5mm Through Hole Resistors ROHS" (at 80.01 60.96 0)
+      (effects (font (size 1.27 1.27)) hide)
+    )
+    (property "LCSC" "C119690" (at 80.01 60.96 0)
       (effects (font (size 1.27 1.27)) hide)
     )
@@
       (effects (font (size 1.27 1.27)) (justify left))
     )
-    (property "Value" "C" (at 134.874 79.502 0)
+    (property "Value" "10uF" (at 134.874 79.502 0)
       (effects (font (size 1.27 1.27)) (justify left))
     )
@@
       (effects (font (size 1.27 1.27)) hide)
     )
-    (property "MFR.Part" "" (at 134.62 77.47 0)
-      (effects (font (size 1.27 1.27)) hide)
-    )
-    (property "Description" "" (at 134.62 77.47 0)
-      (effects (font (size 1.27 1.27)) hide)
-    )
-    (property "LCSC" "" (at 134.62 77.47 0)
+    (property "MFR.Part" "KP106J2E2701" (at 134.62 77.47 0)
+      (effects (font (size 1.27 1.27)) hide)
+    )
+    (property "Description" "10uF ±5% 250V Plugin,P=27.5mm Polypropylene Film Capacitors (CBB) ROHS" (at 134.62 77.47 0)
+      (effects (font (size 1.27 1.27)) hide)
+    )
+    (property "LCSC" "C5116053" (at 134.62 77.47 0)
       (effects (font (size 1.27 1.27)) hide)
     )
@@
       (effects (font (size 1.27 1.27)) (justify left))
     )
-    (property "Value" "C" (at 124.714 79.502 0)
+    (property "Value" "10uF" (at 124.714 79.502 0)
       (effects (font (size 1.27 1.27)) (justify left))
     )
@@
       (effects (font (size 1.27 1.27)) hide)
     )
-    (property "MFR.Part" "" (at 124.46 77.47 0)
-      (effects (font (size 1.27 1.27)) hide)
-    )
-    (property "Description" "" (at 124.46 77.47 0)
-      (effects (font (size 1.27 1.27)) hide)
-    )
-    (property "LCSC" "" (at 124.46 77.47 0)
+    (property "MFR.Part" "KP106J2E2701" (at 124.46 77.47 0)
+      (effects (font (size 1.27 1.27)) hide)
+    )
+    (property "Description" "10uF ±5% 250V Plugin,P=27.5mm Polypropylene Film Capacitors (CBB) ROHS" (at 124.46 77.47 0)
+      (effects (font (size 1.27 1.27)) hide)
+    )
+    (property "LCSC" "C5116053" (at 124.46 77.47 0)
       (effects (font (size 1.27 1.27)) hide)
     )
@@
       (effects (font (size 1.27 1.27)) (justify left))
     )
-    (property "Value" "C" (at 77.47 73.0313 0)
-      (effects (font (size 1.27 1.27)) (justify left))
-    )
-    (property "Footprint" "Capacitor_THT:C_Rect_L7.0mm_W2.0mm_P5.00mm" (at 74.93 71.12 0)
+    (property "Value" "4n7" (at 77.47 73.0313 0)
+      (effects (font (size 1.27 1.27)) (justify left))
+    )
+    (property "Footprint" "Capacitor_THT:C_Rect_L11.5mm_W5.2mm_P10.00mm_MKT" (at 74.93 71.12 0)
       (effects (font (size 1.27 1.27)) hide)
     )
@@
       (effects (font (size 1.27 1.27)) hide)
     )
-    (property "MFR.Part" "" (at 74.93 71.12 0)
-      (effects (font (size 1.27 1.27)) hide)
-    )
-    (property "Description" "" (at 74.93 71.12 0)
-      (effects (font (size 1.27 1.27)) hide)
-    )
-    (property "LCSC" "" (at 74.93 71.12 0)
-      (effects (font (size 1.27 1.27)) hide)
-    )
+    (property "MFR.Part" "MPP472J2J10AJ22610" (at 74.93 71.12 0)
+      (effects (font (size 1.27 1.27)) hide)
+    )
+    (property "Description" "4.7nF ±5% 630V Plugin,P=10mm Polypropylene Film Capacitors (CBB) ROHS" (at 74.93 71.12 0)
+      (effects (font (size 1.27 1.27)) hide)
+    )
+    (property "LCSC" "C506828" (at 74.93 71.12 0)
+      (effects (font (size 1.27 1.27)) hide)
+    )

Commit message: change module1,2
Parts:
- removed J14, J15: Screw_Terminal_01x01, Z_pin:PinD3mm, symbol Connector:Screw_Terminal_01x01
- removed R35: 0,01, Resistor_SMD:R_2816_7142Metric, symbol Device:R
- R27, R28: value 20 -> 120; LCSC C119690 -> C5200479; MFR.Part MF3WS-20Ω±1% T -> RSS3W120RJT76
Changed lines of the file:
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@@
   (junction (at 140.97 97.79) (diameter 0) (color 0 0 0 0)
   )
-  (junction (at 161.29 97.79) (diameter 0) (color 0 0 0 0)
-  )
-  (junction (at 140.97 130.81) (diameter 0) (color 0 0 0 0)
-  )
   (junction (at 80.01 53.34) (diameter 0) (color 0 0 0 0)
   )
   (junction (at 166.37 97.79) (diameter 0) (color 0 0 0 0)
   )
-  (junction (at 144.78 97.79) (diameter 0) (color 0 0 0 0)
-  )
   (junction (at 69.85 53.34) (diameter 0) (color 0 0 0 0)
   )
   (junction (at 74.93 66.04) (diameter 0) (color 0 0 0 0)
   )
-  (junction (at 161.29 130.81) (diameter 0) (color 0 0 0 0)
-  )
   (junction (at 140.97 120.65) (diameter 0) (color 0 0 0 0)
   )
@@
     (stroke (width 0) (type default))
   )
-  (wire (pts (xy 147.32 135.89) (xy 140.97 135.89))
-    (stroke (width 0) (type default))
-  )
   (wire (pts (xy 140.97 130.81) (xy 147.32 130.81))
     (stroke (width 0) (type default))
@@
     (stroke (width 0) (type default))
   )
-  (wire (pts (xy 140.97 130.81) (xy 140.97 135.89))
-    (stroke (width 0) (type default))
-  )
   (wire (pts (xy 87.63 63.5) (xy 91.44 63.5))
     (stroke (width 0) (type default))
@@
     (stroke (width 0) (type default))
   )
-  (wire (pts (xy 161.29 135.89) (xy 161.29 130.81))
-    (stroke (width 0) (type default))
-  )
   (wire (pts (xy 146.05 53.34) (xy 146.05 57.15))
     (stroke (width 0) (type default))
@@
     (stroke (width 0) (type default))
   )
-  (wire (pts (xy 154.94 97.79) (xy 161.29 97.79))
-    (stroke (width 0) (type default))
-  )
   (wire (pts (xy 58.42 66.04) (xy 50.8 66.04))
     (stroke (width 0) (type default))
@@
   )
   (wire (pts (xy 181.61 53.34) (xy 181.61 73.66))
-    (stroke (width 0) (type default))
-  )
-  (wire (pts (xy 154.94 135.89) (xy 161.29 135.89))
     (stroke (width 0) (type default))
   )
@@
       (effects (font (size 1.27 1.27)) (justify left))
     )
-    (property "Value" "20" (at 63.5 59.69 0)
+    (property "Value" "120" (at 63.5 59.69 0)
       (effects (font (size 1.27 1.27)) (justify left))
     )
@@
       (effects (font (size 1.27 1.27)) hide)
     )
-    (property "MFR.Part" "MF3WS-20Ω±1% T" (at 69.85 60.96 0)
-      (effects (font (size 1.27 1.27)) hide)
-    )
-    (property "Description" "Metal Film Resistors 20Ω 3W ±100ppm/℃ ±1% Plugin,5x15.5mm Through Hole Resistors ROHS" (at 69.85 60.96 0)
-      (effects (font (size 1.27 1.27)) hide)
-    )
-    (property "LCSC" "C119690" (at 69.85 60.96 0)
+    (property "MFR.Part" "RSS3W120RJT76" (at 69.85 60.96 0)
+      (effects (font (size 1.27 1.27)) hide)
+    )
+    (property "Description" "120Ω 3W ±5% - Through Hole Resistors ROHS" (at 69.85 60.96 0)
+      (effects (font (size 1.27 1.27)) hide)
+    )
+    (property "LCSC" "C5200479" (at 69.85 60.96 0)
       (effects (font (size 1.27 1.27)) hide)
     )
@@
       (effects (font (size 1.27 1.27)))
     )
-    (property "Value" "20" (at 83.82 59.69 0)
+    (property "Value" "120" (at 83.82 59.69 0)
       (effects (font (size 1.27 1.27)))
     )
@@
       (effects (font (size 1.27 1.27)) hide)
     )
-    (property "MFR.Part" "MF3WS-20Ω±1% T" (at 80.01 60.96 0)
-      (effects (font (size 1.27 1.27)) hide)
-    )
-    (property "Description" "Metal Film Resistors 20Ω 3W ±100ppm/℃ ±1% Plugin,5x15.5mm Through Hole Resistors ROHS" (at 80.01 60.96 0)
-      (effects (font (size 1.27 1.27)) hide)
-    )
-    (property "LCSC" "C119690" (at 80.01 60.96 0)
+    (property "MFR.Part" "RSS3W120RJT76" (at 80.01 60.96 0)
+      (effects (font (size 1.27 1.27)) hide)
+    )
+    (property "Description" "120Ω 3W ±5% - Through Hole Resistors ROHS" (at 80.01 60.96 0)
+      (effects (font (size 1.27 1.27)) hide)
+    )
+    (property "LCSC" "C5200479" (at 80.01 60.96 0)
       (effects (font (size 1.27 1.27)) hide)
     )
@@
         (path "/d9631a92-6a8d-4456-a627-6fb12cee70ca/12944bd1-a933-45dd-a80d-567cfd0dcce0"
           (reference "R34") (unit 1)
-        )
-      )
-    )
-  )
-  (symbol (lib_id "Connector:Screw_Terminal_01x01") (at 154.94 102.87 270) (unit 1)
-    (in_bom yes) (on_board yes) (dnp no)
-    (property "Reference" "J15" (at 157.48 102.87 0)
-      (effects (font (size 1.27 1.27)))
-    )
-    (property "Value" "Screw_Terminal_01x01" (at 152.4 102.87 0)
-      (effects (font (size 1.27 1.27)) hide)
-    )
-    (property "Footprint" "Z_pin:PinD3mm" (at 154.94 102.87 0)
-      (effects (font (size 1.27 1.27)) hide)
-    )
-    (property "Datasheet" "~" (at 154.94 102.87 0)
-      (effects (font (size 1.27 1.27)) hide)
-    )
-    (property "MFR.Part" "" (at 154.94 102.87 0)
-      (effects (font (size 1.27 1.27)) hide)
-    )
-    (property "Description" "" (at 154.94 102.87 0)
-      (effects (font (size 1.27 1.27)) hide)
-    )
-    (property "LCSC" "" (at 154.94 102.87 0)
-      (effects (font (size 1.27 1.27)) hide)
-    )
-    (pin "1")
-    (instances
-      (project "Module_2"
-        (path "/d9631a92-6a8d-4456-a627-6fb12cee70ca/12944bd1-a933-45dd-a80d-567cfd0dcce0"
-          (reference "J15") (unit 1)
-        )
-      )
-    )
-  )
-  (symbol (lib_id "Connector:Screw_Terminal_01x01") (at 144.78 102.87 270) (unit 1)
-    (in_bom yes) (on_board yes) (dnp no)
-    (property "Reference" "J14" (at 147.32 102.87 0)
-      (effects (font (size 1.27 1.27)))
-    )
-    (property "Value" "Screw_Terminal_01x01" (at 142.24 102.87 0)
-      (effects (font (size 1.27 1.27)) hide)
-    )
-    (property "Footprint" "Z_pin:PinD3mm" (at 144.78 102.87 0)
-      (effects (font (size 1.27 1.27)) hide)
-    )
-    (property "Datasheet" "~" (at 144.78 102.87 0)
-      (effects (font (size 1.27 1.27)) hide)
-    )
-    (property "MFR.Part" "" (at 144.78 102.87 0)
-      (effects (font (size 1.27 1.27)) hide)
-    )
-    (property "Description" "" (at 144.78 102.87 0)
-      (effects (font (size 1.27 1.27)) hide)
-    )
-    (property "LCSC" "" (at 144.78 102.87 0)
-      (effects (font (size 1.27 1.27)) hide)
-    )
-    (pin "1")
-    (instances
-      (project "Module_2"
-        (path "/d9631a92-6a8d-4456-a627-6fb12cee70ca/12944bd1-a933-45dd-a80d-567cfd0dcce0"
-          (reference "J14") (unit 1)
         )
       )
@@
         )
       )
-    )
-  )
-  (symbol (lib_id "Device:R") (at 151.13 135.89 90) (unit 1)
-    (in_bom yes) (on_board yes) (dnp no)
-    (property "Reference" "R35" (at 151.13 133.858 90)
-      (effects (font (size 1.27 1.27)))
-    )
-    (property "Value" "0,01" (at 151.13 135.89 90)
-      (effects (font (size 1.27 1.27)))
-    )
-    (property "Footprint" "Resistor_SMD:R_2816_7142Metric" (at 151.13 137.668 90)
-      (effects (font (size 1.27 1.27)) hide)
-    )
-    (property "Datasheet" "~" (at 151.13 135.89 0)
-      (effects (font (size 1.27 1.27)) hide)
-    )
-    (property "MFR.Part" "WSL2816R0100FEH" (at 151.13 135.89 0)
-      (effects (font (size 1.27 1.27)) hide)
-    )
-    (property "Description" "2W ±75ppm/℃ ±1% 10mΩ 2816 Chip Resistor - Surface Mount ROHS" (at 151.13 135.89 0)
-      (effects (font (size 1.27 1.27)) hide)
-    )
-    (property "LCSC" "C843884" (at 151.13 135.89 0)
-      (effects (font (size 1.27 1.27)) hide)
-    )
-    (pin "1")
-    (pin "2")
-    (instances
-      (project "Module_2"
-        (path "/d9631a92-6a8d-4456-a627-6fb12cee70ca/12944bd1-a933-45dd-a80d-567cfd0dcce0"
-          (reference "R35") (unit 1)
-        )
-      )

Commit message: change on 25_02_24
Parts:
- C23, C24, C25, R27, R28, R29, R30, R31, R32, R33, R34, RV2: Mounting (none) -> Yes
- D6, J12, J13, J18, J9: Mounting (none) -> No
Changed lines of the file:
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@@
+      (effects (font (size 1.27 1.27)) hide)
+    )
+    (property "Mounting" "Yes" (at 69.85 60.96 0)
       (effects (font (size 1.27 1.27)) hide)
     )
@@
       (effects (font (size 1.27 1.27)) hide)
     )
+    (property "Mounting" "No" (at 191.77 76.2 0)
+      (effects (font (size 1.27 1.27)) hide)
+    )
     (pin "1")
     (pin "2")
@@
     )
     (property "LCSC" "C5200479" (at 80.01 60.96 0)
+      (effects (font (size 1.27 1.27)) hide)
+    )
+    (property "Mounting" "Yes" (at 80.01 60.96 0)
       (effects (font (size 1.27 1.27)) hide)
     )
@@
       (effects (font (size 1.27 1.27)) hide)
     )
+    (property "Mounting" "Yes" (at 134.62 77.47 0)
+      (effects (font (size 1.27 1.27)) hide)
+    )
     (pin "1")
     (pin "2")
@@
     )
     (property "LCSC" "C118907" (at 154.94 77.47 0)
+      (effects (font (size 1.27 1.27)) hide)
+    )
+    (property "Mounting" "Yes" (at 154.94 77.47 0)
       (effects (font (size 1.27 1.27)) hide)
     )
@@
       (effects (font (size 1.27 1.27)) hide)
     )
+    (property "Mounting" "Yes" (at 124.46 77.47 0)
+      (effects (font (size 1.27 1.27)) hide)
+    )
     (pin "1")
     (pin "2")
@@
       (effects (font (size 1.27 1.27)) hide)
     )
+    (property "Mounting" "Yes" (at 151.13 120.65 0)
+      (effects (font (size 1.27 1.27)) hide)
+    )
     (pin "1")
     (pin "2")
@@
       (effects (font (size 1.27 1.27)) hide)
     )
+    (property "Mounting" "Yes" (at 146.05 71.12 0)
+      (effects (font (size 1.27 1.27)) hide)
+    )
     (pin "1")
     (pin "2")
@@
       (effects (font (size 1.27 1.27)) hide)
     )
+    (property "Mounting" "Yes" (at 151.13 130.81 0)
+      (effects (font (size 1.27 1.27)) hide)
+    )
     (pin "1")
     (pin "2")
@@
     )
     (property "LCSC" "C229910" (at 146.05 60.96 0)
+      (effects (font (size 1.27 1.27)) hide)
+    )
+    (property "Mounting" "Yes" (at 146.05 60.96 0)
       (effects (font (size 1.27 1.27)) hide)
     )
@@
     )
     (property "LCSC" "C916352" (at 96.52 66.04 0)
+      (effects (font (size 1.27 1.27)) hide)
+    )
+    (property "Mounting" "No" (at 96.52 66.04 0)
       (effects (font (size 1.27 1.27)) hide)
     )
@@
       (effects (font (size 1.27 1.27)) hide)
     )
+    (property "Mounting" "Yes" (at 74.93 71.12 0)
+      (effects (font (size 1.27 1.27)) hide)
+    )
     (pin "1")
     (pin "2")
@@
     )
     (property "LCSC" "" (at 116.84 48.26 0)
+      (effects (font (size 1.27 1.27)) hide)
+    )
+    (property "Mounting" "No" (at 116.84 48.26 0)
       (effects (font (size 1.27 1.27)) hide)
     )
@@
       (effects (font (size 1.27 1.27)) hide)
     )
+    (property "Mounting" "Yes" (at 151.13 115.57 0)
+      (effects (font (size 1.27 1.27)) hide)
+    )
     (pin "1")
     (pin "2")
@@
     )
     (property "LCSC" "C843884" (at 151.13 125.73 0)
+      (effects (font (size 1.27 1.27)) hide)
+    )
+    (property "Mounting" "Yes" (at 151.13 125.73 0)
       (effects (font (size 1.27 1.27)) hide)
     )
@@
       (effects (font (size 1.27 1.27)) hide)
     )
+    (property "Mounting" "No" (at 106.68 48.26 0)
+      (effects (font (size 1.27 1.27)) hide)
+    )
     (pin "1")
     (instances
@@
       (effects (font (size 1.27 1.27)) hide)
     )
+    (property "Mounting" "No" (at 45.72 66.04 0)
+      (effects (font (size 1.27 1.27)) hide)
+    )
