File: Projects/StationModules/Module_2/Module2_sheet3.kicad_sch (KiCad schematic)
At the start: 17 parts, among them J12 Screw_Terminal_01x01, J13 Screw_Terminal_01x01, J18 Screw_Terminal_01x03, J9 Screw_Terminal_01x02

Commit message: Corection all modules
Parts:
- added D7: 1.5KExxA, Diode_THT:D_DO-201AE_P15.24mm_Horizontal, symbol Diode:1.5KExxA
Connections:
- net GND: now also D7.2 (A2)
- net at C24.1, C25.1, J13.1 (Pin_1)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: now also D7.1 (A1)
Other:
- moved on the sheet: J9
Changed lines of the file:
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@@
   (junction (at 161.29 120.65) (diameter 0) (color 0 0 0 0)
   )
+  (junction (at 193.04 53.34) (diameter 0) (color 0 0 0 0)
+  )
   (junction (at 140.97 125.73) (diameter 0) (color 0 0 0 0)
   )
@@
   (junction (at 74.93 77.47) (diameter 0) (color 0 0 0 0)
   )
+  (junction (at 193.04 97.79) (diameter 0) (color 0 0 0 0)
+  )
   (junction (at 140.97 97.79) (diameter 0) (color 0 0 0 0)
   )
@@
     (stroke (width 0) (type default))
   )
-  (wire (pts (xy 181.61 73.66) (xy 186.69 73.66))
+  (wire (pts (xy 208.28 73.66) (xy 213.36 73.66))
     (stroke (width 0) (type default))
   )
@@
     (stroke (width 0) (type default))
   )
+  (wire (pts (xy 193.04 97.79) (xy 208.28 97.79))
+    (stroke (width 0) (type default))
+  )
   (wire (pts (xy 74.93 77.47) (xy 87.63 77.47))
     (stroke (width 0) (type default))
@@
     (stroke (width 0) (type default))
   )
+  (wire (pts (xy 193.04 77.47) (xy 193.04 97.79))
+    (stroke (width 0) (type default))
+  )
   (wire (pts (xy 116.84 53.34) (xy 124.46 53.34))
     (stroke (width 0) (type default))
@@
     (stroke (width 0) (type default))
   )
-  (wire (pts (xy 181.61 53.34) (xy 181.61 73.66))
+  (wire (pts (xy 208.28 53.34) (xy 208.28 73.66))
+    (stroke (width 0) (type default))
+  )
+  (wire (pts (xy 193.04 53.34) (xy 193.04 69.85))
     (stroke (width 0) (type default))
   )
@@
     (stroke (width 0) (type default))
   )
-  (wire (pts (xy 166.37 97.79) (xy 181.61 97.79))
+  (wire (pts (xy 166.37 97.79) (xy 193.04 97.79))
     (stroke (width 0) (type default))
   )
@@
     (stroke (width 0) (type default))
   )
-  (wire (pts (xy 181.61 76.2) (xy 186.69 76.2))
+  (wire (pts (xy 208.28 76.2) (xy 213.36 76.2))
     (stroke (width 0) (type default))
   )
@@
     (stroke (width 0) (type default))
   )
-  (wire (pts (xy 181.61 97.79) (xy 181.61 76.2))
+  (wire (pts (xy 208.28 97.79) (xy 208.28 76.2))
     (stroke (width 0) (type default))
   )
@@
     (stroke (width 0) (type default))
   )
+  (wire (pts (xy 193.04 53.34) (xy 208.28 53.34))
+    (stroke (width 0) (type default))
+  )
   (wire (pts (xy 58.42 53.34) (xy 58.42 63.5))
     (stroke (width 0) (type default))
@@
     (stroke (width 0) (type default))
   )
-  (wire (pts (xy 146.05 53.34) (xy 181.61 53.34))
+  (wire (pts (xy 146.05 53.34) (xy 193.04 53.34))
     (stroke (width 0) (type default))
   )
@@
     )
   )
-  (symbol (lib_id "Connector:Screw_Terminal_01x02") (at 191.77 76.2 0) (mirror x) (unit 1)
+  (symbol (lib_id "Diode:1.5KExxA") (at 193.04 73.66 270) (unit 1)
+    (in_bom yes) (on_board yes) (dnp no) (fields_autoplaced)
+    (property "Reference" "D7" (at 195.58 73.025 90)
+      (effects (font (size 1.27 1.27)) (justify left))
+    )
+    (property "Value" "1.5KExxA" (at 195.58 75.565 90)
+      (effects (font (size 1.27 1.27)) (justify left))
+    )
+    (property "Footprint" "Diode_THT:D_DO-201AE_P15.24mm_Horizontal" (at 187.96 73.66 0)
+      (effects (font (size 1.27 1.27)) hide)
+    )
+    (property "Datasheet" "https://www.vishay.com/docs/88301/15ke.pdf" (at 193.04 72.39 0)
+      (effects (font (size 1.27 1.27)) hide)
+    )
+    (property "LCSC" "C7464802" (at 193.04 73.66 0)
+      (effects (font (size 1.27 1.27)) hide)
+    )
+    (property "MFR.Part" "1.5KE220A" (at 193.04 73.66 0)
+      (effects (font (size 1.27 1.27)) hide)
+    )
+    (property "Description" "4.6A 328V 1.5kW Unidirectional 185V DO-201 Electrostatic and Surge Protection (TVS/ESD) ROHS" (at 193.04 73.66 0)
+      (effects (font (size 1.27 1.27)) hide)
+    )
+    (property "Mounting" "Yes" (at 193.04 73.66 0)
+      (effects (font (size 1.27 1.27)) hide)
+    )
+    (pin "1")
+    (pin "2")
+    (instances
+      (project "Module_2"
+        (path "/d9631a92-6a8d-4456-a627-6fb12cee70ca/12944bd1-a933-45dd-a80d-567cfd0dcce0"
+          (reference "D7") (unit 1)
+        )
+      )
+    )
+  )
+  (symbol (lib_id "Connector:Screw_Terminal_01x02") (at 218.44 76.2 0) (mirror x) (unit 1)
     (in_bom yes) (on_board yes) (dnp no)
-    (property "Reference" "J9" (at 191.77 71.12 0)
+    (property "Reference" "J9" (at 218.44 71.12 0)
       (effects (font (size 1.27 1.27)))
     )
-    (property "Value" "Screw_Terminal_01x02" (at 194.31 73.025 0)
+    (property "Value" "Screw_Terminal_01x02" (at 220.98 73.025 0)
       (effects (font (size 1.27 1.27)) (justify left) hide)
     )
-    (property "Footprint" "Z_connectors:Klema2" (at 191.77 76.2 0)
-      (effects (font (size 1.27 1.27)) hide)
-    )
-    (property "Datasheet" "~" (at 191.77 76.2 0)
-      (effects (font (size 1.27 1.27)) hide)
-    )
-    (property "MFR.Part" "" (at 191.77 76.2 0)
-      (effects (font (size 1.27 1.27)) hide)
-    )
-    (property "Description" "" (at 191.77 76.2 0)
-      (effects (font (size 1.27 1.27)) hide)
-    )
-    (property "LCSC" "" (at 191.77 76.2 0)
-      (effects (font (size 1.27 1.27)) hide)
-    )
-    (property "Mounting" "No" (at 191.77 76.2 0)
-      (effects (font (size 1.27 1.27)) hide)
-    )
+    (property "Footprint" "Z_connectors:Klema2" (at 218.44 76.2 0)
+      (effects (font (size 1.27 1.27)) hide)
+    )
+    (property "Datasheet" "~" (at 218.44 76.2 0)
+      (effects (font (size 1.27 1.27)) hide)
+    )
+    (property "MFR.Part" "" (at 218.44 76.2 0)
+      (effects (font (size 1.27 1.27)) hide)
+    )
+    (property "Description" "" (at 218.44 76.2 0)
+      (effects (font (size 1.27 1.27)) hide)
+    )
+    (property "LCSC" "" (at 218.44 76.2 0)
+      (effects (font (size 1.27 1.27)) hide)
+    )
+    (property "Mounting" "No" (at 218.44 76.2 0)
+      (effects (font (size 1.27 1.27)) hide)
+    )
