File: Projects/StationModules/Module_2/Module_2.kicad_sch (KiCad schematic)
At the start: 36 parts, among them J1 Conn_01x03_Pin, J2 Conn_01x03_Pin, Q1 IRLML2803, Q2 IRLML2803, Q3 IRLML2803, U1 ADM1485AR, U2 STM8S105K4T6C, U3 PC817, Y1 16MHz

Commit message: sheet 2 Module 2
Parts:
- Y1: footprint (none) -> Crystal:Crystal_HC49-4H_Vertical
Changed lines of the file:
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@@
       (effects (font (size 1.27 1.27)) (justify left))
     )
-    (property "Footprint" "" (at 81.28 58.42 0)
+    (property "Footprint" "Crystal:Crystal_HC49-4H_Vertical" (at 81.28 58.42 0)
       (effects (font (size 1.27 1.27)) hide)
     )

Commit message: module 2 pcb ver1
Parts:
- added H1, H2, H3, H4: MountingHole, MountingHole:MountingHole_3.5mm, symbol Mechanical:MountingHole
- C3, C5: footprint (none) -> Capacitor_SMD:C_1206_3216Metric
- J1, J2: footprint (none) -> Connector:FanPinHeader_1x03_P2.54mm_Vertical
- J3, J4: footprint (none) -> Connector_IDC:IDC-Header_2x05_P2.54mm_Vertical
- JP1: footprint (none) -> Connector_PinHeader_2.54mm:PinHeader_1x02_P2.54mm_Vertical
- R1, R10, R11, R12, R13, R2, R3, R4, R7, R9: footprint (none) -> Resistor_SMD:R_1206_3216Metric
Connections:
- net +5V: no longer C1.1, C2.1, C3.1, C4.2, C5.1, C6.2, C7.2, C8.2, C9.2, D1.2 (K), J1.2 (Pin_2), J2.3 (Pin_3), J3.1, J3.3, J3.5, J3.7, J3.9, J4.1, J4.3, J4.5, J4.7, J4.9, Q1.2 (S), Q2.2 (S), Q3.2 (S), R11.2, R7.2, R9.2, U1.5 (GND), U2.10 (VSSA), U2.4 (VSS), U3.2, U3.3
- new net GND: C1.1, C2.1, C3.1, C4.2, C5.1, C6.2, C7.2, C8.2, C9.2, D1.2 (K), J1.2 (Pin_2), J2.3 (Pin_3), J3.1, J3.3, J3.5, J3.7, J3.9, J4.1, J4.3, J4.5, J4.7, J4.9, Q1.2 (S), Q2.2 (S), Q3.2 (S), R11.2, R7.2, R9.2, U1.5 (GND), U2.10 (VSSA), U2.4 (VSS), U3.2, U3.3
Changed lines of the file:
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@@
   (junction (at 245.11 116.84) (diameter 0) (color 0 0 0 0)
   )
-  (junction (at 74.93 86.36) (diameter 0) (color 0 0 0 0)
-  )
   (junction (at 93.98 80.01) (diameter 0) (color 0 0 0 0)
   )
@@
   )
   (junction (at 215.9 55.88) (diameter 0) (color 0 0 0 0)
-  )
-  (junction (at 74.93 91.44) (diameter 0) (color 0 0 0 0)
   )
   (junction (at 93.98 86.36) (diameter 0) (color 0 0 0 0)
@@
     (stroke (width 0) (type default))
   )
-  (wire (pts (xy 74.93 86.36) (xy 74.93 91.44))
-    (stroke (width 0) (type default))
-  )
   (wire (pts (xy 210.82 93.98) (xy 245.11 93.98))
     (stroke (width 0) (type default))
@@
       (effects (font (size 1.27 1.27)))
     )
-    (property "Footprint" "" (at 85.852 149.86 90)
+    (property "Footprint" "Resistor_SMD:R_1206_3216Metric" (at 85.852 149.86 90)
       (effects (font (size 1.27 1.27)) hide)
     )
@@
     )
   )
+  (symbol (lib_id "Mechanical:MountingHole") (at 163.83 143.51 0) (unit 1)
+    (in_bom yes) (on_board yes) (dnp no)
+    (property "Reference" "H2" (at 163.83 138.43 0)
+      (effects (font (size 1.27 1.27)))
+    )
+    (property "Value" "MountingHole" (at 163.83 140.335 0)
+      (effects (font (size 1.27 1.27)))
+    )
+    (property "Footprint" "MountingHole:MountingHole_3.5mm" (at 163.83 143.51 0)
+      (effects (font (size 1.27 1.27)) hide)
+    )
+    (property "Datasheet" "~" (at 163.83 143.51 0)
+      (effects (font (size 1.27 1.27)) hide)
+    )
+    (instances
+      (project "Module_2"
+        (path "/d9631a92-6a8d-4456-a627-6fb12cee70ca"
+          (reference "H2") (unit 1)
+        )
+      )
+    )
+  )
   (symbol (lib_id "Device:C_Small") (at 71.12 36.83 0) (unit 1)
     (in_bom yes) (on_board yes) (dnp no)
@@
       (effects (font (size 1.27 1.27)) (justify left))
     )
-    (property "Footprint" "" (at 71.12 36.83 0)
+    (property "Footprint" "Capacitor_SMD:C_1206_3216Metric" (at 71.12 36.83 0)
       (effects (font (size 1.27 1.27)) hide)
     )
@@
       (effects (font (size 1.27 1.27)) hide)
     )
-    (property "Footprint" "" (at 120.65 148.59 0)
+    (property "Footprint" "Connector:FanPinHeader_1x03_P2.54mm_Vertical" (at 120.65 148.59 0)
       (effects (font (size 1.27 1.27)) hide)
     )
@@
       (effects (font (size 1.27 1.27)))
     )
-    (property "Footprint" "" (at 167.64 52.578 90)
+    (property "Footprint" "Resistor_SMD:R_1206_3216Metric" (at 167.64 52.578 90)
       (effects (font (size 1.27 1.27)) hide)
     )
@@
       (effects (font (size 1.27 1.27)))
     )
-    (property "Footprint" "" (at 74.93 147.828 90)
+    (property "Footprint" "Resistor_SMD:R_1206_3216Metric" (at 74.93 147.828 90)
       (effects (font (size 1.27 1.27)) hide)
     )
@@
       (effects (font (size 1.27 1.27)))
     )
-    (property "Footprint" "" (at 262.89 100.838 90)
+    (property "Footprint" "Resistor_SMD:R_1206_3216Metric" (at 262.89 100.838 90)
       (effects (font (size 1.27 1.27)) hide)
     )
@@
       (effects (font (size 1.27 1.27)))
     )
-    (property "Footprint" "" (at 90.17 69.85 0)
+    (property "Footprint" "Capacitor_SMD:C_1206_3216Metric" (at 90.17 69.85 0)
       (effects (font (size 1.27 1.27)) hide)
     )
@@
       (effects (font (size 1.27 1.27)))
     )
-    (property "Footprint" "" (at 264.922 129.54 90)
+    (property "Footprint" "Resistor_SMD:R_1206_3216Metric" (at 264.922 129.54 90)
       (effects (font (size 1.27 1.27)) hide)
     )
@@
       (effects (font (size 1.27 1.27)))
     )
-    (property "Footprint" "" (at 259.842 118.11 90)
+    (property "Footprint" "Resistor_SMD:R_1206_3216Metric" (at 259.842 118.11 90)
       (effects (font (size 1.27 1.27)) hide)
     )
@@
         (path "/d9631a92-6a8d-4456-a627-6fb12cee70ca"
           (reference "R9") (unit 1)
+        )
+      )
+    )
+  )
+  (symbol (lib_id "Mechanical:MountingHole") (at 143.51 143.51 0) (unit 1)
+    (in_bom yes) (on_board yes) (dnp no)
+    (property "Reference" "H1" (at 142.2682 138.4108 0)
+      (effects (font (size 1.27 1.27)) (justify left))
+    )
+    (property "Value" "MountingHole" (at 137.6423 140.2098 0)
+      (effects (font (size 1.27 1.27)) (justify left))
+    )
+    (property "Footprint" "MountingHole:MountingHole_3.5mm" (at 143.51 143.51 0)
+      (effects (font (size 1.27 1.27)) hide)
+    )
+    (property "Datasheet" "~" (at 143.51 143.51 0)
+      (effects (font (size 1.27 1.27)) hide)
+    )
+    (instances
+      (project "Module_2"
+        (path "/d9631a92-6a8d-4456-a627-6fb12cee70ca"
+          (reference "H1") (unit 1)
         )
       )
@@
         (path "/d9631a92-6a8d-4456-a627-6fb12cee70ca"
           (reference "Q2") (unit 1)
+        )
+      )
+    )
+  )
+  (symbol (lib_id "Mechanical:MountingHole") (at 163.83 157.48 0) (unit 1)
+    (in_bom yes) (on_board yes) (dnp no)
+    (property "Reference" "H4" (at 163.83 152.4 0)
+      (effects (font (size 1.27 1.27)))
+    )
+    (property "Value" "MountingHole" (at 163.83 154.305 0)
+      (effects (font (size 1.27 1.27)))
+    )
+    (property "Footprint" "MountingHole:MountingHole_3.5mm" (at 163.83 157.48 0)
+      (effects (font (size 1.27 1.27)) hide)
+    )
+    (property "Datasheet" "~" (at 163.83 157.48 0)
+      (effects (font (size 1.27 1.27)) hide)
+    )
+    (instances
+      (project "Module_2"
+        (path "/d9631a92-6a8d-4456-a627-6fb12cee70ca"
+          (reference "H4") (unit 1)
         )
       )
@@
       (effects (font (size 1.27 1.27)))
     )
-    (property "Footprint" "" (at 267.97 113.538 90)
+    (property "Footprint" "Resistor_SMD:R_1206_3216Metric" (at 267.97 113.538 90)
       (effects (font (size 1.27 1.27)) hide)
     )
@@
       (effects (font (size 1.27 1.27)))
     )
-    (property "Footprint" "" (at 208.28 113.03 0)
+    (property "Footprint" "Connector_IDC:IDC-Header_2x05_P2.54mm_Vertical" (at 208.28 113.03 0)
       (effects (font (size 1.27 1.27)) hide)
     )
@@
     )
   )
+  (symbol (lib_id "Mechanical:MountingHole") (at 143.51 157.48 0) (unit 1)
+    (in_bom yes) (on_board yes) (dnp no)
+    (property "Reference" "H3" (at 143.51 152.4 0)
+      (effects (font (size 1.27 1.27)))
+    )
+    (property "Value" "MountingHole" (at 143.51 154.305 0)
+      (effects (font (size 1.27 1.27)))
+    )
+    (property "Footprint" "MountingHole:MountingHole_3.5mm" (at 143.51 157.48 0)
+      (effects (font (size 1.27 1.27)) hide)
+    )
+    (property "Datasheet" "~" (at 143.51 157.48 0)
+      (effects (font (size 1.27 1.27)) hide)
+    )
+    (instances
+      (project "Module_2"
+        (path "/d9631a92-6a8d-4456-a627-6fb12cee70ca"
+          (reference "H3") (unit 1)
+        )
+      )
+    )
+  )
   (symbol (lib_id "power:GND") (at 226.06 128.27 0) (unit 1)
     (in_bom yes) (on_board yes) (dnp no) (fields_autoplaced)
@@
       (effects (font (size 1.27 1.27)))
     )
-    (property "Footprint" "" (at 236.22 50.8 0)
+    (property "Footprint" "Connector_IDC:IDC-Header_2x05_P2.54mm_Vertical" (at 236.22 50.8 0)
       (effects (font (size 1.27 1.27)) hide)
     )
@@
       (effects (font (size 1.27 1.27)))
     )
-    (property "Footprint" "" (at 74.93 155.448 90)
+    (property "Footprint" "Resistor_SMD:R_1206_3216Metric" (at 74.93 155.448 90)
       (effects (font (size 1.27 1.27)) hide)
     )
@@
       (effects (font (size 1.27 1.27)))
     )
-    (property "Footprint" "" (at 254.762 104.14 90)
+    (property "Footprint" "Resistor_SMD:R_1206_3216Metric" (at 254.762 104.14 90)
       (effects (font (size 1.27 1.27)) hide)
     )
@@
       (effects (font (size 1.27 1.27)) hide)
     )
-    (property "Footprint" "" (at 57.15 34.29 0)
+    (property "Footprint" "Connector:FanPinHeader_1x03_P2.54mm_Vertical" (at 57.15 34.29 0)
       (effects (font (size 1.27 1.27)) hide)
     )
@@
       (effects (font (size 1.27 1.27)))
     )
-    (property "Footprint" "" (at 273.05 124.968 90)
+    (property "Footprint" "Resistor_SMD:R_1206_3216Metric" (at 273.05 124.968 90)
       (effects (font (size 1.27 1.27)) hide)
     )
@@
       (effects (font (size 1.27 1.27)))
     )
-    (property "Footprint" "" (at 99.06 153.67 0)
-      (effects (font (size 1.27 1.27)) hide)
-    )
+    (property "Footprint" "Connector_PinHeader_2.54mm:PinHeader_1x02_P2.54mm_Vertical" (at 99.06 153.67 0)
+      (effects (font (size 1.27 1.27)) hide)
+    )

Commit message: module 2 board complit v1
Parts:
- added C26: 0,1uF, Resistor_SMD:R_1206_3216Metric, symbol Device:C_Small
- added J10: Conn_01x03_Pin, Connector:FanPinHeader_1x03_P2.54mm_Vertical, symbol Connector:Conn_01x03_Pin
Connections:
- net +5V: now also C26.1
- net GND: now also C26.2, J10.3 (Pin_3)
- net RX: now also J10.2 (Pin_2)
- net TX: now also J10.1 (Pin_1)
- net +12V renamed +12VA
Changed lines of the file:
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@@
   (junction (at 215.9 58.42) (diameter 0) (color 0 0 0 0)
+  )
+  (junction (at 55.88 132.08) (diameter 0) (color 0 0 0 0)
   )
   (junction (at 87.63 142.24) (diameter 0) (color 0 0 0 0)
@@
     (stroke (width 0) (type default))
   )
+  (wire (pts (xy 177.8 72.39) (xy 187.96 72.39))
+    (stroke (width 0) (type default))
+  )
   (wire (pts (xy 161.29 101.6) (xy 152.4 101.6))
     (stroke (width 0) (type default))
@@
     (stroke (width 0) (type default))
   )
-  (wire (pts (xy 152.4 73.66) (xy 161.29 73.66))
+  (wire (pts (xy 152.4 73.66) (xy 177.8 73.66))
     (stroke (width 0) (type default))
   )
@@
     (stroke (width 0) (type default))
   )
+  (wire (pts (xy 55.88 132.08) (xy 55.88 138.43))
+    (stroke (width 0) (type default))
+  )
+  (wire (pts (xy 186.69 74.93) (xy 187.96 74.93))
+    (stroke (width 0) (type default))
+  )
   (wire (pts (xy 265.43 48.26) (xy 265.43 50.8))
     (stroke (width 0) (type default))
@@
     (stroke (width 0) (type default))
   )
+  (wire (pts (xy 45.72 132.08) (xy 55.88 132.08))
+    (stroke (width 0) (type default))
+  )
   (wire (pts (xy 265.43 48.26) (xy 271.78 48.26))
     (stroke (width 0) (type default))
@@
     (stroke (width 0) (type default))
   )
-  (wire (pts (xy 55.88 137.16) (xy 55.88 138.43))
+  (wire (pts (xy 55.88 127) (xy 55.88 132.08))
     (stroke (width 0) (type default))
   )
@@
     (stroke (width 0) (type default))
   )
-  (wire (pts (xy 152.4 69.85) (xy 161.29 69.85))
+  (wire (pts (xy 152.4 69.85) (xy 187.96 69.85))
     (stroke (width 0) (type default))
   )
@@
     (stroke (width 0) (type default))
   )
+  (wire (pts (xy 186.69 80.01) (xy 186.69 74.93))
+    (stroke (width 0) (type default))
+  )
   (wire (pts (xy 44.45 148.59) (xy 45.72 148.59))
     (stroke (width 0) (type default))
@@
   )
   (wire (pts (xy 74.93 80.01) (xy 74.93 77.47))
+    (stroke (width 0) (type default))
+  )
+  (wire (pts (xy 177.8 73.66) (xy 177.8 72.39))
     (stroke (width 0) (type default))
   )
@@
     )
   )
+  (symbol (lib_id "power:GND") (at 45.72 137.16 0) (unit 1)
+    (in_bom yes) (on_board yes) (dnp no)
+    (property "Reference" "#PWR041" (at 45.72 143.51 0)
+      (effects (font (size 1.27 1.27)) hide)
+    )
+    (property "Value" "GND" (at 41.91 138.43 0)
+      (effects (font (size 1.27 1.27)))
+    )
+    (property "Footprint" "" (at 45.72 137.16 0)
+      (effects (font (size 1.27 1.27)) hide)
+    )
+    (property "Datasheet" "" (at 45.72 137.16 0)
+      (effects (font (size 1.27 1.27)) hide)
+    )
+    (pin "1")
+    (instances
+      (project "Module_2"
+        (path "/d9631a92-6a8d-4456-a627-6fb12cee70ca"
+          (reference "#PWR041") (unit 1)
+        )
+      )
+    )
+  )
+  (symbol (lib_id "power:+12VA") (at 232.41 41.91 0) (unit 1)
+    (in_bom yes) (on_board yes) (dnp no) (fields_autoplaced)
+    (property "Reference" "#PWR014" (at 232.41 45.72 0)
+      (effects (font (size 1.27 1.27)) hide)
+    )
+    (property "Value" "+12VA" (at 232.41 38.1 0)
+      (effects (font (size 1.27 1.27)))
+    )
+    (property "Footprint" "" (at 232.41 41.91 0)
+      (effects (font (size 1.27 1.27)) hide)
+    )
+    (property "Datasheet" "" (at 232.41 41.91 0)
+      (effects (font (size 1.27 1.27)) hide)
+    )
+    (pin "1")
+    (instances
+      (project "Module_2"
+        (path "/d9631a92-6a8d-4456-a627-6fb12cee70ca"
+          (reference "#PWR014") (unit 1)
+        )
+      )
+    )
+  )
   (symbol (lib_id "Device:R") (at 219.71 118.11 90) (unit 1)
     (in_bom yes) (on_board yes) (dnp no)
@@
         (path "/d9631a92-6a8d-4456-a627-6fb12cee70ca"
           (reference "C2") (unit 1)
+        )
+      )
+    )
+  )
+  (symbol (lib_id "power:GND") (at 186.69 80.01 0) (unit 1)
+    (in_bom yes) (on_board yes) (dnp no) (fields_autoplaced)
+    (property "Reference" "#PWR040" (at 186.69 86.36 0)
+      (effects (font (size 1.27 1.27)) hide)
+    )
+    (property "Value" "GND" (at 186.69 85.09 0)
+      (effects (font (size 1.27 1.27)))
+    )
+    (property "Footprint" "" (at 186.69 80.01 0)
+      (effects (font (size 1.27 1.27)) hide)
+    )
+    (property "Datasheet" "" (at 186.69 80.01 0)
+      (effects (font (size 1.27 1.27)) hide)
+    )
+    (pin "1")
+    (instances
+      (project "Module_2"
+        (path "/d9631a92-6a8d-4456-a627-6fb12cee70ca"
+          (reference "#PWR040") (unit 1)
         )
       )
@@
     )
   )
-  (symbol (lib_id "power:+5V") (at 55.88 137.16 0) (unit 1)
-    (in_bom yes) (on_board yes) (dnp no) (fields_autoplaced)
-    (property "Reference" "#PWR02" (at 55.88 140.97 0)
-      (effects (font (size 1.27 1.27)) hide)
-    )
-    (property "Value" "+5V" (at 55.88 133.35 0)
-      (effects (font (size 1.27 1.27)))
-    )
-    (property "Footprint" "" (at 55.88 137.16 0)
-      (effects (font (size 1.27 1.27)) hide)
-    )
-    (property "Datasheet" "" (at 55.88 137.16 0)
+  (symbol (lib_id "power:+5V") (at 55.88 127 0) (unit 1)
+    (in_bom yes) (on_board yes) (dnp no) (fields_autoplaced)
+    (property "Reference" "#PWR02" (at 55.88 130.81 0)
+      (effects (font (size 1.27 1.27)) hide)
+    )
+    (property "Value" "+5V" (at 55.88 123.19 0)
+      (effects (font (size 1.27 1.27)))
+    )
+    (property "Footprint" "" (at 55.88 127 0)
+      (effects (font (size 1.27 1.27)) hide)
+    )
+    (property "Datasheet" "" (at 55.88 127 0)
       (effects (font (size 1.27 1.27)) hide)
     )
@@
     )
   )
-  (symbol (lib_id "power:+12V") (at 232.41 41.91 0) (unit 1)
-    (in_bom yes) (on_board yes) (dnp no) (fields_autoplaced)
-    (property "Reference" "#PWR014" (at 232.41 45.72 0)
-      (effects (font (size 1.27 1.27)) hide)
-    )
-    (property "Value" "+12V" (at 232.41 38.1 0)
-      (effects (font (size 1.27 1.27)))
-    )
-    (property "Footprint" "" (at 232.41 41.91 0)
-      (effects (font (size 1.27 1.27)) hide)
-    )
-    (property "Datasheet" "" (at 232.41 41.91 0)
-      (effects (font (size 1.27 1.27)) hide)
-    )
-    (pin "1")
-    (instances
-      (project "Module_2"
-        (path "/d9631a92-6a8d-4456-a627-6fb12cee70ca"
-          (reference "#PWR014") (unit 1)
-        )
-      )
-    )
-  )
   (symbol (lib_id "Device:C_Small") (at 271.78 45.72 0) (unit 1)
     (in_bom yes) (on_board yes) (dnp no)
@@
         )
       )
+    )
+  )
+  (symbol (lib_id "Device:C_Small") (at 45.72 134.62 0) (unit 1)
+    (in_bom yes) (on_board yes) (dnp no)
+    (property "Reference" "C26" (at 44.4126 128.9064 0)
+      (effects (font (size 1.27 1.27)) (justify left))
+    )
+    (property "Value" "0,1uF" (at 44.2674 130.6979 0)
+      (effects (font (size 1.27 1.27)) (justify left))
+    )
+    (property "Footprint" "Resistor_SMD:R_1206_3216Metric" (at 45.72 134.62 0)
+      (effects (font (size 1.27 1.27)) hide)
+    )
+    (property "Datasheet" "~" (at 45.72 134.62 0)
+      (effects (font (size 1.27 1.27)) hide)
+    )
+    (property "Mfr. Part. No" "" (at 45.72 134.62 0)
+      (effects (font (size 1.27 1.27)) hide)
+    )
+    (pin "1")
+    (pin "2")
+    (instances
+      (project "Module_2"
+        (path "/d9631a92-6a8d-4456-a627-6fb12cee70ca"
+          (reference "C26") (unit 1)
+        )
+      )
+    )
+  )
+  (symbol (lib_id "Connector:Conn_01x03_Pin") (at 193.04 72.39 0) (mirror y) (unit 1)
+    (in_bom yes) (on_board yes) (dnp no)
+    (property "Reference" "J10" (at 192.405 66.04 0)
+      (effects (font (size 1.27 1.27)))
+    )
+    (property "Value" "Conn_01x03_Pin" (at 192.405 68.58 0)
+      (effects (font (size 1.27 1.27)) hide)
+    )
+    (property "Footprint" "Connector:FanPinHeader_1x03_P2.54mm_Vertical" (at 193.04 72.39 0)
+      (effects (font (size 1.27 1.27)) hide)
+    )
+    (property "Datasheet" "~" (at 193.04 72.39 0)
+      (effects (font (size 1.27 1.27)) hide)
+    )
+    (pin "1")
+    (pin "2")
+    (pin "3")
+    (instances
+      (project "Module_2"
+        (path "/d9631a92-6a8d-4456-a627-6fb12cee70ca"
+          (reference "J10") (unit 1)
+        )
+      )

Commit message: add bom module 1
Parts:
- C4: Mfr. Part. No T491B476M006AT -> (none)
- L1: Mfr. Part. No LB3218T101M -> (none)

Commit message: add bom and pos
Parts:
- C1, C2: LCSC (none) -> C577126; MFR.Part (none) -> CC1206JKNPODBN220
- C26, C6: footprint Resistor_SMD:R_1206_3216Metric -> Capacitor_SMD:C_1206_3216Metric; LCSC (none) -> C82601; MFR.Part (none) -> CC1206KRX7R9BB104
- C3, C7, C9: LCSC (none) -> C82601; MFR.Part (none) -> CC1206KRX7R9BB104
- C4: LCSC (none) -> C116617; MFR.Part (none) -> T491B476K010AT
- C5: LCSC (none) -> C145012; MFR.Part (none) -> CC1206KKX7R9BB684
- C8: LCSC (none) -> C469628; MFR.Part (none) -> CC1206JRNPOBBN100
- D1: LCSC (none) -> C3001646; MFR.Part (none) -> TLHG4400
- J1, J10, J2: LCSC (none) -> C5665; MFR.Part (none) -> C5665
- J3, J4: LCSC (none) -> C6332196; MFR.Part (none) -> HB-PH3-25413PB2GOP
- JP1: LCSC (none) -> C213465; MFR.Part (none) -> 54102-T0600LF
- L1: LCSC (none) -> C128802; MFR.Part (none) -> CMI321611J101KT
- Q1, Q2, Q3: LCSC (none) -> C2590; MFR.Part (none) -> IRLML2803TRPBF
- R1, R10, R12, R13, R2: LCSC (none) -> C134080; MFR.Part (none) -> RC1206JR-0756RL
- R11, R4, R7, R9: LCSC (none) -> C112223; MFR.Part (none) -> RC1206JR-071KL
- R3, R6: LCSC (none) -> C113307; MFR.Part (none) -> RC1206JR-07100RL
- R5: LCSC (none) -> C136458; MFR.Part (none) -> RC1206JR-074K7L
- R8: LCSC (none) -> C137179; MFR.Part (none) -> RC1206JR-0720KL
- U1: LCSC (none) -> C494990; MFR.Part (none) -> ADM1485ARZ-REEL
- U2: LCSC (none) -> C8736; MFR.Part (none) -> STM8S105K4T6C
- U3: LCSC (none) -> C2833074; MFR.Part (none) -> PC817X2YSZW
- Y1: LCSC (none) -> C295075; MFR.Part (none) -> XIHCELNANF-16MHZ

Commit message: change on 25_02_24
Parts:
- C1, C2, C26, C3, C4, C5, C6, C7, C8, C9, D1, L1, Q1, Q2, Q3, R1, R10, R12, R13, R2, R3, R5, R6, R8, U1, U2, U3, Y1: Mounting (none) -> Yes
- H1, H2, H3, H4: Mounting (none) -> No
- J1, J10, J2: LCSC C5665 -> C49257; MFR.Part C5665 -> HB-PH3-25413PB2GOP; Mounting (none) -> Yes
- J3, J4: LCSC C6332196 -> C5665; MFR.Part HB-PH3-25413PB2GOP -> C5665; Mounting (none) -> Yes
- JP1: LCSC C213465 -> C492401; MFR.Part 54102-T0600LF -> PZ254V-11-02P; Mounting (none) -> Yes
- R11, R4, R7, R9: LCSC C112223 -> C4410; MFR.Part RC1206JR-071KL -> 1206W4F1001T5E; Mounting (none) -> Yes
