File: Projects/StationModules/Module_2/Module_2.kicad_sch (KiCad schematic)
At the start: 42 parts, among them J1 Conn_01x03_Pin, J10 Conn_01x03_Pin, J2 Conn_01x03_Pin, Q1 IRLML2803, Q2 IRLML2803, Q3 IRLML2803, U1 ADM1485AR, U2 STM8S105K4T6C, U3 PC817, Y1 16MHz

Commit message: Corection all modules
Parts:
- J10: LCSC C49257 -> (none); Mounting Yes -> No
- J2: LCSC C49257 -> C29275; MFR.Part HB-PH3-25413PB2GOP -> 2510-3A
Connections:
- net GND: now also J10.1 (Pin_1), J2.1 (Pin_1); no longer J10.3 (Pin_3), J2.3 (Pin_3)
- net TX: now also J10.3 (Pin_3); no longer J10.1 (Pin_1)
- net at R2.2, R3.1: now also J2.3 (Pin_3); no longer J2.1 (Pin_1)
Other:
- moved on the sheet: J10, J2
Changed lines of the file:
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@@
     )
   )
-  (symbol (lib_id "Connector:Conn_01x03_Pin") (at 120.65 148.59 0) (mirror y) (unit 1)
-    (in_bom yes) (on_board yes) (dnp no)
-    (property "Reference" "J2" (at 120.015 142.24 0)
-      (effects (font (size 1.27 1.27)))
-    )
-    (property "Value" "Conn_01x03_Pin" (at 120.015 144.78 0)
+  (symbol (lib_id "Connector:Conn_01x03_Pin") (at 120.65 148.59 180) (unit 1)
+    (in_bom yes) (on_board yes) (dnp no)
+    (property "Reference" "J2" (at 120.015 154.94 0)
+      (effects (font (size 1.27 1.27)))
+    )
+    (property "Value" "Conn_01x03_Pin" (at 120.015 152.4 0)
       (effects (font (size 1.27 1.27)) hide)
     )
@@
       (effects (font (size 1.27 1.27)) hide)
     )
-    (property "MFR.Part" "HB-PH3-25413PB2GOP" (at 120.65 148.59 0)
-      (effects (font (size 1.27 1.27)) hide)
-    )
-    (property "Description" "Gold 250V 3A Straight Square Pins 2.54mm 3P 260℃ 6mm -40℃~+105℃ 3mm 2.54mm Brass Black Plugin 2.54mm 1x3P Plugin,P=2.54mm Pin Headers ROHS" (at 120.65 148.59 0)
-      (effects (font (size 1.27 1.27)) hide)
-    )
-    (property "LCSC" "C49257" (at 120.65 148.59 0)
+    (property "MFR.Part" "2510-3A" (at 120.65 148.59 0)
+      (effects (font (size 1.27 1.27)) hide)
+    )
+    (property "Description" "1x3P 3P 1 2.54mm 3 Plugin,P=2.54mm Wire To Board / Wire To Wire Connector ROHS" (at 120.65 148.59 0)
+      (effects (font (size 1.27 1.27)) hide)
+    )
+    (property "LCSC" "C29275" (at 120.65 148.59 0)
       (effects (font (size 1.27 1.27)) hide)
     )
@@
     )
   )
-  (symbol (lib_id "Connector:Conn_01x03_Pin") (at 193.04 72.39 0) (mirror y) (unit 1)
-    (in_bom yes) (on_board yes) (dnp no)
-    (property "Reference" "J10" (at 192.405 66.04 0)
-      (effects (font (size 1.27 1.27)))
-    )
-    (property "Value" "Conn_01x03_Pin" (at 192.405 68.58 0)
+  (symbol (lib_id "Connector:Conn_01x03_Pin") (at 193.04 72.39 180) (unit 1)
+    (in_bom yes) (on_board yes) (dnp no)
+    (property "Reference" "J10" (at 192.405 78.74 0)
+      (effects (font (size 1.27 1.27)))
+    )
+    (property "Value" "Conn_01x03_Pin" (at 192.405 76.2 0)
       (effects (font (size 1.27 1.27)) hide)
     )
@@
       (effects (font (size 1.27 1.27)) hide)
     )
-    (property "LCSC" "C49257" (at 193.04 72.39 0)
-      (effects (font (size 1.27 1.27)) hide)
-    )
-    (property "Mounting" "Yes" (at 193.04 72.39 0)
-      (effects (font (size 1.27 1.27)) hide)
-    )
+    (property "LCSC" "" (at 193.04 72.39 0)
+      (effects (font (size 1.27 1.27)) hide)
+    )
+    (property "Mounting" "No" (at 193.04 72.39 0)
+      (effects (font (size 1.27 1.27)) hide)
+    )
