File: Projects/StationModules/Module_2/Module_2.kicad_pcb (KiCad board)
At the start: 2 copper layers, 125.8 x 114.3 mm, 98 parts, among them J1 Conn_01x03_Pin, J12 Screw_Terminal_01x01, J13 Screw_Terminal_01x01, J14 Screw_Terminal_01x01, J15 Screw_Terminal_01x01, J18 Screw_Terminal_01x03, J2 Conn_01x03_Pin, J5 I, J6 U, J7 GND, J9 Screw_Terminal_01x02, Q1 IRLML2803, Q2 IRLML2803, Q3 IRLML2803, U1 ADM1485AR, U2 STM8S105K4T6C, U3 PC817, U4 LM2904, U5 LM358, Y1 16MHz

Commit message: module 2 board complit v1
Parts:
- added C26: 0,1uF, Resistor_SMD:R_1206_3216Metric, B.Cu at (52.8, 127.7)
- added J10: Conn_01x03_Pin, Connector:FanPinHeader_1x03_P2.54mm_Vertical, F.Cu at (47.8, 123.7)
- added L3: 220uH THT, Inductor_THT:L_Axial_L7.0mm_D3.3mm_P10.16mm_Horizontal_Fastron_MICC, F.Cu at (47.0, 95.5)
- L2: value 220uH -> 220uH SMD
- moved C16 64.9 mm to (131.0, 110.2), turned to 180 degrees
- moved C14 47.9 mm to (102.4, 104.3)
- moved J5 18.9 mm to (116.3, 87.9)
- moved C12 15.9 mm to (78.2, 94.6)
- moved R16 13.0 mm to (121.9, 89.9), turned to 0 degrees
- moved C11 12.2 mm to (62.2, 94.6)
- moved R6 10.1 mm to (129.0, 125.8)
- moved C8 10.1 mm to (126.5, 125.8)
- moved U3 8.08 mm to (119.1, 127.8)
- moved R33 7.11 mm to (119.9, 71.9)
- moved R31 7.11 mm to (119.9, 82.2)
- moved R32 7.11 mm to (119.9, 77.0)
- moved R34 7.11 mm to (119.9, 66.8)
- moved R35 7.11 mm to (119.9, 61.7)
- moved J18 6.44 mm to (43.1, 42.0)
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Connections:
- J4 pad 2: +12V -> +12VA
- J8 pad 1: Net-(J8-Pad1) -> +12VA
- J8 pad 2: Net-(J8-Pad1) -> +12VA
- L2 pad 1: Net-(J8-Pad1) -> +12VA
Routing:
- net +5V: track 0.00 -> 268.3 mm, vias 0 -> 8
- net +12V: track 0.00 -> 149.3 mm
- net /sheet_2/F_IN: track 0.00 -> 113.1 mm, vias 0 -> 1
- net +12VA: track 0.00 -> 105.4 mm, vias 0 -> 2
- net I_IN: track 0.00 -> 67.5 mm, vias 0 -> 2
- net /RX: track 0.00 -> 60.4 mm, vias 0 -> 2
- net Net-(U5A-+): track 0.00 -> 57.9 mm, vias 0 -> 2
- net PWM: track 0.00 -> 53.8 mm, vias 0 -> 2
- net FI: track 0.00 -> 53.6 mm, vias 0 -> 2
- net /TX: track 0.00 -> 52.7 mm
- net U_SET: track 0.00 -> 46.6 mm, vias 0 -> 2
- net /OUT_1: track 0.00 -> 43.5 mm, vias 0 -> 2
- net /IN_1: track 0.00 -> 42.3 mm, vias 0 -> 2
- net /DIR: track 0.00 -> 41.9 mm
- net OS: track 0.00 -> 41.9 mm, vias 0 -> 2
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- added copper zone on F.Cu, net GND
- added copper zone on F.Cu, net I
- added copper zone on F.Cu, net Net-(D6-A)
- added copper zone on F.Cu, net Net-(J13-Pin_1)
- added copper zone on F.Cu, net Net-(J18-Pin_1)
- added copper zone on F.Cu, net Net-(J18-Pin_2)
Other:
- board size 125.8 x 114.3 mm -> 125.8 x 114.8 mm
- board text added: "RS485"
- board text added: "RX/TX"
- board text added: "Дисплей"
- board text added: "Качалка"
- board text added: "Питание"

Commit message: finaly on summer
Parts:
- C16: value 0,1uf -> 0,1uF
- C23: value C -> 4n7; footprint Capacitor_THT:C_Rect_L7.0mm_W2.0mm_P5.00mm -> Capacitor_THT:C_Rect_L11.5mm_W5.2mm_P10.00mm_MKT
- C24, C25: value C -> 10uF
- C26, C6: footprint Resistor_SMD:R_1206_3216Metric -> Capacitor_SMD:C_1206_3216Metric
- R27, R28: value R 2W -> 20
- R29, R30: value R -> 22k
- RV2: value 4k7 3296W -> 5k
Routing:
- net Net-(J18-Pin_2): track 18.8 -> 21.8 mm
Other:
- board text added: "1"

Commit message: change module1,2
Parts:
- removed J14, J15: Screw_Terminal_01x01, Z_pin:PinD3mm
- removed R35: 0,01, Resistor_SMD:R_2816_7142Metric
- added H2: MountingHole, MountingHole:MountingHole_3.5mm, F.Cu at (100.8, 39.1)
- added H2: MountingHole, MountingHole:MountingHole_3.5mm, F.Cu at (80.8, 39.1)
- R18: value 10 -> 0
- R19: value 200k -> 330k
- R20: value 10k -> 39k
- R27, R28: value 20 -> 120
- moved C24 44.0 mm to (149.4, 55.9), turned to 180 degrees
- moved J12 33.6 mm to (108.5, 51.1)
- moved RV2 28.5 mm to (157.7, 49.8), turned to 90 degrees
- moved R30 27.1 mm to (157.7, 45.7)
- moved R29 26.6 mm to (157.7, 42.9)
- moved R14 22.4 mm to (154.2, 61.0), turned to -90 degrees
- moved J6 22.1 mm to (158.5, 61.2)
- moved C25 22.1 mm to (149.4, 39.6), turned to 180 degrees
- moved J9 17.6 mm to (160.5, 74.4)
- moved J13 16.5 mm to (113.0, 34.5)
- moved J7 11.0 mm to (157.0, 87.6)
Routing:
- net GND: track 24.7 -> 48.4 mm
- net U_IN: track 74.8 -> 96.7 mm
- net Net-(J13-Pin_1): track 26.5 -> 8.29 mm
- net U: track 9.27 -> 14.9 mm
- net Net-(R30-Pad2): track 5.93 -> 4.67 mm

Commit message: change on 25_02_24
Parts:
- moved C25 50.3 mm to (99.1, 38.1)
- moved J13 36.8 mm to (146.1, 50.8)
- moved H2 36.1 mm to (136.9, 38.6)
- moved H2 36.1 mm to (116.8, 38.6)
- moved C24 17.9 mm to (135.7, 67.3)
- moved J12 0.25 mm to (108.5, 50.8)
Routing:
- net I: track 36.7 -> 62.2 mm, vias 10 -> 9
- net Net-(J13-Pin_1): track 8.29 -> 17.6 mm
Other:
- board text added: "+"
- board text added: "-"
- board text added: "Общий"
- board text added: "Фаза1"
- board text added: "Фаза2"
Changed lines of the file:
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@@
     (pad_to_mask_clearance 0)
     (pcbplotparams
-      (layerselection 0x0001000_7ffffffe)
-      (plot_on_all_layers_selection 0x00210a8_00000001)
+      (layerselection 0x00010fc_ffffffff)
+      (plot_on_all_layers_selection 0x0000000_00000000)
       (disableapertmacros false)
       (usegerberextensions true)
@@
       (sketchpadsonfab false)
       (subtractmaskfromsilk true)
-      (outputformat 4)
+      (outputformat 1)
       (mirror false)
       (drillshape 0)
       (scaleselection 1)
-      (outputdirectory "Docs/Top/")
+      (outputdirectory "Module_2_gerbers/")
     )
   )
@@
   )
   (footprint "MountingHole:MountingHole_3.5mm" (layer "F.Cu")
-    (at 100.838 39.116)
+    (at 136.906 38.608)
     (descr "Mounting Hole 3.5mm, no annular")
     (tags "mounting hole 3.5mm no annular")
@@
     (property "ki_description" "Mounting Hole without connection")
     (property "ki_keywords" "mounting hole")
+    (clearance 2)
     (attr exclude_from_pos_files)
     (fp_text reference "H2" (at 0 -4.5) (layer "F.SilkS") hide
@@
     (property "ki_keywords" "screw terminal")
     (attr through_hole)
-    (fp_text reference "J18" (at 4.953 32.9295 unlocked) (layer "F.SilkS")
+    (fp_text reference "J18" (at 20.955 32.6755 unlocked) (layer "F.SilkS")
         (effects (font (size 1 1) (thickness 0.1)))
     )
@@
   )
   (footprint "MountingHole:MountingHole_3.5mm" (layer "F.Cu")
-    (at 80.772 39.116)
+    (at 116.84 38.608)
     (descr "Mounting Hole 3.5mm, no annular")
     (tags "mounting hole 3.5mm no annular")
@@
     (property "ki_description" "Mounting Hole without connection")
     (property "ki_keywords" "mounting hole")
+    (clearance 2)
     (attr exclude_from_pos_files)
     (fp_text reference "H2" (at 0 -4.5) (layer "F.SilkS") hide
@@
   )
   (footprint "Capacitor_THT:C_Rect_L31.5mm_W15.0mm_P27.50mm_MKS4" (layer "F.Cu")
-    (at 149.386 55.88 180)
+    (at 135.67 67.31 180)
     (descr "C, Rect series, Radial, pin pitch=27.50mm, , length*width=31.5*15mm^2, Capacitor, http://www.wima.com/EN/WIMA_MKS_4.pdf")
     (tags "C Rect series Radial pin pitch 27.50mm  length 31.5mm width 15mm Capacitor")
@@
     (property "ki_keywords" "capacitor cap")
     (attr through_hole)
-    (fp_text reference "C24" (at 12.988 0) (layer "F.SilkS")
+    (fp_text reference "C24" (at 1.558 2.54) (layer "F.SilkS")
         (effects (font (size 1 1) (thickness 0.15)))
     )
@@
   )
   (footprint "Z_pin:PinD3mm" (layer "F.Cu")
-    (at 108.458 51.054)
+    (at 108.458 50.8)
     (property "Description" "")
     (property "LCSC" "")
@@
   )
   (footprint "Capacitor_THT:C_Rect_L31.5mm_W15.0mm_P27.50mm_MKS4" (layer "F.Cu")
-    (at 149.352 39.624 180)
+    (at 99.06 38.1 180)
     (descr "C, Rect series, Radial, pin pitch=27.50mm, , length*width=31.5*15mm^2, Capacitor, http://www.wima.com/EN/WIMA_MKS_4.pdf")
     (tags "C Rect series Radial pin pitch 27.50mm  length 31.5mm width 15mm Capacitor")
@@
     (property "ki_keywords" "capacitor cap")
     (attr through_hole)
-    (fp_text reference "C25" (at 13.462 0.508) (layer "F.SilkS")
+    (fp_text reference "C25" (at 13.716 -0.254) (layer "F.SilkS")
         (effects (font (size 1 1) (thickness 0.15)))
     )
@@
   )
   (footprint "Z_pin:PinD3mm" (layer "F.Cu")
-    (at 113.03 34.544)
+    (at 146.05 50.8)
     (property "Description" "")
     (property "LCSC" "")
@@
     (property "ki_keywords" "R res resistor")
     (attr smd)
-    (fp_text reference "R33" (at -9.890645 -5.029858 90) (layer "B.SilkS")
+    (fp_text reference "R33" (at -7.3935 0 90) (layer "B.SilkS")
         (effects (font (size 1 1) (thickness 0.15)) (justify mirror))
     )
@@
     )
   )
-  (gr_line (start 110.982907 67.505359) (end 115.163496 70.640801)
-    (stroke (width 0.15) (type default)) (layer "B.SilkS"))
   (gr_line (start 139.540613 115.954239) (end 139.575451 117.812279)
     (stroke (width 0.15) (type default)) (layer "B.SilkS"))
-  (gr_rect (start 75.692 30.988) (end 105.918 43.434)
+  (gr_line (start 115.062 50.8) (end 112.014 50.8)
+    (stroke (width 0.15) (type default)) (layer "F.SilkS"))
+  (gr_arc (start 115.062 50.8) (mid 118.11 47.752) (end 121.158 50.8)
+    (stroke (width 0.15) (type default)) (layer "F.SilkS"))
+  (gr_rect (start 111.76 30.48) (end 141.986 42.926)
+    (stroke (width 0.15) (type default)) (fill none) (layer "F.SilkS"))
+  (gr_arc (start 121.158 50.8) (mid 124.206 47.752) (end 127.254 50.8)
+    (stroke (width 0.15) (type default)) (layer "F.SilkS"))
+  (gr_arc (start 127.254 50.8) (mid 130.302 47.752) (end 133.35 50.8)
+    (stroke (width 0.15) (type default)) (layer "F.SilkS"))
+  (gr_line (start 139.446 50.546) (end 142.494 50.546)
+    (stroke (width 0.15) (type default)) (layer "F.SilkS"))
+  (gr_arc (start 133.35 50.546) (mid 136.398 47.498) (end 139.446 50.546)
+    (stroke (width 0.15) (type default)) (layer "F.SilkS"))
+  (gr_rect (start 101.6 30.48) (end 152.4 58.42)
     (stroke (width 0.15) (type default)) (fill none) (layer "F.SilkS"))
   (gr_rect (start 40.6146 30.28) (end 166.37 145.088)
@@
     (effects (font (size 2 2) (thickness 0.3)) (justify left bottom))
   )
+  (gr_text "Фаза1" (at 53.848 36.322) (layer "F.SilkS")
+    (effects (font (size 3 3) (thickness 0.2)) (justify left bottom))
+  )
+  (gr_text "+" (at 160.782 63.246) (layer "F.SilkS")
+    (effects (font (size 5 5) (thickness 0.5)) (justify left bottom))
+  )
+  (gr_text "Общий" (at 42.926 76.708) (layer "F.SilkS")
+    (effects (font (size 3 3) (thickness 0.2)) (justify left bottom))
+  )
   (gr_text "RS485" (at 55.418512 134.836879) (layer "F.SilkS")
     (effects (font (size 2 2) (thickness 0.3)) (justify left bottom))
   )
+  (gr_text "-" (at 166.116 91.186 90) (layer "F.SilkS")
+    (effects (font (size 5 5) (thickness 0.5)) (justify left bottom))
+  )
+  (gr_text "Фаза2" (at 53.848 41.402) (layer "F.SilkS")
+    (effects (font (size 3 3) (thickness 0.2)) (justify left bottom))
+  )
   (segment (start 133.604 135.128) (end 121.285 135.128) (width 1) (layer "F.Cu") (net 1))
   (segment (start 136.487884 132.244116) (end 133.604 135.128) (width 1) (layer "F.Cu") (net 1))
@@
   (segment (start 71.12 67.31) (end 79.375 67.31) (width 2) (layer "B.Cu") (net 19))
   (segment (start 79.375 67.31) (end 83.86 67.31) (width 2) (layer "B.Cu") (net 19))
+  (segment (start 142.113 67.31) (end 144.145 69.342) (width 3) (layer "B.Cu") (net 20))
   (segment (start 149.352 39.624) (end 152.654 42.926) (width 0.75) (layer "B.Cu") (net 20))
   (segment (start 152.654 42.926) (end 156.2715 42.926) (width 0.75) (layer "B.Cu") (net 20))
-  (segment (start 117.06 60.706) (end 115.316 60.706) (width 3) (layer "F.Cu") (net 21))
-  (segment (start 121.852 55.846) (end 121.886 55.88) (width 3) (layer "F.Cu") (net 21))
-  (segment (start 121.852 39.624) (end 121.852 55.846) (width 3) (layer "F.Cu") (net 21))
-  (segment (start 121.886 55.88) (end 117.06 60.706) (width 3) (layer "F.Cu") (net 21))
+  (segment (start 135.67 67.31) (end 142.113 67.31) (width 3) (layer "B.Cu") (net 20))
   (via (at 114.3 81.28) (size 1.2) (drill 0.5) (layers "F.Cu" "B.Cu") (free) (net 21))
   (via (at 114.3 76.2) (size 1.2) (drill 0.5) (layers "F.Cu" "B.Cu") (free) (net 21))
   (via (at 114.3 66.04) (size 1.2) (drill 0.5) (layers "F.Cu" "B.Cu") (free) (net 21))
-  (via (at 114.3 60.96) (size 1.2) (drill 0.5) (layers "F.Cu" "B.Cu") (free) (net 21))
   (via (at 114.3 63.5) (size 1.2) (drill 0.5) (layers "F.Cu" "B.Cu") (free) (net 21))
   (via (at 114.3 71.12) (size 1.2) (drill 0.5) (layers "F.Cu" "B.Cu") (free) (net 21))
@@
   (via (at 114.3 73.66) (size 1.2) (drill 0.5) (layers "F.Cu" "B.Cu") (free) (net 21))
   (via (at 114.3 83.82) (size 1.2) (drill 0.5) (layers "F.Cu" "B.Cu") (free) (net 21))
+  (segment (start 59.0185 67.4005) (end 55.88 64.262) (width 3) (layer "B.Cu") (net 21))
   (segment (start 116.332 87.884) (end 116.332 89.154) (width 0.75) (layer "B.Cu") (net 21))
+  (segment (start 59.182 38.1) (end 71.56 38.1) (width 3) (layer "B.Cu") (net 21))
   (segment (start 117.3755 82.242) (end 117.148 82.242) (width 0.75) (layer "B.Cu") (net 21))
   (segment (start 116.332 89.154) (end 117.094 89.916) (width 0.75) (layer "B.Cu") (net 21))
+  (segment (start 55.88 41.402) (end 59.182 38.1) (width 3) (layer "B.Cu") (net 21))
+  (segment (start 65.024 67.4005) (end 59.0185 67.4005) (width 3) (layer "B.Cu") (net 21))
   (segment (start 117.148 82.242) (end 116.332 83.058) (width 0.75) (layer "B.Cu") (net 21))
+  (segment (start 55.88 64.262) (end 55.88 41.402) (width 3) (layer "B.Cu") (net 21))
   (segment (start 116.332 83.058) (end 116.332 87.884) (width 0.75) (layer "B.Cu") (net 21))
   (segment (start 117.094 89.916) (end 120.396 89.916) (width 0.75) (layer "B.Cu") (net 21))
@@
         (xy 69.596 70.866)
         (xy 101.854 70.866)
-        (xy 109.22 62.484)
-        (xy 112.268 58.674)
-        (xy 118.618 58.674)
-        (xy 118.872 58.928)
+        (xy 109.22 62.23)
+        (xy 112.268 62.23)
+        (xy 118.11 62.23)
+        (xy 118.872 63.5)
         (xy 118.872 84.328)
         (xy 117.602 85.09)
@@
       (pts
         (xy 120.904 63.5)
-        (xy 121.92 62.484)
-        (xy 129.54 62.484)
+        (xy 121.92 62.23)
+        (xy 129.54 62.23)
         (xy 135.89 76.2)
         (xy 151.638 76.2)
@@
         (xy 141.224 52.832)
         (xy 137.16 48.514)
-        (xy 125.73 36.576)
-        (xy 118.11 36.576)
-        (xy 117.095599 38.1)
-        (xy 109.474 38.1)
-        (xy 109.474 30.988)
+        (xy 131.064 42.926)
+        (xy 95.25 42.926)
+        (xy 95.25 30.988)
       )
     )
   )
-  (group "" (id 4cb24642-d5fa-4a84-bc99-66412e2c01cb)
-    (members
-      1d3c9f4e-f9eb-4d95-bb7d-76ce5effcaef
-      6e7351f5-a9bf-41f6-a3cb-9ddfbf881a5c
-      9759d2a3-4125-42a3-8779-c6c24938409c
-    )
-  )

Commit message: Corection all modules
Parts:
- added D7: 1.5KExxA, Diode_THT:D_DO-201AE_P15.24mm_Horizontal, F.Cu at (140.5, 65.4)
- moved J2 92.1 mm to (149.9, 138.7), turned to 180 degrees
- moved JP1 10.8 mm to (61.0, 135.3), turned to -90 degrees
- moved J10 5.08 mm to (47.8, 128.8), turned to 90 degrees
- moved R3 2.15 mm to (64.1, 129.0), turned to -90 degrees
- moved J9 1.91 mm to (162.4, 74.4)
Connections:
- J10 pad 1: /TX -> GND
- J10 pad 3: GND -> /TX
- J2 pad 1: Net-(J2-Pin_1) -> GND
- J2 pad 3: GND -> Net-(J2-Pin_3)
- R2 pad 2: Net-(J2-Pin_1) -> Net-(J2-Pin_3)
- R3 pad 1: Net-(J2-Pin_1) -> Net-(J2-Pin_3)
Routing:
- net Net-(J2-Pin_3): track 0.00 -> 101.6 mm
- net Net-(J2-Pin_2): track 39.2 -> 101.7 mm
- net Net-(J2-Pin_1): track 14.8 -> 0.00 mm
- net Net-(JP1-A): track 4.61 -> 6.88 mm
- net GND: vias 140 -> 124
Other:
- board text removed: "RX/TX"

Commit message: change for final 20.03.2024
Other:
- board text added: "Телеметрия"
- board text removed: "RS485"
