File: Projects/StationModules/Module_3/Module_3.kicad_pcb (KiCad board)
At the start: 2 copper layers, 186.7 x 90.2 mm, 31 parts, among them J1 Screw_Terminal_01x03, J2 Screw_Terminal_01x02, J4 Screw_Terminal_01x02, U1 LM2576S-5, U2 PC814

Commit message: module 3, route complit 2
Parts:
- added J5: Screw_Terminal_01x01, Z_pin:PinD4mm, F.Cu at (222.2, 62.2)
- added J6: Screw_Terminal_01x01, Z_pin:PinD4mm, F.Cu at (222.2, 80.0)
- added J7: Screw_Terminal_01x01, Z_pin:PinD1_6mm, F.Cu at (209.6, 125.7)
- J1: footprint Z_connectors:DG135T-10.16-03P -> Z_connectors:DB129V-7.62-3P-GN-S
- J2: footprint Z_connectors:DG135T-10.16-02P -> Z_connectors:DB129V-7.62-2P-GN-S
- J4: value Screw_Terminal_01x02 -> Screw_Terminal_01x01; footprint Z_connectors:DG135T-10.16-02P -> Z_pin:PinD1_6mm
- moved J4 54.5 mm to (203.2, 125.7)
- moved J2 11.8 mm to (184.2, 125.2)
- moved J1 4.93 mm to (58.4, 64.8)
- moved C7 4.22 mm to (178.4, 112.7)
- moved C2 2.54 mm to (74.9, 83.9)
Connections:
- J4 pad 1: Net-(D2-+) -> +12V
Routing:
- net +12V: track 167.4 -> 175.6 mm
- net Net-(D2--): track 65.4 -> 59.2 mm
- net Net-(D2-+): track 63.9 -> 57.9 mm
- net /F_IN: track 45.7 -> 50.7 mm
- net Net-(J1-Pin_2): track 89.4 -> 85.2 mm
- net Net-(J1-Pin_3): track 175.4 -> 172.2 mm
- net +5V: track 74.5 -> 76.8 mm
- net Net-(J1-Pin_1): track 94.7 -> 92.4 mm
- net GND: vias 31 -> 27
Other:
- board text added: "+12V"
- board text added: "+300V"
- board text added: "-300V"
- board text added: "Earth"
- board text added: "GND"
- board text added: "L"
- board text added: "N"
- board text added: "Potencial_In"
- board text removed: "+"
- board text removed: "-"
- board text removed: "Out 300V"
- board text removed: "Potencial"

Commit message: change on 25_02_24
Parts:
- added C10: 0.1uF, Capacitor_SMD:C_1206_3216Metric, F.Cu at (107.3, 130.0)
- added R5: 1M, Resistor_SMD:R_1206_3216Metric, F.Cu at (109.9, 130.0)
- added R6: 330k, Resistor_SMD:R_1206_3216Metric, F.Cu at (206.4, 65.8)
- added R7: 330k, Resistor_SMD:R_1206_3216Metric, F.Cu at (206.4, 71.1)
- added R8: 330k, Resistor_SMD:R_1206_3216Metric, F.Cu at (206.4, 76.2)
- F1: footprint Fuse:Fuseholder_Clip-5x20mm_Keystone_3517_Inline_P23.11x6.76mm_D1.70mm_Horizontal -> Fuse:Fuse_Littelfuse_395Series
- J5, J6: footprint Z_pin:PinD4mm -> Z_pin:PinD3mm
- moved M1 107.5 mm to (175.9, 94.6), turned to -90 degrees
- moved J4 88.8 mm to (114.9, 135.1), turned to 0 degrees
- moved J7 87.5 mm to (122.6, 135.1), turned to 180 degrees
- moved J2 86.4 mm to (97.8, 127.0), turned to 0 degrees
- moved F1 85.1 mm to (140.7, 111.3), turned to 0 degrees
- moved L1 63.3 mm to (147.1, 106.4), turned to 180 degrees
- moved C2 60.6 mm to (127.5, 114.0), turned to 180 degrees
- moved L3 46.3 mm to (212.7, 123.2)
- moved D1 43.3 mm to (194.1, 121.9)
- moved J3 43.2 mm to (188.0, 134.6), turned to 90 degrees
- moved C1 37.3 mm to (187.3, 110.8)
- moved C7 35.6 mm to (214.0, 110.8)
- moved C3 35.1 mm to (90.2, 104.4)
- moved U1 34.1 mm to (199.8, 107.0)
- moved J1 32.5 mm to (90.2, 57.8)
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Connections:
- F1 pad 1: Net-(J1-Pin_1) -> Net-(C3-Pad1)
- L2 pad 3: Net-(C4-Pad2) -> Net-(C4-Pad1)
- L2 pad 4: Net-(C4-Pad1) -> Net-(C4-Pad2)
- M1 pad 1: Net-(J1-Pin_2) -> Net-(F1-Pad2)
- M1 pad 2: Net-(F1-Pad2) -> Net-(C3-Pad2)
- M1 pad 3: GND -> +12V
- M1 pad 4: +12V -> GND
Routing:
- net GND: track 0.00 -> 168.2 mm, vias 27 -> 31
- net /F_IN: track 50.7 -> 130.4 mm
- net Net-(C3-Pad1): track 38.4 -> 112.2 mm
- net Net-(J1-Pin_3): track 172.2 -> 107.7 mm
- net Net-(C3-Pad2): track 38.3 -> 102.3 mm
- net +12V: track 175.6 -> 118.2 mm, vias 0 -> 1
- net Net-(C4-Pad1): track 44.9 -> 93.6 mm
- net Net-(J1-Pin_2): track 85.2 -> 96.8 mm
- net Net-(C4-Pad2): track 96.8 -> 85.7 mm
- net +5V: track 76.8 -> 66.5 mm
- net Net-(D2--): track 59.2 -> 67.5 mm
- net Net-(D2-+): track 57.9 -> 65.5 mm
- net Net-(J1-Pin_1): track 92.4 -> 99.6 mm
- net Net-(F1-Pad2): track 40.2 -> 34.5 mm
- net /U_SET: track 45.4 -> 40.4 mm
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Other:
- board size 186.7 x 90.2 mm -> 143.6 x 94 mm
- board text added: "Pot.max5V"
- board text removed: "Potencial_In"

Commit message: Corection all modules
Parts:
- added D3: 1.5KExxCA, Diode_THT:D_DO-201AE_P15.24mm_Horizontal, F.Cu at (92.8, 102.5)
- added F2: Fuse, Resistor_THT:R_Axial_Power_L20.0mm_W6.4mm_P25.40mm, F.Cu at (102.2, 51.2)
- added PS1: HLK-PM12, Converter_ACDC:Converter_ACDC_HiLink_HLK-5Mxx, F.Cu at (168.1, 100.6)
- added RV1: Varistor, Varistor:RV_Disc_D21.5mm_W4.3mm_P10mm, F.Cu at (109.6, 69.1)
- C2, C3, C4: value 470nF -> 1uF; footprint Capacitor_THT:C_Rect_L24.0mm_W10.9mm_P22.50mm_MKT -> Capacitor_THT:C_Rect_L18.0mm_W11.0mm_P15.00mm_FKS3_FKP3
- L1, L2: footprint Z_inductors:B82726S6123N020 -> Z_inductors:FilterSetevoy_20x30_p20
- moved C3 28.2 mm to (107.4, 82.2), turned to -90 degrees
- moved C2 7.67 mm to (120.3, 111.5), turned to 0 degrees
- moved L1 6.55 mm to (143.3, 101.1)
- moved L2 4.80 mm to (143.3, 72.4)
- moved C4 3.78 mm to (158.8, 80.1)
- moved F1 2.57 mm to (143.3, 110.9)
Connections:
- C2 pad 1: Net-(J1-Pin_2) -> Net-(D3-A1)
- C2 pad 2: Net-(J1-Pin_1) -> Net-(D3-A2)
- C4 pad 2: Net-(C4-Pad2) -> Net-(PS1-AC/N)
- C6 pad 2: Net-(C4-Pad2) -> Net-(PS1-AC/N)
- D2 pad 3: Net-(C4-Pad2) -> Net-(PS1-AC/N)
- F1 pad 1: Net-(C3-Pad1) -> Net-(C4-Pad1)
- J1 pad 2: Net-(J1-Pin_2) -> Net-(D3-A2)
- L1 pad 1: Net-(J1-Pin_2) -> Net-(D3-A1)
- L1 pad 2: Net-(J1-Pin_1) -> Net-(D3-A2)
- L2 pad 3: Net-(C4-Pad1) -> Net-(PS1-AC/N)
- L2 pad 4: Net-(C4-Pad2) -> Net-(C4-Pad1)
- M1 pad 2: Net-(C3-Pad2) -> Net-(PS1-AC/N)
- R2 pad 1: Net-(C4-Pad2) -> Net-(PS1-AC/N)
Routing:
- net Net-(PS1-AC/N): track 0.00 -> 126.1 mm
- net Net-(D3-A2): track 0.00 -> 117.8 mm
- net Net-(D3-A1): track 0.00 -> 97.3 mm
- net Net-(J1-Pin_2): track 96.8 -> 0.00 mm
- net Net-(C3-Pad1): track 112.2 -> 24.5 mm
- net Net-(C4-Pad2): track 85.7 -> 0.00 mm
- net Net-(J1-Pin_1): track 99.6 -> 14.8 mm
- net Net-(C3-Pad2): track 102.3 -> 52.8 mm
- net Net-(C4-Pad1): track 93.6 -> 110.0 mm
- net Net-(J1-Pin_3): track 107.7 -> 116.4 mm
- net +12V: track 118.2 -> 121.5 mm
- net GND: track 168.2 -> 169.5 mm
