File: Projects/StationModules/Module_3/Module_3.kicad_sch (KiCad schematic)
At the start: 31 parts, among them J1 Screw_Terminal_01x03, J2 Screw_Terminal_01x02, J4 Screw_Terminal_01x02, U1 LM2576S-5, U2 PC814

Commit message: module 3, route complit 2
Parts:
- removed J4: Screw_Terminal_01x02, Z_connectors:DG135T-10.16-02P, symbol Connector:Screw_Terminal_01x02
- added J4, J7: Screw_Terminal_01x01, Z_pin:PinD1_6mm, symbol Connector:Screw_Terminal_01x01
- added J5, J6: Screw_Terminal_01x01, Z_pin:PinD4mm, symbol Connector:Screw_Terminal_01x01
- J1: footprint Z_connectors:DG135T-10.16-03P -> Z_connectors:DB129V-7.62-3P-GN-S; JLCPCB Part (none) -> C395859; MFR.Part (none) -> DB129V-7.62-3P-GN-S
- J2: footprint Z_connectors:DG135T-10.16-02P -> Z_connectors:DB129V-7.62-2P-GN-S; JLCPCB Part (none) -> C395858; MFR.Part (none) -> DB129V-7.62-2P-GN-S
Connections:
- net +12V: now also J4.1 (Pin_1)
- net GND: now also J7.1 (Pin_1)
- net at C9.2, D2.1 (+): now also J6.1 (Pin_1)
- net at C9.1, D2.4 (-): now also J5.1 (Pin_1)
Changed lines of the file:
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@@
   (junction (at 120.65 50.8) (diameter 0) (color 0 0 0 0)
   )
+  (junction (at 96.52 78.74) (diameter 0) (color 0 0 0 0)
+  )
   (junction (at 71.12 167.64) (diameter 0) (color 0 0 0 0)
   )
@@
   )
   (junction (at 171.45 134.62) (diameter 0) (color 0 0 0 0)
+  )
+  (junction (at 96.52 83.82) (diameter 0) (color 0 0 0 0)
   )
   (junction (at 106.68 151.13) (diameter 0) (color 0 0 0 0)
@@
     (stroke (width 0) (type default))
   )
-  (wire (pts (xy 194.31 39.37) (xy 199.39 39.37))
+  (wire (pts (xy 194.31 43.18) (xy 199.39 43.18))
     (stroke (width 0) (type default))
   )
@@
     (stroke (width 0) (type default))
   )
+  (wire (pts (xy 96.52 83.82) (xy 101.6 83.82))
+    (stroke (width 0) (type default))
+  )
   (wire (pts (xy 128.27 95.25) (xy 143.51 95.25))
     (stroke (width 0) (type default))
@@
     (stroke (width 0) (type default))
   )
-  (wire (pts (xy 194.31 30.48) (xy 194.31 36.83))
+  (wire (pts (xy 194.31 30.48) (xy 194.31 35.56))
     (stroke (width 0) (type default))
   )
@@
     (stroke (width 0) (type default))
   )
-  (wire (pts (xy 194.31 36.83) (xy 199.39 36.83))
+  (wire (pts (xy 194.31 35.56) (xy 199.39 35.56))
     (stroke (width 0) (type default))
   )
@@
     (stroke (width 0) (type default))
   )
-  (wire (pts (xy 194.31 48.26) (xy 194.31 39.37))
+  (wire (pts (xy 194.31 48.26) (xy 194.31 43.18))
     (stroke (width 0) (type default))
   )
@@
   )
   (wire (pts (xy 138.43 161.29) (xy 138.43 167.64))
+    (stroke (width 0) (type default))
+  )
+  (wire (pts (xy 96.52 78.74) (xy 101.6 78.74))
     (stroke (width 0) (type default))
   )
@@
       (effects (font (size 1.27 1.27)) (justify left) hide)
     )
-    (property "Footprint" "Z_connectors:DG135T-10.16-03P" (at 48.26 57.15 0)
+    (property "Footprint" "Z_connectors:DB129V-7.62-3P-GN-S" (at 48.26 57.15 0)
       (effects (font (size 1.27 1.27)) hide)
     )
@@
       (effects (font (size 1.27 1.27)) hide)
     )
-    (property "Description" "" (at 48.26 57.15 0)
+    (property "Description" "1x3P 24A -40℃~+105℃ 250V Green 12~26 Straight pin 7.62mm 2.5 1 3 Plugin,P=7.62mm Screw terminal ROHS" (at 48.26 57.15 0)
+      (effects (font (size 1.27 1.27)) hide)
+    )
+    (property "JLCPCB Part" "C395859" (at 48.26 57.15 0)
+      (effects (font (size 1.27 1.27)) hide)
+    )
+    (property "MFR.Part" "DB129V-7.62-3P-GN-S" (at 48.26 57.15 0)
       (effects (font (size 1.27 1.27)) hide)
     )
@@
       (effects (font (size 1.27 1.27)) (justify left) hide)
     )
-    (property "Footprint" "Z_connectors:DG135T-10.16-02P" (at 52.07 111.76 0)
+    (property "Footprint" "Z_connectors:DB129V-7.62-2P-GN-S" (at 52.07 111.76 0)
       (effects (font (size 1.27 1.27)) hide)
     )
@@
       (effects (font (size 1.27 1.27)) hide)
     )
-    (property "Description" "" (at 52.07 111.76 0)
+    (property "Description" "1x2P 24A -40℃~+105℃ 250V Green 12~26 Straight pin 7.62mm 2.5 1 2 Plugin,P=7.62mm Screw terminal ROHS" (at 52.07 111.76 0)
+      (effects (font (size 1.27 1.27)) hide)
+    )
+    (property "JLCPCB Part" "C395858" (at 52.07 111.76 0)
+      (effects (font (size 1.27 1.27)) hide)
+    )
+    (property "MFR.Part" "DB129V-7.62-2P-GN-S" (at 52.07 111.76 0)
       (effects (font (size 1.27 1.27)) hide)
     )
@@
     )
   )
-  (symbol (lib_id "Connector:Screw_Terminal_01x02") (at 204.47 39.37 0) (mirror x) (unit 1)
-    (in_bom yes) (on_board yes) (dnp no)
-    (property "Reference" "J4" (at 204.47 41.91 0)
-      (effects (font (size 1.27 1.27)))
-    )
-    (property "Value" "Screw_Terminal_01x02" (at 204.47 34.29 0)
-      (effects (font (size 1.27 1.27)) hide)
-    )
-    (property "Footprint" "Z_connectors:DG135T-10.16-02P" (at 204.47 39.37 0)
-      (effects (font (size 1.27 1.27)) hide)
-    )
-    (property "Datasheet" "~" (at 204.47 39.37 0)
-      (effects (font (size 1.27 1.27)) hide)
-    )
-    (property "Description" "" (at 204.47 39.37 0)
-      (effects (font (size 1.27 1.27)) hide)
-    )
-    (pin "1")
-    (pin "2")
-    (instances
-      (project "Module_3"
-        (path "/b93deadb-f253-4391-86ff-d3610036e76a"
-          (reference "J4") (unit 1)
-        )
-      )
-    )
-  )
   (symbol (lib_id "Device:L_Iron_Coupled_1423") (at 86.36 48.26 0) (unit 1)
     (in_bom yes) (on_board yes) (dnp no)
@@
     )
   )
+  (symbol (lib_id "Connector:Screw_Terminal_01x01") (at 204.47 35.56 0) (unit 1)
+    (in_bom yes) (on_board yes) (dnp no) (fields_autoplaced)
+    (property "Reference" "J5" (at 207.01 34.925 0)
+      (effects (font (size 1.27 1.27)) (justify left))
+    )
+    (property "Value" "Screw_Terminal_01x01" (at 207.01 37.465 0)
+      (effects (font (size 1.27 1.27)) (justify left) hide)
+    )
+    (property "Footprint" "Z_pin:PinD4mm" (at 204.47 35.56 0)
+      (effects (font (size 1.27 1.27)) hide)
+    )
+    (property "Datasheet" "~" (at 204.47 35.56 0)
+      (effects (font (size 1.27 1.27)) hide)
+    )
+    (pin "1")
+    (instances
+      (project "Module_3"
+        (path "/b93deadb-f253-4391-86ff-d3610036e76a"
+          (reference "J5") (unit 1)
+        )
+      )
+    )
+  )
   (symbol (lib_id "power:GND") (at 83.82 170.18 0) (unit 1)
     (in_bom yes) (on_board yes) (dnp no) (fields_autoplaced)
@@
         (path "/b93deadb-f253-4391-86ff-d3610036e76a"
           (reference "R2") (unit 1)
+        )
+      )
+    )
+  )
+  (symbol (lib_id "Connector:Screw_Terminal_01x01") (at 106.68 83.82 0) (unit 1)
+    (in_bom yes) (on_board yes) (dnp no)
+    (property "Reference" "J7" (at 110.49 83.82 0)
+      (effects (font (size 1.27 1.27)))
+    )
+    (property "Value" "Screw_Terminal_01x01" (at 106.68 86.36 0)
+      (effects (font (size 1.27 1.27)) hide)
+    )
+    (property "Footprint" "Z_pin:PinD1_6mm" (at 106.68 83.82 0)
+      (effects (font (size 1.27 1.27)) hide)
+    )
+    (property "Datasheet" "~" (at 106.68 83.82 0)
+      (effects (font (size 1.27 1.27)) hide)
+    )
+    (pin "1")
+    (instances
+      (project "Module_3"
+        (path "/b93deadb-f253-4391-86ff-d3610036e76a"
+          (reference "J7") (unit 1)
         )
       )
@@
     )
   )
+  (symbol (lib_id "Connector:Screw_Terminal_01x01") (at 106.68 78.74 0) (unit 1)
+    (in_bom yes) (on_board yes) (dnp no)
+    (property "Reference" "J4" (at 109.22 78.74 0)
+      (effects (font (size 1.27 1.27)) (justify left))
+    )
+    (property "Value" "Screw_Terminal_01x01" (at 109.22 80.645 0)
+      (effects (font (size 1.27 1.27)) (justify left) hide)
+    )
+    (property "Footprint" "Z_pin:PinD1_6mm" (at 106.68 78.74 0)
+      (effects (font (size 1.27 1.27)) hide)
+    )
+    (property "Datasheet" "~" (at 106.68 78.74 0)
+      (effects (font (size 1.27 1.27)) hide)
+    )
+    (pin "1")
+    (instances
+      (project "Module_3"
+        (path "/b93deadb-f253-4391-86ff-d3610036e76a"
+          (reference "J4") (unit 1)
+        )
+      )
+    )
+  )
   (symbol (lib_id "Device:C_Small") (at 120.65 48.26 0) (unit 1)
     (in_bom yes) (on_board yes) (dnp no) (fields_autoplaced)
@@
         )
       )
+    )
+  )
+  (symbol (lib_id "Connector:Screw_Terminal_01x01") (at 204.47 43.18 0) (unit 1)
+    (in_bom yes) (on_board yes) (dnp no) (fields_autoplaced)
+    (property "Reference" "J6" (at 207.01 42.545 0)
+      (effects (font (size 1.27 1.27)) (justify left))
+    )
+    (property "Value" "Screw_Terminal_01x01" (at 207.01 45.085 0)
+      (effects (font (size 1.27 1.27)) (justify left) hide)
+    )
+    (property "Footprint" "Z_pin:PinD4mm" (at 204.47 43.18 0)
+      (effects (font (size 1.27 1.27)) hide)
+    )
+    (property "Datasheet" "~" (at 204.47 43.18 0)
+      (effects (font (size 1.27 1.27)) hide)
+    )
+    (pin "1")
+    (instances
+      (project "Module_3"
+        (path "/b93deadb-f253-4391-86ff-d3610036e76a"
+          (reference "J6") (unit 1)
+        )
+      )

Commit message: add bom module 1
Parts:
- C1: LCSC (none) -> C432444
- C2, C3, C4: LCSC (none) -> C518924
- C5, C6: LCSC (none) -> C2914701
- C7: LCSC (none) -> C159828
- C9: LCSC (none) -> C2846750
- D1: LCSC (none) -> C110487
- D2: LCSC (none) -> C970324
- F1: LCSC (none) -> C3029536 2pts
- J1: LCSC (none) -> C395859
- J2: LCSC (none) -> C395858
- L1, L2: LCSC (none) -> B82726S6123N020
- L3: LCSC (none) -> C2981394
- U1: LCSC (none) -> C880552
Changed lines of the file:
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@@
+      (effects (font (size 1.27 1.27)) hide)
+    )
+    (property "LCSC" "C395859" (at 48.26 57.15 0)
       (effects (font (size 1.27 1.27)) hide)
     )
@@
     )
     (property "Description" "" (at 180.34 129.54 0)
+      (effects (font (size 1.27 1.27)) hide)
+    )
+    (property "LCSC" "" (at 180.34 129.54 0)
       (effects (font (size 1.27 1.27)) hide)
     )
@@
       (effects (font (size 1.27 1.27)) hide)
     )
+    (property "LCSC" "C395858" (at 52.07 111.76 0)
+      (effects (font (size 1.27 1.27)) hide)
+    )
     (pin "1")
     (pin "2")
@@
     )
     (property "Description" "60V 700mV@3A 3A SMC(DO-214AB) Schottky Barrier Diodes (SBD)" (at 106.68 158.75 0)
+      (effects (font (size 1.27 1.27)) hide)
+    )
+    (property "LCSC" "C110487" (at 106.68 158.75 0)
       (effects (font (size 1.27 1.27)) hide)
     )
@@
       (effects (font (size 1.27 1.27)) hide)
     )
+    (property "LCSC" "" (at 189.23 87.63 0)
+      (effects (font (size 1.27 1.27)) hide)
+    )
     (pin "1")
     (pin "2")
@@
     )
     (property "MFR.Part" "MBH125-470M" (at 114.3 151.13 0)
+      (effects (font (size 1.27 1.27)) hide)
+    )
+    (property "LCSC" "C2981394" (at 114.3 151.13 0)
       (effects (font (size 1.27 1.27)) hide)
     )
@@
       (effects (font (size 1.27 1.27)) hide)
     )
+    (property "LCSC" "" (at 241.3 144.78 0)
+      (effects (font (size 1.27 1.27)) hide)
+    )
     (instances
       (project "Module_3"
@@
       (effects (font (size 1.27 1.27)) hide)
     )
+    (property "LCSC" "B82726S6123N020" (at 86.36 48.26 0)
+      (effects (font (size 1.27 1.27)) hide)
+    )
     (pin "1")
     (pin "2")
@@
       (effects (font (size 1.27 1.27)) hide)
     )
+    (property "LCSC" "" (at 204.47 35.56 0)
+      (effects (font (size 1.27 1.27)) hide)
+    )
     (pin "1")
     (instances
@@
       (effects (font (size 1.27 1.27)) hide)
     )
+    (property "LCSC" "C518924" (at 96.52 48.26 0)
+      (effects (font (size 1.27 1.27)) hide)
+    )
     (pin "1")
     (pin "2")
@@
     )
     (property "Description" "" (at 147.32 95.25 0)
+      (effects (font (size 1.27 1.27)) hide)
+    )
+    (property "LCSC" "" (at 147.32 95.25 0)
       (effects (font (size 1.27 1.27)) hide)
     )
@@
       (effects (font (size 1.27 1.27)) hide)
     )
+    (property "LCSC" "" (at 106.68 83.82 0)
+      (effects (font (size 1.27 1.27)) hide)
+    )
     (pin "1")
     (instances
@@
       (effects (font (size 1.27 1.27)) hide)
     )
+    (property "LCSC" "B82726S6123N020" (at 110.49 48.26 0)
+      (effects (font (size 1.27 1.27)) hide)
+    )
     (pin "1")
     (pin "2")
@@
       (effects (font (size 1.27 1.27)) hide)
     )
+    (property "LCSC" "" (at 162.56 81.28 0)
+      (effects (font (size 1.27 1.27)) hide)
+    )
     (pin "1")
     (pin "2")
@@
       (effects (font (size 1.27 1.27)) hide)
     )
+    (property "LCSC" "" (at 147.32 81.28 0)
+      (effects (font (size 1.27 1.27)) hide)
+    )
     (pin "1")
     (pin "2")
@@
     )
     (property "MFR.Part" "16YXF220MEFC8X11.5" (at 138.43 158.75 0)
+      (effects (font (size 1.27 1.27)) hide)
+    )
+    (property "LCSC" "C159828" (at 138.43 158.75 0)
       (effects (font (size 1.27 1.27)) hide)
     )
@@
       (effects (font (size 1.27 1.27)) hide)
     )
+    (property "LCSC" "" (at 106.68 78.74 0)
+      (effects (font (size 1.27 1.27)) hide)
+    )
     (pin "1")
     (instances
@@
       (effects (font (size 1.27 1.27)) hide)
     )
+    (property "LCSC" "C518924" (at 120.65 48.26 0)
+      (effects (font (size 1.27 1.27)) hide)
+    )
     (pin "1")
     (pin "2")
@@
     )
     (property "MFR.Part" "3517 2pts" (at 59.69 71.12 0)
+      (effects (font (size 1.27 1.27)) hide)
+    )
+    (property "LCSC" "C3029536 2pts" (at 59.69 71.12 0)
       (effects (font (size 1.27 1.27)) hide)
     )
@@
       (effects (font (size 1.27 1.27)) hide)
     )
+    (property "LCSC" "C970324" (at 160.02 38.1 0)
+      (effects (font (size 1.27 1.27)) hide)
+    )
     (pin "1")
     (pin "2")
@@
       (effects (font (size 1.27 1.27)) hide)
     )
+    (property "LCSC" "" (at 241.3 132.08 0)
+      (effects (font (size 1.27 1.27)) hide)
+    )
     (instances
       (project "Module_3"
@@
       (effects (font (size 1.27 1.27)) hide)
     )
+    (property "LCSC" "C2914701" (at 135.89 50.8 0)
+      (effects (font (size 1.27 1.27)) hide)
+    )
     (pin "1")
     (pin "2")
@@
       (effects (font (size 1.27 1.27)) hide)
     )
+    (property "LCSC" "C518924" (at 71.12 48.26 0)
+      (effects (font (size 1.27 1.27)) hide)
+    )
     (pin "1")
     (pin "2")
@@
     )
     (property "Datasheet" "" (at 80.01 81.28 0)
+      (effects (font (size 1.27 1.27)) hide)
+    )
+    (property "LCSC" "" (at 80.01 81.28 0)
       (effects (font (size 1.27 1.27)) hide)
     )
@@
       (effects (font (size 1.27 1.27)) hide)
     )
+    (property "LCSC" "" (at 204.47 43.18 0)
+      (effects (font (size 1.27 1.27)) hide)
+    )
     (pin "1")
     (instances
@@
     )
     (property "MFR.Part" "LM2576S-5.0/NOPB" (at 83.82 153.67 0)
+      (effects (font (size 1.27 1.27)) hide)
+    )
+    (property "LCSC" "C880552" (at 83.82 153.67 0)
       (effects (font (size 1.27 1.27)) hide)
     )
@@
       (effects (font (size 1.27 1.27)) hide)
     )
+    (property "LCSC" "" (at 217.17 144.78 0)
+      (effects (font (size 1.27 1.27)) hide)
+    )
     (instances
       (project "Module_3"
@@
       (effects (font (size 1.27 1.27)) hide)
     )
+    (property "LCSC" "" (at 162.56 95.25 0)
+      (effects (font (size 1.27 1.27)) hide)
+    )
     (pin "1")
     (pin "2")
@@
     )
     (property "Description" "" (at 173.99 87.63 0)
+      (effects (font (size 1.27 1.27)) hide)
+    )
+    (property "LCSC" "" (at 173.99 87.63 0)
       (effects (font (size 1.27 1.27)) hide)
     )
@@
       (effects (font (size 1.27 1.27)) hide)
     )
+    (property "LCSC" "" (at 232.41 135.89 0)
+      (effects (font (size 1.27 1.27)) hide)
+    )
     (instances
       (project "Module_3"
@@
       (effects (font (size 1.27 1.27)) hide)
     )
+    (property "LCSC" "" (at 217.17 132.08 0)
+      (effects (font (size 1.27 1.27)) hide)
+    )
     (instances
       (project "Module_3"
@@
       (effects (font (size 1.27 1.27)) hide)
     )
+    (property "LCSC" "C2846750" (at 180.34 38.1 0)
+      (effects (font (size 1.27 1.27)) hide)
+    )
     (pin "1")
     (pin "2")
@@
       (effects (font (size 1.27 1.27)) hide)
     )
+    (property "LCSC" "C432444" (at 57.15 158.75 0)
+      (effects (font (size 1.27 1.27)) hide)
+    )
     (pin "1")
     (pin "2")
@@
       (effects (font (size 1.27 1.27)) hide)
     )
+    (property "LCSC" "C2914701" (at 135.89 43.18 0)
+      (effects (font (size 1.27 1.27)) hide)
+    )
