File: Projects/StationModules/Module_3/Module_3.kicad_sch (KiCad schematic)
At the start: 34 parts, among them J1 Screw_Terminal_01x03, J2 Screw_Terminal_01x02, J4 Screw_Terminal_01x01, J5 Screw_Terminal_01x01, J6 Screw_Terminal_01x01, J7 Screw_Terminal_01x01, U1 LM2576S-5, U2 PC814

Commit message: add bom and pos
Parts:
- C1: JLCPCB Part C432444 -> (none)
- C2, C3, C4: JLCPCB Part C518924 -> (none)
- C5, C6: JLCPCB Part C2914701 -> (none)
- C7: JLCPCB Part C159828 -> (none)
- C8: LCSC (none) -> C23631; MFR.Part (none) -> CC1206KKX7RDBB102
- C9: JLCPCB Part C2846750 -> (none)
- D1: JLCPCB Part C110487 -> (none)
- D2: JLCPCB Part C970324 -> (none)
- F1: JLCPCB Part C3029536 2pts -> (none); LCSC C3029536 2pts -> C3029536; MFR.Part 3517 2pts -> 3517
- J1: JLCPCB Part C395859 -> (none)
- J2: JLCPCB Part C395858 -> (none)
- J3: LCSC (none) -> C6332196; MFR.Part (none) -> HB-PH3-25413PB2GOP
- L3: JLCPCB Part C2981394 -> (none)
- R1, R2, R3, R4: LCSC (none) -> C137234; MFR.Part (none) -> RC1206FR-0775KL
- U1: JLCPCB Part C880552 -> (none)
- U2: LCSC (none) -> C2833074; MFR.Part (none) -> PC817X2YSZW
Changed lines of the file:
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@@
-      (effects (font (size 1.27 1.27)) hide)
-    )
-    (property "JLCPCB Part" "C395859" (at 48.26 57.15 0)
       (effects (font (size 1.27 1.27)) hide)
     )
@@
       (effects (font (size 1.27 1.27)) hide)
     )
-    (property "Description" "" (at 180.34 129.54 0)
-      (effects (font (size 1.27 1.27)) hide)
-    )
-    (property "LCSC" "" (at 180.34 129.54 0)
+    (property "Description" "Gold 250V 3A Straight Square Pins 2.54mm 3P 260℃ 6mm -40℃~+105℃ 3mm 2.54mm Brass Black Plugin 2.54mm 1x3P Plugin,P=2.54mm Pin Headers ROHS" (at 180.34 129.54 0)
+      (effects (font (size 1.27 1.27)) hide)
+    )
+    (property "LCSC" "C6332196" (at 180.34 129.54 0)
+      (effects (font (size 1.27 1.27)) hide)
+    )
+    (property "MFR.Part" "HB-PH3-25413PB2GOP" (at 180.34 129.54 0)
       (effects (font (size 1.27 1.27)) hide)
     )
@@
       (effects (font (size 1.27 1.27)) hide)
     )
-    (property "JLCPCB Part" "C395858" (at 52.07 111.76 0)
-      (effects (font (size 1.27 1.27)) hide)
-    )
     (property "MFR.Part" "DB129V-7.62-2P-GN-S" (at 52.07 111.76 0)
       (effects (font (size 1.27 1.27)) hide)
@@
     )
     (property "MFR.Part" "B360-13-F" (at 106.68 158.75 90)
-      (effects (font (size 1.27 1.27)) hide)
-    )
-    (property "JLCPCB Part" "C110487" (at 106.68 158.75 90)
       (effects (font (size 1.27 1.27)) hide)
     )
@@
       (effects (font (size 1.27 1.27)) (justify left) hide)
     )
-    (property "Description" "" (at 189.23 87.63 0)
-      (effects (font (size 1.27 1.27)) hide)
-    )
-    (property "LCSC" "" (at 189.23 87.63 0)
+    (property "Description" "80V 5000V 50mA 0.1V@1mA,20mA 1 6V 1.2V DC DIP-4 Optocouplers - Phototransistor Output ROHS" (at 189.23 87.63 0)
+      (effects (font (size 1.27 1.27)) hide)
+    )
+    (property "LCSC" "C2833074" (at 189.23 87.63 0)
+      (effects (font (size 1.27 1.27)) hide)
+    )
+    (property "MFR.Part" "PC817X2YSZW" (at 189.23 87.63 0)
       (effects (font (size 1.27 1.27)) hide)
     )
@@
     )
     (property "Description" "47uH SMD,12.5x12.5mm Power Inductors ROHS" (at 114.3 151.13 0)
-      (effects (font (size 1.27 1.27)) hide)
-    )
-    (property "JLCPCB Part" "C2981394" (at 114.3 151.13 0)
       (effects (font (size 1.27 1.27)) hide)
     )
@@
       (effects (font (size 1.27 1.27)) hide)
     )
-    (property "JLCPCB Part" "C518924" (at 96.52 48.26 0)
-      (effects (font (size 1.27 1.27)) hide)
-    )
     (property "MFR.Part" "CBB80-400V-474J" (at 96.52 48.26 0)
       (effects (font (size 1.27 1.27)) hide)
@@
       (effects (font (size 1.27 1.27)) hide)
     )
-    (property "Description" "" (at 147.32 95.25 0)
-      (effects (font (size 1.27 1.27)) hide)
-    )
-    (property "LCSC" "" (at 147.32 95.25 0)
+    (property "Description" "250mW Thick Film Resistors ±100ppm/℃ ±1% 75kΩ 1206 Chip Resistor - Surface Mount ROHS" (at 147.32 95.25 0)
+      (effects (font (size 1.27 1.27)) hide)
+    )
+    (property "LCSC" "C137234" (at 147.32 95.25 0)
+      (effects (font (size 1.27 1.27)) hide)
+    )
+    (property "MFR.Part" "RC1206FR-0775KL" (at 147.32 95.25 0)
       (effects (font (size 1.27 1.27)) hide)
     )
@@
       (effects (font (size 1.27 1.27)) hide)
     )
-    (property "Description" "" (at 162.56 81.28 0)
-      (effects (font (size 1.27 1.27)) hide)
-    )
-    (property "LCSC" "" (at 162.56 81.28 0)
+    (property "Description" "250mW Thick Film Resistors ±100ppm/℃ ±1% 75kΩ 1206 Chip Resistor - Surface Mount ROHS" (at 162.56 81.28 0)
+      (effects (font (size 1.27 1.27)) hide)
+    )
+    (property "LCSC" "C137234" (at 162.56 81.28 0)
+      (effects (font (size 1.27 1.27)) hide)
+    )
+    (property "MFR.Part" "RC1206FR-0775KL" (at 162.56 81.28 0)
       (effects (font (size 1.27 1.27)) hide)
     )
@@
       (effects (font (size 1.27 1.27)) hide)
     )
-    (property "Description" "" (at 147.32 81.28 0)
-      (effects (font (size 1.27 1.27)) hide)
-    )
-    (property "LCSC" "" (at 147.32 81.28 0)
+    (property "Description" "250mW Thick Film Resistors ±100ppm/℃ ±1% 75kΩ 1206 Chip Resistor - Surface Mount ROHS" (at 147.32 81.28 0)
+      (effects (font (size 1.27 1.27)) hide)
+    )
+    (property "LCSC" "C137234" (at 147.32 81.28 0)
+      (effects (font (size 1.27 1.27)) hide)
+    )
+    (property "MFR.Part" "RC1206FR-0775KL" (at 147.32 81.28 0)
       (effects (font (size 1.27 1.27)) hide)
     )
@@
     )
     (property "Description" "220uF ±20% 16V 8mm 11.5mm 3.5mm 400mA 100kHz 250mΩ 100kHz 7000Hrs @ 105℃ -40℃ ~ +105℃ ,8x11.5mm Aluminum Electrolytic Capacitors - Leaded RoHS" (at 138.43 158.75 0)
-      (effects (font (size 1.27 1.27)) hide)
-    )
-    (property "JLCPCB Part" "C159828" (at 138.43 158.75 0)
       (effects (font (size 1.27 1.27)) hide)
     )
@@
       (effects (font (size 1.27 1.27)) hide)
     )
-    (property "JLCPCB Part" "C518924" (at 120.65 48.26 0)
-      (effects (font (size 1.27 1.27)) hide)
-    )
     (property "MFR.Part" "CBB80-400V-474J" (at 120.65 48.26 0)
       (effects (font (size 1.27 1.27)) hide)
@@
       (effects (font (size 1.27 1.27)) hide)
     )
-    (property "JLCPCB Part" "C3029536 2pts" (at 59.69 71.12 0)
-      (effects (font (size 1.27 1.27)) hide)
-    )
-    (property "MFR.Part" "3517 2pts" (at 59.69 71.12 0)
-      (effects (font (size 1.27 1.27)) hide)
-    )
-    (property "LCSC" "C3029536 2pts" (at 59.69 71.12 0)
+    (property "MFR.Part" "3517" (at 59.69 71.12 0)
+      (effects (font (size 1.27 1.27)) hide)
+    )
+    (property "LCSC" "C3029536" (at 59.69 71.12 0)
       (effects (font (size 1.27 1.27)) hide)
     )
@@
       (effects (font (size 1.27 1.27)) hide)
     )
-    (property "JLCPCB Part" "C970324" (at 160.02 38.1 0)
-      (effects (font (size 1.27 1.27)) hide)
-    )
     (property "MFR.Part" "GBU15M" (at 160.02 38.1 0)
       (effects (font (size 1.27 1.27)) hide)
@@
       (effects (font (size 1.27 1.27)) hide)
     )
-    (property "JLCPCB Part" "C2914701" (at 135.89 50.8 0)
-      (effects (font (size 1.27 1.27)) hide)
-    )
     (property "MFR.Part" "R06B1E221KN0B0S0N0" (at 135.89 50.8 0)
       (effects (font (size 1.27 1.27)) hide)
@@
     )
     (property "Description" "470nF ±5% 400V Plugin,P=22.5mm Polypropylene Film Capacitors" (at 71.12 48.26 0)
-      (effects (font (size 1.27 1.27)) hide)
-    )
-    (property "JLCPCB Part" "C518924" (at 71.12 48.26 0)
       (effects (font (size 1.27 1.27)) hide)
     )
@@
       (effects (font (size 1.27 1.27)) hide)
     )
-    (property "JLCPCB Part" "C880552" (at 83.82 153.67 0)
-      (effects (font (size 1.27 1.27)) hide)
-    )
     (property "MFR.Part" "LM2576S-5.0/NOPB" (at 83.82 153.67 0)
       (effects (font (size 1.27 1.27)) hide)
@@
       (effects (font (size 1.27 1.27)) hide)
     )
-    (property "Description" "" (at 162.56 95.25 0)
-      (effects (font (size 1.27 1.27)) hide)
-    )
-    (property "LCSC" "" (at 162.56 95.25 0)
+    (property "Description" "250mW Thick Film Resistors ±100ppm/℃ ±1% 75kΩ 1206 Chip Resistor - Surface Mount ROHS" (at 162.56 95.25 0)
+      (effects (font (size 1.27 1.27)) hide)
+    )
+    (property "LCSC" "C137234" (at 162.56 95.25 0)
+      (effects (font (size 1.27 1.27)) hide)
+    )
+    (property "MFR.Part" "RC1206FR-0775KL" (at 162.56 95.25 0)
       (effects (font (size 1.27 1.27)) hide)
     )
@@
       (effects (font (size 1.27 1.27)) hide)
     )
-    (property "Description" "" (at 173.99 87.63 0)
-      (effects (font (size 1.27 1.27)) hide)
-    )
-    (property "LCSC" "" (at 173.99 87.63 0)
+    (property "Description" "2kV 1nF X7R ±10% 1206 Multilayer Ceramic Capacitors MLCC - SMD/SMT ROHS" (at 173.99 87.63 0)
+      (effects (font (size 1.27 1.27)) hide)
+    )
+    (property "LCSC" "C23631" (at 173.99 87.63 0)
+      (effects (font (size 1.27 1.27)) hide)
+    )
+    (property "MFR.Part" "CC1206KKX7RDBB102" (at 173.99 87.63 0)
       (effects (font (size 1.27 1.27)) hide)
     )
@@
       (effects (font (size 1.27 1.27)) hide)
     )
-    (property "JLCPCB Part" "C2846750" (at 180.34 38.1 0)
-      (effects (font (size 1.27 1.27)) hide)
-    )
     (property "MFR.Part" "1DH547D400-06" (at 180.34 38.1 0)
       (effects (font (size 1.27 1.27)) hide)
@@
       (effects (font (size 1.27 1.27)) hide)
     )
-    (property "JLCPCB Part" "C432444" (at 57.15 158.75 0)
-      (effects (font (size 1.27 1.27)) hide)
-    )
     (property "MFR.Part" "16YXJ470M8X11.5" (at 57.15 158.75 0)
       (effects (font (size 1.27 1.27)) hide)
@@
       (effects (font (size 1.27 1.27)) hide)
     )
-    (property "JLCPCB Part" "C2914701" (at 135.89 43.18 0)
-      (effects (font (size 1.27 1.27)) hide)
-    )

Commit message: change on 25_02_24
Parts:
- added C10: 0.1uF, Capacitor_SMD:C_1206_3216Metric, symbol Device:C_Small
- added R5: 1M, Resistor_SMD:R_1206_3216Metric, symbol Device:R
- added R6, R7, R8: 330k, Resistor_SMD:R_1206_3216Metric, symbol Device:R
- C1, C8, D1, J1, J2, L1, L2, L3, R1, R2, R3, R4, U2: Mounting (none) -> Yes
- C2, C3, C4: LCSC C518924 -> C2803198; MFR.Part CBB80-400V-474J -> MPP474J2J20AJ22800; Mounting (none) -> Yes
- C5, C6: LCSC C2914701 -> C249173; MFR.Part R06B1E221KN0B0S0N0 -> S07B1E221KN0B0S0N0; Mounting (none) -> Yes
- C7: LCSC C159828 -> C334323; MFR.Part 16YXF220MEFC8X11.5 -> 16YXF220MFFC8X11.5; Mounting (none) -> Yes
- C9: LCSC C2846750 -> C3019080; MFR.Part 1DH547D400-06 -> KP475J2J2603; Mounting (none) -> Yes
- D2, H1, H2, H3, H4, H5, J4, J7, M1: Mounting (none) -> No
- F1: footprint Fuse:Fuseholder_Clip-5x20mm_Keystone_3517_Inline_P23.11x6.76mm_D1.70mm_Horizontal -> Fuse:Fuse_Littelfuse_395Series; LCSC C3029536 -> C354900; MFR.Part 3517 -> 2010T1A250V; Mounting (none) -> Yes
- J3: LCSC C6332196 -> C5665; MFR.Part HB-PH3-25413PB2GOP -> C5665; Mounting (none) -> Yes
- J5, J6: footprint Z_pin:PinD4mm -> Z_pin:PinD3mm; Mounting (none) -> No
- U1: LCSC C880552 -> C347413; MFR.Part LM2576S-5.0/NOPB -> LM2576S-5; Mounting (none) -> Yes
Connections:
- net +12V: now also M1.3 (+12V); no longer M1.4 (+12V)
- net F_IN: now also C10.1, R5.2
- net GND: now also M1.4 (GND), C10.2, R5.1; no longer M1.3 (GND)
- net at C2.2, J1.1 (Pin_1), L1.2: no longer F1.1
- net at C2.1, J1.2 (Pin_2), L1.1: no longer M1.1 (AC_220)
- net at C3.2, L1.3, L2.2: now also M1.2 (AC_220)
- net at C3.1, L1.4, L2.1: now also F1.1
- net at C9.1, D2.4 (-), J5.1 (Pin_1): now also R6.2
- net at C4.2, C6.2, D2.3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: now also L2.4; no longer L2.3
- net at C4.1, C5.1, D2.2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: now also L2.3; no longer L2.4
- net at F1.2: now also M1.1 (AC_220); no longer M1.2 (AC_220)
- net at C9.2, D2.1 (+), J6.1 (Pin_1): now also R8.2
- new net: R7.1, R8.1
- new net: R6.1, R7.2
- no-connect marks 1 -> 0

Commit message: Corection all modules
Parts:
- added D3: 1.5KExxCA, Diode_THT:D_DO-201AE_P15.24mm_Horizontal, symbol Diode:1.5KExxCA
- added F2: Fuse, Resistor_THT:R_Axial_Power_L20.0mm_W6.4mm_P25.40mm, symbol Device:Fuse
- added PS1: HLK-PM12, Converter_ACDC:Converter_ACDC_HiLink_HLK-5Mxx, symbol Converter_ACDC:HLK-PM12
- added RV1: Varistor, Varistor:RV_Disc_D21.5mm_W4.3mm_P10mm, symbol Device:Varistor
- C2, C3, C4: value 470nF -> 1uF; footprint Capacitor_THT:C_Rect_L24.0mm_W10.9mm_P22.50mm_MKT -> Capacitor_THT:C_Rect_L18.0mm_W11.0mm_P15.00mm_FKS3_FKP3; LCSC C2803198 -> C504224; MFR.Part MPP474J2J20AJ22800 -> MPX105K31D5KN15800
- L1, L2: footprint Z_inductors:B82726S6123N020 -> Z_inductors:FilterSetevoy_20x30_p20
- U2: LCSC C2833074 -> C7435550; MFR.Part PC817X2YSZW -> LTV-814-B
Connections:
- net +12V: now also PS1.4 (+Vout)
- net GND: now also PS1.3 (-Vout)
- net at C2.2, L1.2: now also J1.2 (Pin_2), D3.2 (A2), RV1.2; no longer J1.1 (Pin_1)
- net at C2.1, L1.1: now also D3.1 (A1), F2.2, RV1.1; no longer J1.2 (Pin_2)
- net at C3.2, L1.3, L2.2: no longer M1.2 (AC_220)
- net at C3.1, L1.4, L2.1: no longer F1.1
- net at C4.2, C6.2, D2.3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: now also L2.3, M1.2 (AC_220), PS1.2 (AC/N); no longer L2.4
- net at C4.1, C5.1, D2.2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: now also F1.1, L2.4; no longer L2.3
- net at F1.2, M1.1 (AC_220): now also PS1.1 (AC/L)
- new net: F2.1, J1.1 (Pin_1)
Other:
- moved on the sheet: J1
